File: mainboard/mainboard.brd (EAGLE design)
At the start: 100 x 61 mm, 25 parts, among them J1 BATTERY_CONNDEANS, J1Z CLONOLU, J1Z1 CLONOLU, P1 IMU, P2 analogin, P3 analogin, P4 I2C, U1 DWM1000, U2 ESP8266, X1 04-JST-B4B-XH-A, X2 04-JST-B4B-XH-A

Commit message: allsmd
Parts:
- removed J1Z, J1Z1: CLONOLU, pololu-allegro:CLONOLU
- removed U$2: ARDUINONANO, CRE-Lib1:PDIP-32
- removed U$3: 03-JST-B3B-XH-A, bt_con-jst-xh:B3B-XH
- added JP1: Nucleo R, pinhead-2:1X15SMD
- added JP2: Nucleo L, pinhead-2:1X15SMD
- added JP3: Motor LR, pinhead-2:1X07SMD
- added JP4: Motor LL, pinhead-2:1X07SMD
- added JP5: Motor RL, pinhead-2:1X07SMD
- added JP6: Motor RR, pinhead-2:1X07SMD
Connections:
- removed net GND$1: J1Z.GND$1, J1Z1.GND$1
- removed net GND$2: J1Z.GND$2, J1Z1.GND$2
- net N$17: no longer J1Z.VMOT
- net N$18: no longer J1Z1.VMOT
- net N$19: no longer J1Z.2B
- net N$20: no longer J1Z.2A
- net N$21: no longer J1Z.1A
- net N$22: no longer J1Z.1B
- net N$23: no longer J1Z1.2B
- net N$24: no longer J1Z1.2A
- net N$25: no longer J1Z1.1A
- net N$26: no longer J1Z1.1B
- net VDD: no longer J1Z.VDD, J1Z1.VDD
Changed lines of the file:
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@@
 </autorouter>
 <elements>
-<element name="J1Z" library="pololu-allegro" package="CLONOLU" value="CLONOLU" x="71.12" y="12.7"/>
-<element name="J1Z1" library="pololu-allegro" package="CLONOLU" value="CLONOLU" x="20.32" y="12.7"/>
 <element name="LED1" library="WS2812B" package="WS2812B" value="WS2812B" x="24.13" y="55.88"/>
 <element name="P1" library="jst-ph" package="JST-PH4" value="IMU" x="91.44" y="24.13" rot="R270"/>
@@
 <element name="S1" library="switch" package="255SB" value="" x="52.07" y="55.88"/>
 <element name="U$1" library="ST1S10PHR" package="HSOP8" value="ST1S10PHR" x="67.31" y="46.99"/>
-<element name="U$2" library="CRE-Lib1" package="PDIP-32" value="ARDUINONANO" x="43.18" y="41.91"/>
-<element name="U$3" library="bt_con-jst-xh" package="B3B-XH" value="03-JST-B3B-XH-A" x="25.4" y="41.91" rot="R90"/>
 <element name="U1" library="DWM1000" package="XCVR_DWM1000" value="DWM1000" x="8.89" y="46.99"/>
 <element name="U2" library="esp8266modules" package="ESP12-SMD" value="ESP8266" x="88.9" y="45.72"/>
@@
 <element name="C6" library="rcl" package="153CLV-0405" value="" x="21.59" y="26.67" rot="R180"/>
 <element name="J1" library="SparkFun-Connectors" package="DEANS" value="BATTERY_CONNDEANS" x="36.83" y="57.15"/>
+<element name="JP1" library="pinhead-2" package="1X15SMD" value="Nucleo R" x="57.15" y="36.83" rot="R270"/>
+<element name="JP2" library="pinhead-2" package="1X15SMD" value="Nucleo L" x="43.18" y="36.83" rot="R270"/>
+<element name="JP3" library="pinhead-2" package="1X07SMD" value="Motor LR" x="27.94" y="16.51" rot="R270"/>
+<element name="JP4" library="pinhead-2" package="1X07SMD" value="Motor LL" x="17.78" y="16.51" rot="R270"/>
+<element name="JP5" library="pinhead-2" package="1X07SMD" value="Motor RL" x="74.93" y="16.51" rot="R270"/>
+<element name="JP6" library="pinhead-2" package="1X07SMD" value="Motor RR" x="66.04" y="16.51" rot="R270"/>
 </elements>
 <signals>
@@
 <wire x1="15.29" y1="48.79" x2="15.29" y2="47.39" width="0" layer="19" extent="1-1"/>
 </signal>
-<signal name="GND$1">
-<contactref element="J1Z" pad="GND$1"/>
-<contactref element="J1Z1" pad="GND$1"/>
-<wire x1="26.67" y1="19.05" x2="77.47" y2="19.05" width="0" layer="19" extent="1-1"/>
-</signal>
 <signal name="VDD">
-<contactref element="J1Z" pad="VDD"/>
-<contactref element="J1Z1" pad="VDD"/>
 <contactref element="LED1" pad="VDD"/>
-<wire x1="26.67" y1="6.35" x2="22.13" y2="57.58" width="0" layer="19" extent="1-1"/>
-<wire x1="77.47" y1="6.35" x2="26.67" y2="6.35" width="0" layer="19" extent="1-1"/>
-</signal>
-<signal name="GND$2">
-<contactref element="J1Z" pad="GND$2"/>
-<contactref element="J1Z1" pad="GND$2"/>
-<wire x1="26.67" y1="3.81" x2="77.47" y2="3.81" width="0" layer="19" extent="1-1"/>
 </signal>
 <signal name="GND">
@@
 <contactref element="LED1" pad="DIN"/>
 </signal>
-<signal name="N$17">
-<contactref element="C5" pad="+"/>
-<contactref element="J1Z" pad="VMOT"/>
-<wire x1="82.02" y1="27.94" x2="77.47" y2="21.59" width="0" layer="19" extent="1-1"/>
-</signal>
-<signal name="N$18">
-<contactref element="J1Z1" pad="VMOT"/>
-<contactref element="C6" pad="+"/>
-<wire x1="26.67" y1="21.59" x2="19.79" y2="26.67" width="0" layer="19" extent="1-1"/>
-</signal>
 <signal name="N$19">
 <contactref element="X2" pad="P$4"/>
-<contactref element="J1Z" pad="2B"/>
-<wire x1="85.09" y1="16.51" x2="77.47" y2="16.51" width="0" layer="19" extent="1-1"/>
 </signal>
 <signal name="N$20">
-<contactref element="J1Z" pad="2A"/>
 <contactref element="X2" pad="P$3"/>
-<wire x1="85.09" y1="13.97" x2="77.47" y2="13.97" width="0" layer="19" extent="1-1"/>
 </signal>
 <signal name="N$21">
 <contactref element="X2" pad="P$2"/>
-<contactref element="J1Z" pad="1A"/>
-<wire x1="85.09" y1="11.43" x2="77.47" y2="11.43" width="0" layer="19" extent="1-1"/>
 </signal>
 <signal name="N$22">
 <contactref element="X2" pad="P$1"/>
-<contactref element="J1Z" pad="1B"/>
-<wire x1="85.09" y1="8.89" x2="77.47" y2="8.89" width="0" layer="19" extent="1-1"/>
 </signal>
 <signal name="N$23">
 <contactref element="X1" pad="P$4"/>
-<contactref element="J1Z1" pad="2B"/>
-<wire x1="26.67" y1="16.51" x2="35.56" y2="16.51" width="0" layer="19" extent="1-1"/>
 </signal>
 <signal name="N$24">
 <contactref element="X1" pad="P$3"/>
-<contactref element="J1Z1" pad="2A"/>
-<wire x1="26.67" y1="13.97" x2="35.56" y2="13.97" width="0" layer="19" extent="1-1"/>
 </signal>
 <signal name="N$25">
 <contactref element="X1" pad="P$2"/>
-<contactref element="J1Z1" pad="1A"/>
-<wire x1="26.67" y1="11.43" x2="35.56" y2="11.43" width="0" layer="19" extent="1-1"/>
 </signal>
 <signal name="N$26">
 <contactref element="X1" pad="P$1"/>
-<contactref element="J1Z1" pad="1B"/>
-<wire x1="26.67" y1="8.89" x2="35.56" y2="8.89" width="0" layer="19" extent="1-1"/>
+</signal>
+<signal name="N$17">
+<contactref element="C5" pad="+"/>
+</signal>
+<signal name="N$18">
+<contactref element="C6" pad="+"/>
 </signal>
 </signals>

Commit message: fit
Parts:
- removed J1: BATTERY_CONNDEANS, SparkFun-Connectors:DEANS
- removed P1: IMU, jst-ph:JST-PH4
- removed P2, P3: analogin, jst-ph:JST-PH4
- removed P4: I2C, jst-ph:JST-PH4
- added X3: (no value), con-molex-micro-fit-3_0:43045-0415
- X1, X2: value 04-JST-B4B-XH-A -> (none); device bt_con-jst-xh:B4B-XH -> con-molex-micro-fit-3_0:43045-0412
- moved C1 36.4 mm to (21.6, 31.8), turned to 180 degrees
- moved X2 24.4 mm to (66.0, 27.9), turned to 0 degrees
- moved C4 19.1 mm to (19.1, 40.6)
- moved X1 15.7 mm to (31.8, 27.9), turned to 0 degrees
- moved C5 10.9 mm to (74.9, 21.6)
- moved S1 10.8 mm to (44.5, 48.3)
- moved U2 10.2 mm to (83.8, 36.8)
- moved R1 10.2 mm to (64.8, 48.3)
- moved R2 10.2 mm to (67.3, 48.3)
- moved L1 10.2 mm to (54.6, 49.5)
- moved LED1 10.2 mm to (19.1, 47.0)
- moved U$1 9.16 mm to (59.7, 41.9)
- moved U1 7.73 mm to (7.62, 39.4)
- moved JP5 6.48 mm to (81.3, 15.2)
- moved C2 6.35 mm to (68.6, 39.4)
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Connections:
- removed net N$1: P1.3
- removed net N$10: P3.3
- removed net N$11: P3.2
- removed net N$12: P3.1
- removed net N$13: P4.3
- removed net N$14: P4.2
- removed net N$15: P4.1
- removed net N$3: P1.2
- removed net N$6: P1.1
- removed net N$7: P2.3
- removed net N$8: P2.2
- removed net N$9: P2.1
- net +12V: now also X3.P$3, X3.P$4; no longer J1.+
- net GND: now also X3.P$1, X3.P$2; no longer P1.4, P2.4, P3.4, P4.4
Other:
- board size 100 x 61 mm -> 93.7 x 52.1 mm

Commit message: allparts
Parts:
- removed C1: (no value), rcl:153CLV-0405
- removed C3: (no value), rcl:C0603K
- removed L1: (no value), rcl:L4035M
- removed R1, R2: (no value), rcl:R0603
- removed S1: (no value), switch:255SB
- removed U$1: ST1S10PHR, ST1S10PHR:HSOP8
- removed X3: (no value), con-molex-micro-fit-3_0:43045-0415
- added JP10, JP7, JP8, JP9: 3PIN, jst_eph:B3B-PH-K-S
- added JP11, JP12: 4PIN, jst_eph:B4B-PH-K-S
- added JP13: (no value), pinhead-2:1X04SMD
- added X4: (no value), con-molex-micro-fit-3_0:43045-0412
- JP3: value Motor LR -> (none); device pinhead-2:1X07SMD -> pinhead-2:1X08SMD
- JP4: value Motor LL -> (none); device pinhead-2:1X07SMD -> pinhead-2:1X08SMD
- JP5: value Motor RL -> (none); device pinhead-2:1X07SMD -> pinhead-2:1X08SMD
- JP6: value Motor RR -> (none); device pinhead-2:1X07SMD -> pinhead-2:1X08SMD
- moved LED1 82.1 mm to (88.9, 3.81)
- moved U1 77.5 mm to (85.1, 39.4)
- moved C4 77.4 mm to (90.2, 10.2), turned to 180 degrees
- moved U2 73.7 mm to (10.2, 38.1)
- moved JP5 66.3 mm to (15.2, 21.6)
- moved JP3 51.6 mm to (81.3, 6.35), turned to 90 degrees
- moved X1 40.7 mm to (72.4, 30.5), turned to 90 degrees
- moved X2 36.9 mm to (29.2, 30.5), turned to 90 degrees
- moved JP1 26.7 mm to (57.1, 8.89), turned to 90 degrees
- moved C2 22.9 mm to (47.0, 31.8)
- moved C6 19.1 mm to (20.3, 6.35), turned to 270 degrees
- moved JP4 14.5 mm to (29.2, 6.35), turned to 90 degrees
- moved C5 12.8 mm to (87.6, 20.3), turned to 90 degrees
- moved JP2 7.41 mm to (38.1, 41.9)
- moved JP6 6.84 mm to (66.0, 21.6)
Connections:
- removed net N$16: C4.1, LED1.VSS
- removed net N$17: C5.+
- removed net N$18: C6.+
- removed net N$4: R1.1, R2.2, U$1.3
- removed net N$5: C1.+, C3.1, S1.1, U$1.1, U$1.2, U$1.6
- removed net VDD: LED1.VDD
- removed net VDD3V3: U1.6, U1.7
- removed net VSS: U1.16, U1.21, U1.23, U1.24, U1.8
- new net +3V3: C2.+, JP10.3, JP13.4, JP9.3, U1.6, U1.7, U2.VCC
- new net 3V3: JP1.2
- new net 5V: JP1.12
- new net AREF: JP1.3
- new net CSN: JP1.7
- new net FL: JP5.2
- new net FR: JP3.2
- new net M0L: JP6.2
- new net M0R: JP4.2
- new net M1L: JP6.3
- new net M1R: JP4.3
- new net M2L: JP6.4
- new net M2R: JP4.4
- new net MISO: JP1.9, U1.19
- new net MLDIR: JP1.1, JP6.8
- new net MLEN: JP1.5, JP6.1
- new net MLSTEP: JP1.4, JP6.7
- new net MOSI: JP1.10, U1.18
- new net MRDIR: JP2.13, JP4.8
- new net MREN: JP2.15, JP4.1
- new net MRSTEP: JP2.14, JP4.7
- new net N$1: JP9.1
- new net N$10: JP8.2
- new net N$12: JP3.6, X1.P$1
- new net N$13: JP7.2
- new net N$15: JP3.5, X1.P$2
- new net N$27: JP10.2
- new net N$3: JP9.2
- new net N$7: U1.17
- new net NRST: JP1.13
- new net NRST1: JP2.3
- new net P1: JP2.10
- new net P2: JP2.11
- new net P3: JP2.12
- new net PA12: JP2.5
- new net PA2: JP1.11
- new net PA3: JP1.6
- new net PB0: JP2.6
- new net PB1: JP2.9
- new net RX: JP2.2, U2.TXD0
- new net SCK: JP1.8, U1.20
- new net SCL: JP11.3, JP12.3, JP2.8
- new net SDA: JP11.2, JP12.2, JP2.7
- new net TX: JP2.1, U2.RXD0
- new net VIN: JP1.15
- new net WIPOWER: JP13.1
- net +12V: now also C5.+, C6.+, JP13.2, JP3.8, JP5.8, X4.P$2, X4.P$4; no longer S1.2, X3.P$3, X3.P$4
- net +5V: now also C4.1, JP11.4, JP12.4, JP4.5, JP4.6, JP6.5, JP6.6, JP7.3, JP8.3, LED1.VDD; no longer C2.+, L1.2, R1.2
- net GND: now also C4.2, JP1.14, JP11.1, JP12.1, JP13.3, JP2.4, JP3.1, JP3.7, JP5.1, JP5.7, JP7.1, JP8.1, LED1.VSS, U1.16, U1.21, U1.23, U1.24, U1.8, U2.GND, X4.P$1, X4.P$3; no longer C1.-, C3.2, R2.1, U$1.4, U$1.5, U$1.8, U$1.9, X3.P$1, X3.P$2
- net N$19: now also JP3.4, X1.P$4; no longer X2.P$4
- net N$2: now also U2.CH_PD; no longer L1.1, U$1.7
- net N$20: now also JP3.3, X1.P$3; no longer X2.P$3
- net N$21: now also JP5.6, X2.P$1; no longer X2.P$2
- net N$22: now also JP5.5, X2.P$2; no longer X2.P$1
- net N$23: now also JP5.4, X2.P$4; no longer X1.P$4
- net N$24: now also JP5.3, X2.P$3; no longer X1.P$3
- net N$25: now also U1.3; no longer X1.P$2
- net N$26: now also JP10.1; no longer X1.P$1

Commit message: boardf
Parts:
- added LED2, LED3: (no value), led:SML0603
- added R1: 10k, rcl:R0603
- added R2, R3: 330R, rcl:R0603
- added R4, R5, R6, R7, R8, R9: (no value), rcl:R0603
- JP1, JP2: device pinhead-2:1X15SMD -> pinhead:1X15
- JP13: device pinhead-2:1X04SMD -> pinhead:1X04
- JP3, JP4, JP5, JP6: device pinhead-2:1X08SMD -> pinhead:1X08
- moved LED1 73.1 mm to (27.3, 43.2), turned to 270 degrees
- moved C4 67.7 mm to (31.1, 43.2), turned to 270 degrees
- moved JP3 65.8 mm to (15.9, 13.3), turned to 270 degrees
- moved JP5 62.1 mm to (76.8, 13.3), turned to 90 degrees
- moved X1 42.5 mm to (29.8, 29.8)
- moved X2 36.2 mm to (65.4, 29.8)
- moved C2 29.9 mm to (17.1, 29.8), turned to 180 degrees
- moved JP9 19.7 mm to (31.1, 49.5)
- moved JP2 19.1 mm to (38.7, 22.9)
- moved JP1 14.3 mm to (54.0, 22.9)
- moved U1 9.94 mm to (80.6, 48.3)
- moved C5 9.92 mm to (80.0, 26.7), turned to 0 degrees
- moved JP6 8.47 mm to (64.1, 13.3)
- moved JP4 7.01 mm to (28.6, 13.3)
- moved JP7 6.35 mm to (39.4, 49.5)
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Connections:
- removed net 5V: JP1.12
- removed net M0L: JP6.2
- removed net M0R: JP4.2
- removed net M1L: JP6.3
- removed net M1R: JP4.3
- removed net M2L: JP6.4
- removed net M2R: JP4.4
- removed net N$1 (its old number): JP9.1
- removed net N$13 (its old number): JP7.2
- removed net N$25: U1.3
- removed net N$26: JP10.1
- removed net N$27: JP10.2
- removed net P1: JP2.10
- removed net P2: JP2.11
- removed net P3: JP2.12
- removed net PA12: JP2.5
- removed net PA2: JP1.11
- removed net PA3: JP1.6
- removed net VDDAON: U1.5
- removed net VIN: JP1.15
- new net DWMRES: JP1.11, U1.3
- new net ESPEN: JP2.10, U2.CH_PD
- new net IRQ: JP1.6, R1.2, U1.22
- new net N$11: JP6.4, R8.2
- new net N$4: JP4.2, R4.2
- new net N$5: LED2.A, R3.1
- new net N$6: LED3.A, R2.1
- new net N$8: JP4.4, R6.2
- new net N$9: JP6.2, R7.2
- new net PWM1: JP10.2, JP2.12
- new net PWM2: JP2.11, JP9.2
- net +12V: now also JP1.15
- net +3V3: now also U1.5; no longer JP9.3
- net +5V: now also JP1.12, JP9.3, R4.1, R5.1, R6.1, R7.1, R8.1, R9.1
- net CSN: now also U1.17
- net GND: now also JP10.1, JP9.1, LED2.C, LED3.C, R1.1
- net LED1: now also JP2.5
- net N$10: now also JP6.3, R9.2; no longer JP8.2
- net N$2: now also R3.2, U1.13; no longer U2.CH_PD
- net N$3: now also R2.2, U1.12; no longer JP9.2
- net N$7: now also JP4.3, R5.2; no longer U1.17
- net PB0: now also JP8.2
- net PB1: now also JP7.2
Routing:
- net GND: track 0.00 -> 389.4 mm
- net +12V: track 0.00 -> 159.2 mm
- net +5V: track 0.00 -> 154.4 mm
- net +3V3: track 0.00 -> 125.4 mm, vias 0 -> 3
- net ESPEN: track 0.00 -> 100.5 mm, vias 0 -> 1
- net IRQ: track 0.00 -> 78.9 mm
- net CSN: track 0.00 -> 78.3 mm, vias 0 -> 2
- net SCK: track 0.00 -> 64.3 mm
- net MISO: track 0.00 -> 59.6 mm
- net MOSI: track 0.00 -> 54.8 mm
- net SDA: track 0.00 -> 52.6 mm
- net SCL: track 0.00 -> 49.0 mm
- net PWM1: track 0.00 -> 46.0 mm
- net RX: track 0.00 -> 37.8 mm
- net PWM2: track 0.00 -> 37.8 mm
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- added copper zone on layer 1, net GND
- added copper zone on layer 16, net GND
Other:
- board size 93.7 x 52.1 mm -> 95.3 x 52.7 mm
- board text added: "MINI RYŚ"
