File: mainboard/mainboard.brd (EAGLE design)
At the start: 95.3 x 52.7 mm, 34 parts, among them U1 DWM1000, U2 ESP8266

Commit message: useful mods
Parts:
- added R10, R11: 10k, rcl:R0603
- turned PWM1 to 180 degrees
Connections:
- new net N$16: R11.1, U2.RESET
- new net N$21: R10.1, U2.GPIO15
- net +3V3: now also R11.2; no longer PWM1.3
- net +5V: now also PWM1.3
- net GND: now also R10.2
Routing:
- net N$16: track 0.00 -> 23.6 mm
- net +3V3: track 125.4 -> 115.3 mm, vias 3 -> 4
- net +5V: track 154.4 -> 158.6 mm
- net GND: track 389.4 -> 393.4 mm
- net N$21: track 0.00 -> 3.18 mm
Changed lines of the file:
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@@
 <element name="ADC1" library="jst_eph" package="B3B-PH-K-S" value="3PIN" x="47.625" y="49.53"/>
 <element name="PWM2" library="jst_eph" package="B3B-PH-K-S" value="3PIN" x="31.115" y="49.53"/>
-<element name="PWM1" library="jst_eph" package="B3B-PH-K-S" value="3PIN" x="22.86" y="49.53"/>
+<element name="PWM1" library="jst_eph" package="B3B-PH-K-S" value="3PIN" x="22.86" y="49.53" rot="R180"/>
 <element name="I2C1" library="jst_eph" package="B4B-PH-K-S" value="4PIN" x="67.31" y="49.53"/>
 <element name="I2C2" library="jst_eph" package="B4B-PH-K-S" value="4PIN" x="57.15" y="49.53"/>
@@
 <element name="R8" library="rcl" package="R0603" value="0R" x="60.96" y="14.605"/>
 <element name="R9" library="rcl" package="R0603" value="0R" x="60.96" y="17.145"/>
+<element name="R10" library="rcl" package="R0603" value="10k" x="20.955" y="36.83"/>
+<element name="R11" library="rcl" package="R0603" value="10k" x="11.43" y="31.75"/>
 </elements>
 <signals>
@@
 <wire x1="60.325" y1="51.435" x2="49.53" y2="51.435" width="0.8128" layer="1"/>
 <wire x1="49.53" y1="51.435" x2="41.275" y2="51.435" width="0.8128" layer="1"/>
-<wire x1="41.275" y1="51.435" x2="33.02" y2="51.435" width="0.8128" layer="1"/>
 <wire x1="60.15" y1="49.53" x2="60.15" y2="51.26" width="0.8128" layer="1"/>
 <wire x1="60.15" y1="51.26" x2="60.325" y2="51.435" width="0.8128" layer="1"/>
@@
 <wire x1="41.37" y1="49.53" x2="41.37" y2="51.34" width="0.8128" layer="1"/>
 <wire x1="41.37" y1="51.34" x2="41.275" y2="51.435" width="0.8128" layer="1"/>
-<wire x1="33.115" y1="49.53" x2="33.115" y2="51.34" width="0.8128" layer="1"/>
-<wire x1="33.115" y1="51.34" x2="33.02" y2="51.435" width="0.8128" layer="1"/>
-<wire x1="24.86" y1="49.53" x2="24.86" y2="50.895" width="0.8128" layer="1"/>
-<wire x1="24.86" y1="50.895" x2="25.4" y2="51.435" width="0.8128" layer="1"/>
-<wire x1="25.4" y1="51.435" x2="33.02" y2="51.435" width="0.8128" layer="1"/>
-<wire x1="24.86" y1="49.53" x2="24.86" y2="51.34" width="0.8128" layer="16"/>
-<wire x1="24.86" y1="51.34" x2="24.765" y2="51.435" width="0.8128" layer="16"/>
-<wire x1="24.765" y1="51.435" x2="10.795" y2="51.435" width="0.8128" layer="16"/>
-<wire x1="10.795" y1="51.435" x2="8.255" y2="48.895" width="0.8128" layer="16"/>
-<wire x1="8.255" y1="48.895" x2="8.255" y2="26.9" width="0.8128" layer="16"/>
+<wire x1="8.255" y1="49.53" x2="8.255" y2="26.9" width="0.8128" layer="16"/>
 <wire x1="8.255" y1="26.9" x2="7.85" y2="26.495" width="0.8128" layer="16"/>
 <wire x1="76.835" y1="19.685" x2="75.565" y2="19.685" width="1.27" layer="1"/>
@@
 <wire x1="18.945" y1="29.845" x2="18.945" y2="33.025" width="1.016" layer="1"/>
 <wire x1="18.945" y1="33.025" x2="16.99" y2="34.98" width="1.016" layer="1"/>
-<wire x1="24.86" y1="49.53" x2="24.86" y2="47.72" width="0.6096" layer="1"/>
-<wire x1="24.86" y1="47.72" x2="23.495" y2="46.355" width="0.6096" layer="1"/>
-<wire x1="23.495" y1="46.355" x2="23.495" y2="43.29" width="0.6096" layer="1"/>
+<wire x1="23.495" y1="46.895" x2="23.495" y2="43.29" width="0.6096" layer="1"/>
 <wire x1="23.495" y1="43.29" x2="25.605" y2="41.18" width="0.6096" layer="1"/>
 <wire x1="53.975" y1="38.1" x2="64.77" y2="38.1" width="0.8128" layer="1"/>
@@
 <vertex x="93.98" y="52.07"/>
 </polygon>
+<contactref element="R10" pad="2"/>
+<wire x1="41.275" y1="51.435" x2="35.02" y2="51.435" width="0.8128" layer="1"/>
+<wire x1="35.02" y1="51.435" x2="33.115" y2="49.53" width="0.8128" layer="1"/>
+<wire x1="23.495" y1="46.895" x2="20.86" y2="49.53" width="0.6096" layer="1"/>
+<wire x1="18.945" y1="33.025" x2="19.055" y2="33.025" width="0.6096" layer="1"/>
+<wire x1="19.055" y1="33.025" x2="21.59" y2="35.56" width="0.6096" layer="1"/>
+<wire x1="21.59" y1="35.56" x2="21.59" y2="36.615" width="0.6096" layer="1"/>
+<wire x1="21.59" y1="36.615" x2="21.805" y2="36.83" width="0.6096" layer="1"/>
+<wire x1="8.255" y1="49.53" x2="10.16" y2="51.435" width="0.8128" layer="16"/>
+<wire x1="10.16" y1="51.435" x2="20.13" y2="51.435" width="0.8128" layer="16"/>
+<wire x1="20.13" y1="51.435" x2="20.86" y2="50.705" width="0.8128" layer="16"/>
+<wire x1="20.86" y1="49.53" x2="20.86" y2="50.705" width="0.8128" layer="16"/>
+<wire x1="20.86" y1="50.705" x2="21.59" y2="51.435" width="0.8128" layer="16"/>
+<wire x1="21.59" y1="51.435" x2="31.21" y2="51.435" width="0.8128" layer="16"/>
+<wire x1="31.21" y1="51.435" x2="33.115" y2="49.53" width="0.8128" layer="16"/>
 </signal>
 <signal name="+12V">
@@
 <wire x1="51.435" y1="34.29" x2="51.435" y2="48.26" width="0.8128" layer="1"/>
 <wire x1="28.575" y1="17.145" x2="28.575" y2="14.605" width="0.4064" layer="1"/>
+<contactref element="PWM1" pad="3"/>
+<wire x1="24.86" y1="49.53" x2="29.115" y2="49.53" width="0.6096" layer="16"/>
 </signal>
 <signal name="LED1">
@@
 <signal name="ESPEN">
 <contactref element="JP2" pad="10"/>
-<contactref element="U2" pad="CH_PD"/>
 <wire x1="38.735" y1="17.78" x2="40.005" y2="17.78" width="0.4064" layer="16"/>
 <wire x1="40.005" y1="17.78" x2="41.275" y2="16.51" width="0.4064" layer="16"/>
@@
 <via x="4.445" y="45.085" extent="1-16" drill="0.6"/>
 <wire x1="4.445" y1="45.085" x2="0.695" y2="45.085" width="0.4064" layer="1"/>
-<wire x1="0.695" y1="45.085" x2="0.59" y2="44.98" width="0.4064" layer="1"/>
+<contactref element="U2" pad="CH_PD"/>
+<wire x1="0.695" y1="45.085" x2="0.59" y2="44.98" width="0" layer="19" extent="1-1"/>
 </signal>
 <signal name="N$19">
@@
 </signal>
 <signal name="+3V3">
-<contactref element="PWM1" pad="3"/>
 <contactref element="C2" pad="+"/>
 <contactref element="U2" pad="VCC"/>
@@
 <wire x1="15.345" y1="29.845" x2="15.345" y2="32.28" width="0.8128" layer="1"/>
 <wire x1="15.345" y1="32.28" x2="13.97" y2="33.655" width="0.8128" layer="1"/>
-<wire x1="13.97" y1="33.655" x2="13.97" y2="50.165" width="0.8128" layer="1"/>
-<wire x1="13.97" y1="50.165" x2="15.24" y2="51.435" width="0.8128" layer="1"/>
-<wire x1="15.24" y1="51.435" x2="18.955" y2="51.435" width="0.8128" layer="1"/>
-<wire x1="18.955" y1="51.435" x2="20.86" y2="49.53" width="0.8128" layer="1"/>
 <wire x1="74.245" y1="44.46" x2="74.245" y2="43.06" width="0.4064" layer="1"/>
 <wire x1="74.245" y1="43.06" x2="74.245" y2="41.66" width="0.4064" layer="1"/>
@@
 <wire x1="36.195" y1="44.45" x2="32.385" y2="40.64" width="0.6096" layer="1"/>
 <via x="32.385" y="40.64" extent="1-16" drill="0.6"/>
-<wire x1="32.385" y1="40.64" x2="29.75" y2="40.64" width="0.6096" layer="16"/>
-<wire x1="29.75" y1="40.64" x2="20.86" y2="49.53" width="0.6096" layer="16"/>
+<wire x1="32.385" y1="40.64" x2="29.845" y2="40.64" width="0.6096" layer="16"/>
 <via x="48.895" y="44.45" extent="1-16" drill="0.6"/>
+<wire x1="29.845" y1="40.64" x2="29.75" y2="40.64" width="0.6096" layer="16"/>
 <wire x1="48.895" y1="44.45" x2="71.12" y2="44.45" width="0.6096" layer="16"/>
 <via x="71.12" y="44.45" extent="1-16" drill="0.6"/>
 <wire x1="71.12" y1="44.45" x2="74.235" y2="44.45" width="0.6096" layer="1"/>
 <wire x1="74.235" y1="44.45" x2="74.245" y2="44.46" width="0.6096" layer="1"/>
+<contactref element="R11" pad="2"/>
+<wire x1="13.97" y1="33.655" x2="13.97" y2="33.44" width="0.6096" layer="1"/>
+<wire x1="13.97" y1="33.44" x2="12.28" y2="31.75" width="0.6096" layer="1"/>
+<wire x1="13.97" y1="33.655" x2="13.97" y2="39.37" width="0.8128" layer="1"/>
+<wire x1="13.97" y1="39.37" x2="12.7" y2="40.64" width="0.8128" layer="1"/>
+<via x="12.7" y="40.64" extent="1-16" drill="0.6"/>
+<wire x1="12.7" y1="40.64" x2="29.75" y2="40.64" width="0.6096" layer="16"/>
 </signal>
 <signal name="WIPOWER">
@@
 <contactref element="JP2" pad="12"/>
 <contactref element="PWM1" pad="2"/>
-<wire x1="22.86" y1="49.53" x2="22.86" y2="48.895" width="0.4064" layer="16"/>
-<wire x1="22.86" y1="48.895" x2="24.765" y2="46.99" width="0.4064" layer="16"/>
-<wire x1="24.765" y1="46.99" x2="28.575" y2="46.99" width="0.4064" layer="16"/>
 <wire x1="28.575" y1="46.99" x2="34.29" y2="41.275" width="0.4064" layer="16"/>
 <wire x1="34.29" y1="41.275" x2="34.29" y2="16.51" width="0.4064" layer="16"/>
 <wire x1="34.29" y1="16.51" x2="38.1" y2="12.7" width="0.4064" layer="16"/>
 <wire x1="38.1" y1="12.7" x2="38.735" y2="12.7" width="0.4064" layer="16"/>
+<wire x1="28.575" y1="46.99" x2="25.4" y2="46.99" width="0.4064" layer="16"/>
+<wire x1="25.4" y1="46.99" x2="22.86" y2="49.53" width="0.4064" layer="16"/>
 </signal>
 <signal name="PWM2">
@@
 <wire x1="66.445" y1="30.48" x2="65.405" y2="31.345" width="1.27" layer="1"/>
 </signal>
+<signal name="N$16">
+<contactref element="R11" pad="1"/>
+<contactref element="U2" pad="RESET"/>
+<wire x1="10.58" y1="31.75" x2="10.58" y2="42.76" width="0.6096" layer="1"/>
+<wire x1="10.58" y1="42.76" x2="4.445" y2="48.895" width="0.6096" layer="1"/>
+<wire x1="4.445" y1="48.895" x2="0.675" y2="48.895" width="0.6096" layer="1"/>
+<wire x1="0.675" y1="48.895" x2="0.59" y2="48.98" width="0.6096" layer="1"/>
+</signal>
+<signal name="N$21">
+<contactref element="U2" pad="GPIO15"/>
+<contactref element="R10" pad="1"/>
+<wire x1="16.99" y1="36.98" x2="19.955" y2="36.98" width="0.6096" layer="1"/>
+<wire x1="19.955" y1="36.98" x2="20.105" y2="36.83" width="0.6096" layer="1"/>
+</signal>
 </signals>
