File: mainboard/mainboard.sch (EAGLE design)
At the start: 25 parts, among them J1 BATTERY_CONNDEANS, J1Z CLONOLU, J1Z1 CLONOLU, P1 IMU, P2 analogin, P3 analogin, P4 I2C, U1 DWM1000, U2 ESP8266, X1 04-JST-B4B-XH-A, X2 04-JST-B4B-XH-A

Commit message: allsmd
Parts:
- removed J1Z, J1Z1: CLONOLU, pololu-allegro:CLONOLU
- removed U$2: ARDUINONANO, CRE-Lib1:ARDUINONANO
- removed U$3: 03-JST-B3B-XH-A, bt_con-jst-xh:03-JST-B3B-XH-A
- added JP1: Nucleo R, pinhead-2:PINHD-1X15_2.54-SMD
- added JP2: Nucleo L, pinhead-2:PINHD-1X15_2.54-SMD
- added JP3: Motor LR, pinhead-2:PINHD-1X07_2.54-SMD
- added JP4: Motor LL, pinhead-2:PINHD-1X07_2.54-SMD
- added JP5: Motor RL, pinhead-2:PINHD-1X07_2.54-SMD
- added JP6: Motor RR, pinhead-2:PINHD-1X07_2.54-SMD
Connections:
- net N$17: no longer J1ZA4983$2.VMOT
- net N$18: no longer J1Z1A4983$2.VMOT
- net N$19: no longer J1ZA4983$2.2B
- net N$20: no longer J1ZA4983$2.2A
- net N$21: no longer J1ZA4983$2.1A
- net N$22: no longer J1ZA4983$2.1B
- net N$23: no longer J1Z1A4983$2.2B
- net N$24: no longer J1Z1A4983$2.2A
- net N$25: no longer J1Z1A4983$2.1A
- net N$26: no longer J1Z1A4983$2.1B
Changed lines of the file:
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@@
 <part name="U$1" library="ST1S10PHR" deviceset="ST1S10PHR" device=""/>
 <part name="U1" library="DWM1000" deviceset="DWM1000" device=""/>
-<part name="U$2" library="CRE-Lib1" deviceset="ARDUINONANO" device=""/>
 <part name="U2" library="esp8266modules" deviceset="ESP12" device="SMD" value="ESP8266"/>
-<part name="J1Z" library="pololu-allegro" deviceset="CLONOLU" device=""/>
-<part name="J1Z1" library="pololu-allegro" deviceset="CLONOLU" device=""/>
 <part name="P1" library="jst-ph" deviceset="JST-PH4" device="" value="IMU"/>
 <part name="P2" library="jst-ph" deviceset="JST-PH4" device="" value="analogin"/>
 <part name="P3" library="jst-ph" deviceset="JST-PH4" device="" value="analogin"/>
 <part name="P4" library="jst-ph" deviceset="JST-PH4" device="" value="I2C"/>
-<part name="U$3" library="bt_con-jst-xh" deviceset="03-JST" device="-B3B-XH-A"/>
 <part name="X1" library="bt_con-jst-xh" deviceset="04-JST" device="-B4B-XH-A"/>
 <part name="X2" library="bt_con-jst-xh" deviceset="04-JST" device="-B4B-XH-A"/>
@@
 <part name="GND10" library="supply1" deviceset="GND" device=""/>
 <part name="J1" library="SparkFun-Connectors" deviceset="BATTERY_CONN" device="DEANS"/>
+<part name="JP1" library="pinhead-2" deviceset="PINHD-1X15" device="_2.54-SMD" value="Nucleo R"/>
+<part name="JP2" library="pinhead-2" deviceset="PINHD-1X15" device="_2.54-SMD" value="Nucleo L"/>
+<part name="JP3" library="pinhead-2" deviceset="PINHD-1X07" device="_2.54-SMD" value="Motor LR"/>
+<part name="JP4" library="pinhead-2" deviceset="PINHD-1X07" device="_2.54-SMD" value="Motor LL"/>
+<part name="JP5" library="pinhead-2" deviceset="PINHD-1X07" device="_2.54-SMD" value="Motor RL"/>
+<part name="JP6" library="pinhead-2" deviceset="PINHD-1X07" device="_2.54-SMD" value="Motor RR"/>
 </parts>
 <sheets>
@@
 <instance part="U$1" gate="G$1" x="218.44" y="58.42"/>
 <instance part="U1" gate="G$1" x="30.48" y="5.08"/>
-<instance part="U$2" gate="G$1" x="96.52" y="86.36"/>
 <instance part="U2" gate="G$1" x="33.02" y="86.36"/>
-<instance part="J1Z" gate="A4983$1" x="190.5" y="-5.08" rot="R270"/>
-<instance part="J1Z" gate="A4983$2" x="170.18" y="-5.08" rot="R270"/>
-<instance part="J1Z1" gate="A4983$1" x="269.24" y="-5.08" rot="R270"/>
-<instance part="J1Z1" gate="A4983$2" x="251.46" y="-5.08" rot="R270"/>
 <instance part="P1" gate="A" x="152.4" y="129.54" rot="R270"/>
 <instance part="P2" gate="A" x="172.72" y="129.54" rot="R270"/>
 <instance part="P3" gate="A" x="193.04" y="129.54" rot="R270"/>
 <instance part="P4" gate="A" x="213.36" y="129.54" rot="R270"/>
-<instance part="U$3" gate="-1" x="251.46" y="121.92"/>
-<instance part="U$3" gate="-2" x="251.46" y="119.38"/>
-<instance part="U$3" gate="-3" x="251.46" y="116.84"/>
 <instance part="X1" gate="-1" x="220.98" y="-7.62" rot="R180"/>
 <instance part="X1" gate="-2" x="220.98" y="-5.08" rot="R180"/>
@@
 <instance part="GND10" gate="1" x="236.22" y="5.08"/>
 <instance part="J1" gate="G$1" x="160.02" y="60.96"/>
+<instance part="JP1" gate="A" x="96.52" y="48.26" rot="R180"/>
+<instance part="JP2" gate="A" x="91.44" y="48.26"/>
+<instance part="JP3" gate="A" x="180.34" y="-5.08" rot="R180"/>
+<instance part="JP4" gate="A" x="175.26" y="-5.08"/>
+<instance part="JP5" gate="A" x="256.54" y="-5.08"/>
+<instance part="JP6" gate="A" x="261.62" y="-5.08" rot="R180"/>
 </instances>
 <busses>
@@
 </segment>
 </net>
-<net name="N$17" class="0">
-<segment>
-<pinref part="C5" gate="G$1" pin="+"/>
-<pinref part="J1Z" gate="A4983$2" pin="VMOT"/>
-<wire x1="152.4" y1="20.32" x2="165.1" y2="12.7" width="0.1524" layer="91"/>
-</segment>
-</net>
-<net name="N$18" class="0">
-<segment>
-<pinref part="J1Z1" gate="A4983$2" pin="VMOT"/>
-<pinref part="C6" gate="G$1" pin="+"/>
-<wire x1="246.38" y1="12.7" x2="236.22" y2="20.32" width="0.1524" layer="91"/>
-</segment>
-</net>
 <net name="N$19" class="0">
 <segment>
@@
 <wire x1="139.7" y1="0" x2="157.48" y2="0" width="0.1524" layer="91"/>
 <wire x1="157.48" y1="0" x2="157.48" y2="2.54" width="0.1524" layer="91"/>
-<pinref part="J1Z" gate="A4983$2" pin="2B"/>
 <wire x1="157.48" y1="2.54" x2="165.1" y2="2.54" width="0.1524" layer="91"/>
 </segment>
@@
 <net name="N$20" class="0">
 <segment>
-<pinref part="J1Z" gate="A4983$2" pin="2A"/>
 <pinref part="X2" gate="-3" pin="1"/>
 <wire x1="165.1" y1="-2.54" x2="139.7" y2="-2.54" width="0.1524" layer="91"/>
@@
 <wire x1="139.7" y1="-5.08" x2="157.48" y2="-5.08" width="0.1524" layer="91"/>
 <wire x1="157.48" y1="-5.08" x2="157.48" y2="-7.62" width="0.1524" layer="91"/>
-<pinref part="J1Z" gate="A4983$2" pin="1A"/>
 <wire x1="157.48" y1="-7.62" x2="165.1" y2="-7.62" width="0.1524" layer="91"/>
 </segment>
@@
 <wire x1="139.7" y1="-7.62" x2="152.4" y2="-7.62" width="0.1524" layer="91"/>
 <wire x1="152.4" y1="-7.62" x2="152.4" y2="-12.7" width="0.1524" layer="91"/>
-<pinref part="J1Z" gate="A4983$2" pin="1B"/>
 <wire x1="152.4" y1="-12.7" x2="165.1" y2="-12.7" width="0.1524" layer="91"/>
 </segment>
@@
 <wire x1="226.06" y1="0" x2="241.3" y2="0" width="0.1524" layer="91"/>
 <wire x1="241.3" y1="0" x2="241.3" y2="2.54" width="0.1524" layer="91"/>
-<pinref part="J1Z1" gate="A4983$2" pin="2B"/>
 <wire x1="241.3" y1="2.54" x2="246.38" y2="2.54" width="0.1524" layer="91"/>
 </segment>
@@
 <segment>
 <pinref part="X1" gate="-3" pin="1"/>
-<pinref part="J1Z1" gate="A4983$2" pin="2A"/>
 <wire x1="226.06" y1="-2.54" x2="246.38" y2="-2.54" width="0.1524" layer="91"/>
 </segment>
@@
 <wire x1="226.06" y1="-5.08" x2="241.3" y2="-5.08" width="0.1524" layer="91"/>
 <wire x1="241.3" y1="-5.08" x2="241.3" y2="-7.62" width="0.1524" layer="91"/>
-<pinref part="J1Z1" gate="A4983$2" pin="1A"/>
 <wire x1="241.3" y1="-7.62" x2="246.38" y2="-7.62" width="0.1524" layer="91"/>
 </segment>
@@
 <wire x1="226.06" y1="-7.62" x2="236.22" y2="-7.62" width="0.1524" layer="91"/>
 <wire x1="236.22" y1="-7.62" x2="236.22" y2="-12.7" width="0.1524" layer="91"/>
-<pinref part="J1Z1" gate="A4983$2" pin="1B"/>
 <wire x1="236.22" y1="-12.7" x2="246.38" y2="-12.7" width="0.1524" layer="91"/>
 </segment>
 </net>
+<net name="N$17" class="0">
+<segment>
+<wire x1="165.1" y1="12.7" x2="165.1" y2="20.32" width="0.1524" layer="91"/>
+<pinref part="C5" gate="G$1" pin="+"/>
+<wire x1="165.1" y1="20.32" x2="152.4" y2="20.32" width="0.1524" layer="91"/>
+</segment>
+</net>
+<net name="N$18" class="0">
+<segment>
+<wire x1="246.38" y1="12.7" x2="246.38" y2="20.32" width="0.1524" layer="91"/>
+<pinref part="C6" gate="G$1" pin="+"/>
+<wire x1="246.38" y1="20.32" x2="236.22" y2="20.32" width="0.1524" layer="91"/>
+</segment>
+</net>

Commit message: fit
Parts:
- removed J1: BATTERY_CONNDEANS, SparkFun-Connectors:BATTERY_CONNDEANS
- removed P1: IMU, jst-ph:JST-PH4
- removed P2, P3: analogin, jst-ph:JST-PH4
- removed P4: I2C, jst-ph:JST-PH4
- added X3: (no value), con-molex-micro-fit-3_0:HEADER_POS4_43045-0415
- X1, X2: value 04-JST-B4B-XH-A -> (none); device bt_con-jst-xh:04-JST-B4B-XH-A -> con-molex-micro-fit-3_0:HEADER_POS4_43045-0412
Connections:
- removed net N$1: P1.3
- removed net N$10: P3.3
- removed net N$11: P3.2
- removed net N$12: P3.1
- removed net N$13: P4.3
- removed net N$14: P4.2
- removed net N$15: P4.1
- removed net N$3: P1.2
- removed net N$6: P1.1
- removed net N$7: P2.3
- removed net N$8: P2.2
- removed net N$9: P2.1
- net +12V: now also X3.3, X3.4; no longer J1.+
- net GND: now also X3.1, X3.2; no longer P1.4, P2.4, P3.4, P4.4
- net N$19: now also X2.4; no longer X2-4.1
- net N$20: now also X2.3; no longer X2-3.1
- net N$21: now also X2.2; no longer X2-2.1
- net N$22: now also X2.1; no longer X2-1.1
- net N$23: now also X1.4; no longer X1-4.1
- net N$24: now also X1.3; no longer X1-3.1
- net N$25: now also X1.2; no longer X1-2.1
- net N$26: now also X1.1; no longer X1-1.1

Commit message: allparts
Parts:
- removed C1: (no value), rcl:CPOL-EU153CLV-0405
- removed C3: (no value), rcl:C-EUC0603K
- removed L1: (no value), rcl:L-USL4035M
- removed R1, R2: (no value), rcl:R-EU_R0603
- removed S1: (no value), switch:255SB
- removed U$1: ST1S10PHR, ST1S10PHR:ST1S10PHR
- removed X3: (no value), con-molex-micro-fit-3_0:HEADER_POS4_43045-0415
- added JP10, JP7, JP8, JP9: 3PIN, jst_eph:3PIN
- added JP11, JP12: 4PIN, jst_eph:4PIN
- added JP13: (no value), pinhead-2:PINHD-1X04_2.54-SMD
- added X4: (no value), con-molex-micro-fit-3_0:HEADER_POS4_43045-0412
- JP3: value Motor LR -> (none); device pinhead-2:PINHD-1X07_2.54-SMD -> pinhead-2:PINHD-1X08_2.54-SMD
- JP4: value Motor LL -> (none); device pinhead-2:PINHD-1X07_2.54-SMD -> pinhead-2:PINHD-1X08_2.54-SMD
- JP5: value Motor RL -> (none); device pinhead-2:PINHD-1X07_2.54-SMD -> pinhead-2:PINHD-1X08_2.54-SMD
- JP6: value Motor RR -> (none); device pinhead-2:PINHD-1X07_2.54-SMD -> pinhead-2:PINHD-1X08_2.54-SMD
Connections:
- removed net N$16: C4.1, LED1.GND
- removed net N$17: C5.+
- removed net N$18: C6.+
- removed net N$4: R1.1, R2.2, U$1.VFB
- removed net N$5: C1.+, C3.1, S1.O, U$1.EN, U$1.VIN_A, U$1.VIN_SW
- new net +3V3: C2.+, JP10.3, JP13.4, JP9.3, U1.VDD3V3@1, U1.VDD3V3@2, U2.VCC
- new net 3V3: JP1.2
- new net 5V: JP1.12
- new net AREF: JP1.3
- new net CSN: JP1.7
- new net FL: JP5.2
- new net FR: JP3.2
- new net M0L: JP6.2
- new net M0R: JP4.2
- new net M1L: JP6.3
- new net M1R: JP4.3
- new net M2L: JP6.4
- new net M2R: JP4.4
- new net MISO: JP1.9, U1.SPIMISO
- new net MLDIR: JP1.1, JP6.8
- new net MLEN: JP1.5, JP6.1
- new net MLSTEP: JP1.4, JP6.7
- new net MOSI: JP1.10, U1.SPIMOSI
- new net MRDIR: JP2.13, JP4.8
- new net MREN: JP2.15, JP4.1
- new net MRSTEP: JP2.14, JP4.7
- new net N$1: JP9.1
- new net N$10: JP8.2
- new net N$12: JP3.6, X1.1
- new net N$13: JP7.2
- new net N$15: JP3.5, X1.2
- new net N$27: JP10.2
- new net N$3: JP9.2
- new net N$7: U1.SPICSN
- new net NRST: JP1.13
- new net NRST1: JP2.3
- new net P1: JP2.10
- new net P2: JP2.11
- new net P3: JP2.12
- new net PA12: JP2.5
- new net PA2: JP1.11
- new net PA3: JP1.6
- new net PB0: JP2.6
- new net PB1: JP2.9
- new net RX: JP2.2, U2.TX
- new net SCK: JP1.8, U1.SPICLK
- new net SCL: JP11.3, JP12.3, JP2.8
- new net SDA: JP11.2, JP12.2, JP2.7
- new net TX: JP2.1, U2.RX
- new net VIN: JP1.15
- new net WIPOWER: JP13.1
- net +12V: now also C5.+, C6.+, JP13.2, JP3.8, JP5.8, X4.2, X4.4; no longer S1.P, X3.3, X3.4
- net +5V: now also C4.1, JP11.4, JP12.4, JP4.5, JP4.6, JP6.5, JP6.6, JP7.3, JP8.3, LED1.VDD; no longer C2.+, L1.2, R1.2
- net GND: now also C4.2, JP1.14, JP11.1, JP12.1, JP13.3, JP2.4, JP3.1, JP3.7, JP5.1, JP5.7, JP7.1, JP8.1, LED1.GND, U1.VSS@1, U1.VSS@2, U1.VSS@3, U1.VSS@4, U1.VSS@5, U2.GND, X4.1, X4.3; no longer C1.-, C3.2, R2.1, U$1.AGND, U$1.PAD_GND, U$1.PGND, U$1.SYNC, X3.1, X3.2
- net N$19: now also JP3.4, X1.4; no longer X2.4
- net N$2: now also U2.CH_PD; no longer L1.1, U$1.SW
- net N$20: now also JP3.3, X1.3; no longer X2.3
- net N$21: now also JP5.6, X2.1; no longer X2.2
- net N$22: now also JP5.5, X2.2; no longer X2.1
- net N$23: now also JP5.4, X2.4; no longer X1.4
- net N$24: now also JP5.3, X2.3; no longer X1.3
- net N$25: now also U1.RSTN; no longer X1.2
- net N$26: now also JP10.1; no longer X1.1
Other:
- moved on the sheet: C2, C4, C5, C6, JP1, JP2, U2, X1, X2

Commit message: boardf
Parts:
- added LED2, LED3: (no value), led:LEDSML0603
- added R1: 10k, rcl:R-EU_R0603
- added R2, R3: 330R, rcl:R-EU_R0603
- added R4, R5, R6, R7, R8, R9: (no value), rcl:R-EU_R0603
- JP1, JP2: device pinhead-2:PINHD-1X15_2.54-SMD -> pinhead:PINHD-1X15
- JP13: device pinhead-2:PINHD-1X04_2.54-SMD -> pinhead:PINHD-1X4
- JP3, JP4, JP5, JP6: device pinhead-2:PINHD-1X08_2.54-SMD -> pinhead:PINHD-1X8
Connections:
- removed net 5V: JP1.12
- removed net M0L: JP6.2
- removed net M0R: JP4.2
- removed net M1L: JP6.3
- removed net M1R: JP4.3
- removed net M2L: JP6.4
- removed net M2R: JP4.4
- removed net N$1 (its old number): JP9.1
- removed net N$13 (its old number): JP7.2
- removed net N$25: U1.RSTN
- removed net N$26: JP10.1
- removed net N$27: JP10.2
- removed net P1: JP2.10
- removed net P2: JP2.11
- removed net P3: JP2.12
- removed net PA12: JP2.5
- removed net PA2: JP1.11
- removed net PA3: JP1.6
- removed net VIN: JP1.15
- new net DWMRES: JP1.11, U1.RSTN
- new net ESPEN: JP2.10, U2.CH_PD
- new net IRQ: JP1.6, R1.2, U1.IRQ/GPIO8
- new net N$11: JP6.4, R8.2
- new net N$4: JP4.2, R4.2
- new net N$5: LED2.A, R3.1
- new net N$6: LED3.A, R2.1
- new net N$8: JP4.4, R6.2
- new net N$9: JP6.2, R7.2
- new net PWM1: JP10.2, JP2.12
- new net PWM2: JP2.11, JP9.2
- net +12V: now also JP1.15
- net +3V3: now also U1.VDDAON; no longer JP9.3
- net +5V: now also JP1.12, JP9.3, R4.1, R5.1, R6.1, R7.1, R8.1, R9.1
- net CSN: now also U1.SPICSN
- net GND: now also JP10.1, JP9.1, LED2.C, LED3.C, R1.1
- net LED1: now also JP2.5
- net N$10: now also JP6.3, R9.2; no longer JP8.2
- net N$2: now also R3.2, U1.GPIO2; no longer U2.CH_PD
- net N$3: now also R2.2, U1.GPIO3; no longer JP9.2
- net N$7: now also JP4.3, R5.2; no longer U1.SPICSN
- net PB0: now also JP8.2
- net PB1: now also JP7.2
