File: board_v2/beagleboard.brd (EAGLE design)
At the start: 69.8 x 54.6 mm, 24 parts, among them U1 DWM1000

Commit message: powerconectors
Parts:
- removed POWCON: (no value), con-molex-micro-fit-3_0:43045-0412
- added X1: 5566-2, con-molex:5566-2
Connections:
- net +12V: now also X1.2; no longer POWCON.P$2, POWCON.P$4
- net GND: now also X1.1; no longer POWCON.P$1, POWCON.P$3
Changed lines of the file:
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@@
 <element name="MOTORL" library="pinhead" package="1X08" value="" x="25.4" y="19.05" rot="R270"/>
 <element name="REGCON" library="pinhead" package="1X04" value="" x="8.89" y="44.45"/>
-<element name="POWCON" library="con-molex-micro-fit-3_0" package="43045-0412" value="" x="31.75" y="34.29"/>
 <element name="R1" library="rcl" package="R0603" value="10k" x="66.675" y="24.765"/>
 <element name="R2" library="rcl" package="R0603" value="330R" x="66.675" y="20.955"/>
@@
 <element name="R9" library="rcl" package="R0603" value="0R" x="22.225" y="22.86"/>
 <element name="U$1" library="adafruit" package="BEAGLEBONE_SHIELD" value="BEAGLEBONE_OUTLINE" x="2.54" y="55.245" rot="R270"/>
+<element name="X1" library="con-molex" package="5566-2" value="5566-2" x="-5.08" y="7.62">
+<attribute name="OC_NEWARK" value="unknown" x="-5.08" y="7.62" size="1.778" layer="27" display="off"/>
+<attribute name="MPN" value="" x="-5.08" y="7.62" size="1.778" layer="27" display="off"/>
+<attribute name="MF" value="" x="-5.08" y="7.62" size="1.778" layer="27" display="off"/>
+<attribute name="OC_FARNELL" value="1822072" x="-5.08" y="7.62" size="1.778" layer="27" display="off"/>
+</element>
 </elements>
 <signals>
@@
 <contactref element="U1" pad="24"/>
 <contactref element="REGCON" pad="3"/>
-<contactref element="POWCON" pad="P$1"/>
-<contactref element="POWCON" pad="P$3"/>
 <contactref element="R1" pad="1"/>
 <contactref element="LED3" pad="C"/>
@@
 <contactref element="U$1" pad="91"/>
 <contactref element="U$1" pad="47"/>
+<contactref element="X1" pad="1"/>
 <wire x1="58.92" y1="31.295" x2="61.215" y2="42.595" width="0" layer="19" extent="1-1"/>
 <wire x1="66.815" y1="29.795" x2="58.92" y2="31.295" width="0" layer="19" extent="1-1"/>
@@
 <wire x1="38.1" y1="10.16" x2="46.885" y2="11.43" width="0" layer="19" extent="1-1"/>
 <wire x1="38.1" y1="25.4" x2="38.1" y2="10.16" width="0" layer="19" extent="1-1"/>
-<wire x1="33.25" y1="34.29" x2="38.1" y2="25.4" width="0" layer="19" extent="1-1"/>
-<wire x1="33.25" y1="37.29" x2="33.25" y2="34.29" width="0" layer="19" extent="1-1"/>
-<wire x1="23.39" y1="33.02" x2="33.25" y2="34.29" width="0" layer="19" extent="1-1"/>
+<wire x1="23.39" y1="33.02" x2="38.1" y2="25.4" width="0" layer="19" extent="1-1"/>
 <wire x1="23.39" y1="41.275" x2="23.39" y2="33.02" width="0" layer="19" extent="1-1"/>
 <wire x1="10.16" y1="44.45" x2="23.39" y2="41.275" width="0" layer="19" extent="1-1"/>
@@
 <wire x1="5.08" y1="12.7" x2="5.08" y2="27.94" width="0" layer="19" extent="1-1"/>
 <wire x1="5.08" y1="2.54" x2="5.08" y2="12.7" width="0" layer="19" extent="1-1"/>
+<wire x1="-5.08" y1="4.87" x2="5.08" y2="2.54" width="0" layer="19" extent="1-1"/>
 </signal>
 <signal name="+12V">
@@
 <contactref element="MOTORR1" pad="8"/>
 <contactref element="REGCON" pad="2"/>
-<contactref element="POWCON" pad="P$4"/>
-<contactref element="POWCON" pad="P$2"/>
-<wire x1="30.25" y1="34.29" x2="38.1" y2="27.94" width="0" layer="19" extent="1-1"/>
-<wire x1="30.25" y1="37.29" x2="30.25" y2="34.29" width="0" layer="19" extent="1-1"/>
-<wire x1="19.79" y1="41.275" x2="30.25" y2="37.29" width="0" layer="19" extent="1-1"/>
+<contactref element="X1" pad="2"/>
+<wire x1="43.285" y1="11.43" x2="38.1" y2="27.94" width="0" layer="19" extent="1-1"/>
+<wire x1="19.79" y1="41.275" x2="38.1" y2="27.94" width="0" layer="19" extent="1-1"/>
 <wire x1="7.62" y1="44.45" x2="19.79" y2="41.275" width="0" layer="19" extent="1-1"/>
-<wire x1="43.285" y1="11.43" x2="38.1" y2="27.94" width="0" layer="19" extent="1-1"/>
-<wire x1="5.08" y1="10.16" x2="30.25" y2="34.29" width="0" layer="19" extent="1-1"/>
+<wire x1="5.08" y1="10.16" x2="7.62" y2="44.45" width="0" layer="19" extent="1-1"/>
+<wire x1="-5.08" y1="10.37" x2="5.08" y2="10.16" width="0" layer="19" extent="1-1"/>
 </signal>
 <signal name="+5V">

Commit message: beaglepinout
Connections:
- removed net N$80: U$1.78
- removed net N$81: U$1.80
- net +3V3: now also U$1.78
- net GND: now also U$1.80
Changed lines of the file:
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@@
 <contactref element="U$1" pad="47"/>
 <contactref element="X1" pad="1"/>
+<contactref element="U$1" pad="80"/>
 <wire x1="58.92" y1="31.295" x2="61.215" y2="42.595" width="0" layer="19" extent="1-1"/>
 <wire x1="66.815" y1="29.795" x2="58.92" y2="31.295" width="0" layer="19" extent="1-1"/>
@@
 <wire x1="60.96" y1="2.54" x2="60.96" y2="5.08" width="0" layer="19" extent="1-1"/>
 <wire x1="58.42" y1="2.54" x2="58.42" y2="5.08" width="0" layer="19" extent="1-1"/>
-<wire x1="46.885" y1="11.43" x2="58.42" y2="5.08" width="0" layer="19" extent="1-1"/>
+<wire x1="45.72" y1="5.08" x2="58.42" y2="5.08" width="0" layer="19" extent="1-1"/>
+<wire x1="46.885" y1="11.43" x2="45.72" y2="5.08" width="0" layer="19" extent="1-1"/>
 <wire x1="38.1" y1="10.16" x2="46.885" y2="11.43" width="0" layer="19" extent="1-1"/>
 <wire x1="38.1" y1="25.4" x2="38.1" y2="10.16" width="0" layer="19" extent="1-1"/>
@@
 <contactref element="U$1" pad="49"/>
 <contactref element="U$1" pad="50"/>
-<wire x1="19.79" y1="33.02" x2="62.615" y2="42.595" width="0" layer="19" extent="1-1"/>
+<contactref element="U$1" pad="78"/>
+<wire x1="43.18" y1="5.08" x2="62.615" y2="42.595" width="0" layer="19" extent="1-1"/>
+<wire x1="7.62" y1="5.08" x2="43.18" y2="5.08" width="0" layer="19" extent="1-1"/>
+<wire x1="7.62" y1="2.54" x2="7.62" y2="5.08" width="0" layer="19" extent="1-1"/>
+<wire x1="19.79" y1="33.02" x2="7.62" y2="5.08" width="0" layer="19" extent="1-1"/>
 <wire x1="12.7" y1="44.45" x2="19.79" y2="33.02" width="0" layer="19" extent="1-1"/>
-<wire x1="7.62" y1="5.08" x2="19.79" y2="33.02" width="0" layer="19" extent="1-1"/>
-<wire x1="7.62" y1="2.54" x2="7.62" y2="5.08" width="0" layer="19" extent="1-1"/>
 </signal>
 <signal name="WIPOWER">
@@
 <contactref element="U$1" pad="76"/>
 </signal>
-<signal name="N$80">
-<contactref element="U$1" pad="78"/>
-</signal>
-<signal name="N$81">
-<contactref element="U$1" pad="80"/>
-</signal>
 <signal name="N$82">
