File: board_v2/beagleboard.sch (EAGLE design)
At the start: 24 parts, among them U1 DWM1000

Commit message: powerconectors
Parts:
- removed POWCON: (no value), con-molex-micro-fit-3_0:HEADER_POS4_43045-0412
- added X1: 5566-2, con-molex:5566-2
Connections:
- net +12V: now also X1-2.S; no longer POWCON.2, POWCON.4
- net GND: now also X1-1.S; no longer POWCON.1, POWCON.3
Changed lines of the file:
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@@
 <part name="+3V5" library="supply1" deviceset="+3V3" device=""/>
 <part name="REGCON" library="pinhead" deviceset="PINHD-1X4" device=""/>
-<part name="POWCON" library="con-molex-micro-fit-3_0" deviceset="HEADER_POS4_?" device="43045-0412"/>
 <part name="P+1" library="supply1" deviceset="+5V" device=""/>
 <part name="P+9" library="supply1" deviceset="+5V" device=""/>
@@
 <part name="P+6" library="supply1" deviceset="+5V" device=""/>
 <part name="+3V2" library="supply1" deviceset="+3V3" device=""/>
+<part name="X1" library="con-molex" deviceset="5566-2" device=""/>
 </parts>
 <sheets>
@@
 <instance part="+3V5" gate="G$1" x="60.96" y="81.28"/>
 <instance part="REGCON" gate="A" x="7.62" y="127" rot="R90"/>
-<instance part="POWCON" gate="G$1" x="-17.78" y="104.14" rot="R180"/>
 <instance part="P+1" gate="1" x="-12.7" y="7.62"/>
 <instance part="P+9" gate="1" x="48.26" y="12.7"/>
@@
 <instance part="P+6" gate="1" x="121.92" y="58.42"/>
 <instance part="+3V2" gate="G$1" x="129.54" y="58.42"/>
+<instance part="X1" gate="-1" x="-17.78" y="101.6" rot="R180"/>
+<instance part="X1" gate="-2" x="-17.78" y="106.68" rot="R180"/>
 </instances>
 <busses>
@@
 <segment>
 <pinref part="GND11" gate="1" pin="GND"/>
-<wire x1="-10.16" y1="99.06" x2="-10.16" y2="93.98" width="0.1524" layer="91"/>
-<wire x1="-12.7" y1="99.06" x2="-10.16" y2="99.06" width="0.1524" layer="91"/>
-<pinref part="POWCON" gate="G$1" pin="1"/>
-<pinref part="POWCON" gate="G$1" pin="3"/>
-<wire x1="-12.7" y1="104.14" x2="-10.16" y2="104.14" width="0.1524" layer="91"/>
-<wire x1="-10.16" y1="104.14" x2="-10.16" y2="99.06" width="0.1524" layer="91"/>
-<junction x="-10.16" y="99.06"/>
+<wire x1="-10.16" y1="101.6" x2="-10.16" y2="93.98" width="0.1524" layer="91"/>
+<pinref part="X1" gate="-1" pin="S"/>
+<wire x1="-10.16" y1="101.6" x2="-15.24" y2="101.6" width="0.1524" layer="91"/>
 </segment>
 <segment>
@@
 <wire x1="5.08" y1="124.46" x2="5.08" y2="106.68" width="0.1524" layer="91"/>
 <wire x1="5.08" y1="106.68" x2="-2.54" y2="106.68" width="0.1524" layer="91"/>
-<pinref part="POWCON" gate="G$1" pin="4"/>
-<wire x1="-12.7" y1="106.68" x2="-2.54" y2="106.68" width="0.1524" layer="91"/>
+<wire x1="-15.24" y1="106.68" x2="-2.54" y2="106.68" width="0.1524" layer="91"/>
 <junction x="-2.54" y="106.68"/>
-<pinref part="POWCON" gate="G$1" pin="2"/>
-<wire x1="-12.7" y1="101.6" x2="-2.54" y2="101.6" width="0.1524" layer="91"/>
-<wire x1="-2.54" y1="101.6" x2="-2.54" y2="106.68" width="0.1524" layer="91"/>
-</segment>
-<segment>
+<pinref part="X1" gate="-2" pin="S"/>
+</segment>
+<segment>

Commit message: beaglepinout
Connections:
- removed net N$80: U$1.VDD_ADC
- removed net N$81: U$1.GNDA_ADC
- net +3V3: now also U$1.VDD_ADC
- net GND: now also U$1.GNDA_ADC
- net N$100: now also U$1.GPIO_117; no longer U$1.GPIO3_21
- net N$101: now also U$1.GPIO_115; no longer U$1.GPIO3_19
- net N$108: now also U$1.GPIO_20; no longer U$1.CLKOUT2
- net N$18: now also U$1.GPIO_39; no longer U$1.GPIO1_7
- net N$21: now also U$1.GPIO_35; no longer U$1.GPIO1_3
- net N$24: now also U$1.GPIO_44; no longer U$1.GPIO1_12
- net N$25: now also U$1.GPIO_26; no longer U$1.GPIO0_26
- net N$26: now also U$1.GPIO_46; no longer U$1.GPIO1_14
- net N$27: now also U$1.GPIO_65; no longer U$1.GPIO2_1
- net N$28: now also U$1.GPIO_63; no longer U$1.GPIO1_31
- net N$29: now also U$1.GPIO_37; no longer U$1.GPIO1_5
- net N$30: now also U$1.GPIO_33; no longer U$1.GPIO1_1
- net N$31: now also U$1.GPIO_61; no longer U$1.GPIO1_29
- net N$32: now also U$1.GPIO_88; no longer U$1.GPIO2_24
- net N$33: now also U$1.GPIO_89; no longer U$1.GPIO2_25
- net N$34: now also U$1.GPIO_11; no longer U$1.UART5_RTSN
- net N$35: now also U$1.PWM1B; no longer U$1.UART3_RTSN
- net N$36: now also U$1.PWM1A; no longer U$1.UART3_CTSN
- net N$37: now also U$1.GPIO_79; no longer U$1.UART5_RXD
- net N$38: now also U$1.GPIO_77; no longer U$1.GPIO2_13
- net N$39: now also U$1.GPIO_75; no longer U$1.GPIO2_11
- net N$40: now also U$1.GPIO_73; no longer U$1.GPIO2_9
- net N$41: now also U$1.PWM2B; no longer U$1.GPIO2_7
- net N$43: now also U$1.GPIO_38; no longer U$1.GPIO1_6
- net N$44: now also U$1.GPIO_34; no longer U$1.GPIO1_2
- net N$47: now also U$1.GPIO_45; no longer U$1.GPIO1_13
- net N$48: now also U$1.GPIO_23; no longer U$1.EHRPWM2B
- net N$49: now also U$1.GPIO_47; no longer U$1.GPIO1_15
- net N$50: now also U$1.GPIO_27; no longer U$1.GPIO0_27
- net N$51: now also U$1.GPIO_22; no longer U$1.EHRPWM2A
- net N$52: now also U$1.GPIO_62; no longer U$1.GPIO1_30
- net N$53: now also U$1.GPIO_36; no longer U$1.GPIO1_4
- net N$54: now also U$1.GPIO_32; no longer U$1.GPIO1_0
- net N$55: now also U$1.GPIO_86; no longer U$1.GPIO2_22
- net N$56: now also U$1.GPIO_87; no longer U$1.GPIO2_23
- net N$57: now also U$1.GPIO_10; no longer U$1.UART5_CTSN
- net N$58: now also U$1.GPIO_9; no longer U$1.UART4_RTSN
- net N$59: now also U$1.GPIO_8; no longer U$1.UART4_CTSN
- net N$60: now also U$1.GPIO_78; no longer U$1.UART5_TXD
- net N$61: now also U$1.GPIO_76; no longer U$1.GPIO2_12
- net N$62: now also U$1.GPIO_74; no longer U$1.GPIO2_10
- net N$63: now also U$1.GPIO_72; no longer U$1.GPIO2_8
- net N$64: now also U$1.PWM2A; no longer U$1.GPIO2_6
- net N$70: now also U$1.GPIO_60; no longer U$1.GPIO1_28
- net N$71: now also U$1.GPIO_50; no longer U$1.EHRPWM1A
- net N$72: now also U$1.GPIO_51; no longer U$1.EHRPWM1B
- net N$85: now also U$1.GPIO_7; no longer U$1.GPIO0_7
- net N$93: now also U$1.GPIO_30; no longer U$1.UART4_RXD
- net N$94: now also U$1.GPIO_31; no longer U$1.UART4_TXD
- net N$95: now also U$1.GPIO_48; no longer U$1.GPIO1_16
- net N$99: now also U$1.GPIO_49; no longer U$1.GPIO1_17
