File: board_v3/beagleboard.sch (EAGLE design)
At the start: 38 parts, among them U1 DWM1000, X1 5566-2, X2 04-JST-B4B-XH-A, X3 53398-05, X4 53398-05, X5 53398-05, X6 53398-05, X7 53398-05

Commit message: sd
Parts:
- removed SJ1, SJ2, SJ4, SJ5: (no value), jumper:SJ
- removed X3, X4, X5, X6, X7: 53398-05, con-molex:53398-05
- R7: value 1,5k -> 4,5k
- R8: value 1,5k -> 3k
Connections:
- net D1ECHO renamed N$42
- net D2ECHO renamed N$38
- net D3ECHO renamed N$43
- net TRIG renamed N$37
- net +5V: no longer SJ1.2, SJ2.2, SJ4.2, SJ5.2
- net LM0: no longer SJ1.1
- net LM1: no longer SJ2.1
- net RM0: no longer SJ4.1
- net RM1: no longer SJ5.1

Commit message: sds
Parts:
- removed SJ3, SJ6: (no value), jumper:SJ
- added JP1, JP2, JP3, JP4, JP5: 5PIN, jst_eph:5PIN
Connections:
- removed net LM0: MOTORL.2, U$1.GPIO_77
- removed net LM1: MOTORL.3, U$1.GPIO_76
- removed net MLEN: MOTORL.1, R17.1, U$1.GPIO_79
- removed net MREN: MOTOTR.1, R16.1, U$1.GPIO_78
- removed net N$38: U$1.TIMER5
- removed net N$42: U$1.TIMER7
- removed net N$43: U$1.TIMER6
- removed net N$52: MOTORL.4, SJ3.1
- removed net N$66: MOTOTR.4, SJ6.1
- removed net N$68: U$1.I2C1_SDA
- removed net N$79: U$1.I2C1_SCL
- removed net RM0: MOTOTR.2, U$1.PWM2A
- removed net RM1: MOTOTR.3, U$1.PWM2B
- new net I2C1_SCL: JP1.4, JP2.4, JP3.4, JP4.4, JP5.4, U$1.I2C1_SCL
- new net I2C1_SDA: JP1.3, JP2.3, JP3.3, JP4.3, JP5.3, U$1.I2C1_SDA
- new net M0: MOTORL.2, MOTOTR.2, U$1.PWM2B
- new net M1: MOTORL.3, MOTOTR.3, U$1.PWM2A
- new net M2: MOTORL.4, MOTOTR.4, U$1.GPIO_77
- new net MEN: MOTORL.1, MOTOTR.1, R16.1, R17.1, U$1.GPIO_76
- new net TOF1: JP1.5, U$1.TIMER4
- new net TOF2: JP2.5, U$1.TIMER7
- new net TOF3: JP3.5, U$1.TIMER5
- new net TOF4: JP4.5, U$1.TIMER6
- new net TOF5: JP5.5, U$1.GPIO_45
- net +3V3: now also JP1.1, JP2.1, JP3.1, JP4.1, JP5.1
- net +5V: no longer SJ3.2, SJ6.2
- net GND: now also JP1.2, JP2.2, JP3.2, JP4.2, JP5.2
- net N$23: now also U$1.GPIO_78; no longer U$1.GPIO_45
- net N$37: now also U$1.GPIO_79; no longer U$1.TIMER4
Other:
- moved on the sheet: C2, SV1

Commit message: sdsd
Other:
- moved on the sheet: R5, R6, R7, R8
Changed lines of the file:
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@@
 <instance part="GND13" gate="1" x="101.6" y="43.18"/>
 <instance part="R4" gate="G$1" x="96.52" y="50.8" rot="R90"/>
-<instance part="R5" gate="G$1" x="91.44" y="50.8" rot="R90"/>
-<instance part="R6" gate="G$1" x="86.36" y="50.8" rot="R90"/>
-<instance part="R7" gate="G$1" x="86.36" y="68.58" rot="R90"/>
-<instance part="R8" gate="G$1" x="91.44" y="66.04" rot="R90"/>
+<instance part="R5" gate="G$1" x="88.9" y="50.8" rot="R90"/>
+<instance part="R6" gate="G$1" x="81.28" y="50.8" rot="R90"/>
+<instance part="R7" gate="G$1" x="81.28" y="68.58" rot="R90"/>
+<instance part="R8" gate="G$1" x="88.9" y="66.04" rot="R90"/>
 <instance part="R9" gate="G$1" x="96.52" y="63.5" rot="R90"/>
 <instance part="P+8" gate="1" x="0" y="121.92"/>
@@
 <junction x="101.6" y="45.72"/>
 <pinref part="R5" gate="G$1" pin="1"/>
-<wire x1="96.52" y1="45.72" x2="91.44" y2="45.72" width="0.1524" layer="91"/>
+<wire x1="96.52" y1="45.72" x2="88.9" y2="45.72" width="0.1524" layer="91"/>
 <junction x="96.52" y="45.72"/>
 <pinref part="R6" gate="G$1" pin="1"/>
-<wire x1="91.44" y1="45.72" x2="86.36" y2="45.72" width="0.1524" layer="91"/>
-<junction x="91.44" y="45.72"/>
+<wire x1="88.9" y1="45.72" x2="81.28" y2="45.72" width="0.1524" layer="91"/>
+<junction x="88.9" y="45.72"/>
 </segment>
 <segment>
@@
 <net name="CELL2" class="0">
 <segment>
-<wire x1="91.44" y1="60.96" x2="91.44" y2="55.88" width="0.1524" layer="91"/>
+<wire x1="88.9" y1="60.96" x2="88.9" y2="55.88" width="0.1524" layer="91"/>
 <pinref part="R5" gate="G$1" pin="2"/>
-<label x="91.44" y="60.96" size="1.27" layer="95" rot="R180" xref="yes"/>
+<label x="88.9" y="60.96" size="1.27" layer="95" rot="R180" xref="yes"/>
 <pinref part="R8" gate="G$1" pin="1"/>
 </segment>
@@
 <net name="CELL3" class="0">
 <segment>
-<wire x1="86.36" y1="63.5" x2="86.36" y2="55.88" width="0.1524" layer="91"/>
+<wire x1="81.28" y1="63.5" x2="81.28" y2="55.88" width="0.1524" layer="91"/>
 <pinref part="R6" gate="G$1" pin="2"/>
-<label x="86.36" y="63.5" size="1.27" layer="95" rot="R180" xref="yes"/>
+<label x="81.28" y="63.5" size="1.27" layer="95" rot="R180" xref="yes"/>
 <pinref part="R7" gate="G$1" pin="1"/>
 </segment>
@@
 <pinref part="R7" gate="G$1" pin="2"/>
 <pinref part="X2" gate="-1" pin="1"/>
-<wire x1="86.36" y1="73.66" x2="109.22" y2="73.66" width="0.1524" layer="91"/>
+<wire x1="81.28" y1="73.66" x2="109.22" y2="73.66" width="0.1524" layer="91"/>
 </segment>
 </net>
@@
 <pinref part="R8" gate="G$1" pin="2"/>
 <pinref part="X2" gate="-2" pin="1"/>
-<wire x1="91.44" y1="71.12" x2="109.22" y2="71.12" width="0.1524" layer="91"/>
-</segment>
-</net>
+<wire x1="88.9" y1="71.12" x2="109.22" y2="71.12" width="0.1524" layer="91"/>
+</segment>
+</net>

Commit message: v3-ready
Parts:
- X1: value 5566-2 -> (none); device con-molex:5566-2 -> con-molex-micro-fit-3_0:HEADER_POS2_43045-0212
Connections:
- removed net N$61: U$1.VDD_3V3EXP@2
- new net ENABLE: SV1.1
- net +12V: now also SV1.2, X1.2; no longer SV1.3, X1-2.S
- net +3V3: now also U$1.VDD_3V3EXP@2
- net GND: now also X1.1; no longer X1-1.S
- net M0: now also U$1.GPIO_74; no longer U$1.PWM2B
- net M1: now also U$1.GPIO_73; no longer U$1.PWM2A
- net M2: now also U$1.GPIO_72; no longer U$1.GPIO_77
- net MEN: now also U$1.GPIO_75; no longer U$1.GPIO_76
- net MLDIR: now also U$1.GPIO_76; no longer U$1.GPIO_74
- net MLSTEP: now also U$1.GPIO_77; no longer U$1.GPIO_75
- net MRDIR: now also U$1.PWM2A; no longer U$1.GPIO_73
- net MRSTEP: now also U$1.PWM2B; no longer U$1.GPIO_72
- net N$1: now also MCONL.4; no longer MCONL.3
- net N$10: now also MCONL.2; no longer MCONL.1
- net N$11: now also MCONL.3; no longer MCONL.4
- net N$12: now also MCONR.1; no longer MCONR.2
- net N$13: now also MCONR.2, MOTORR1.5; no longer MCONR.3, MOTORR1.4
- net N$14: now also MOTORR1.4; no longer MOTORR1.3
- net N$15: now also MCONR.3, MOTORR1.3; no longer MCONR.1, MOTORR1.5
- net N$9: now also MCONL.1; no longer MCONL.2

Commit message: ojojoj
Parts:
- removed C2: 33u, rcl:CPOL-EU153CLV-0405
- removed X2: 04-JST-B4B-XH-A, bt_con-jst-xh:04-JST-B4B-XH-A
- added JP6: 3PIN, jst_eph:3PIN
- R4, R5, R6, R7, R8, R9: device rcl:R-EU_R0805 -> rcl:R-EU_R0603
- X1: device con-molex-micro-fit-3_0:HEADER_POS2_43045-0212 -> con-molex-micro-fit-3_0:HEADER_POS4_43045-0412
Connections:
- removed net N$4: R7.2, X2-1.1
- removed net N$67: U$1.AIN6
- removed net N$7: R8.2, X2-2.1
- removed net N$8: R9.2, X2-3.1
- new net 3V5: R9.2, X1.2
- new net 7V: R8.2, X1.3
- new net TEMPSENS: JP6.2, U$1.AIN5
- net +12V: now also R7.2, X1.4; no longer X1.2
- net +5V: now also JP6.1; no longer C2.+
- net CELL1: now also U$1.AIN6; no longer U$1.AIN5
- net GND: now also JP6.3; no longer C2.-, X2-4.1
Other:
- moved on the sheet: SV1
