File: board_v3/beagleboard.brd (EAGLE design)
At the start: 69.8 x 54.6 mm, 38 parts, among them U1 DWM1000, X1 5566-2, X2 04-JST-B4B-XH-A, X3 53398-05, X4 53398-05, X5 53398-05, X6 53398-05, X7 53398-05

Commit message: sd
Parts:
- removed SJ1, SJ2, SJ4, SJ5: (no value), jumper:SJ
- removed X3, X4, X5, X6, X7: 53398-05, con-molex:53398-05
- R7: value 1,5k -> 4,5k
- R8: value 1,5k -> 3k
- moved C5 23.0 mm to (11.1, 13.0)
- moved R16 22.5 mm to (48.6, 16.2), turned to 270 degrees
- moved SJ6 18.5 mm to (44.8, 28.9), turned to 90 degrees
- moved MOTOTR 17.8 mm to (47.9, 28.9)
- moved C6 15.5 mm to (29.2, 11.1)
- moved C2 14.8 mm to (35.2, 11.1)
- moved SV1 7.62 mm to (54.6, 46.0)
- moved MOTORL 7.62 mm to (27.0, 28.9)
- moved MCONL 7.62 mm to (21.9, 12.4)
- moved MOTORL1 7.62 mm to (14.3, 28.9)
- moved MOTORR1 7.62 mm to (35.2, 28.9)
- moved R17 7.62 mm to (24.1, 37.1)
- moved MCONR 5.08 mm to (43.5, 12.4)
- moved SJ3 1.42 mm to (23.8, 28.9), turned to 270 degrees
Connections:
- net D1ECHO renamed N$42
- net D2ECHO renamed N$38
- net D3ECHO renamed N$43
- net TRIG renamed N$37
- net +5V: no longer SJ1.2, SJ2.2, SJ4.2, SJ5.2
- net LM0: no longer SJ1.1
- net LM1: no longer SJ2.1
- net RM0: no longer SJ4.1
- net RM1: no longer SJ5.1
Routing:
- net GND: track 276.7 -> 79.5 mm
- net +5V: track 144.0 -> 2.54 mm, vias 1 -> 0
- net +12V: track 101.6 -> 0.00 mm
- net MLSTEP: track 58.6 -> 0.00 mm
- net MLDIR: track 58.4 -> 0.00 mm
- net RM1: track 53.0 -> 0.00 mm
- net RM0: track 53.0 -> 0.00 mm
- net LM1: track 48.6 -> 0.00 mm
- net LM0: track 47.3 -> 0.00 mm
- net MREN: track 47.0 -> 0.00 mm
- net CELL1: track 47.0 -> 2.86 mm, vias 1 -> 0
- net MLEN: track 43.1 -> 0.00 mm
- net MRDIR: track 38.0 -> 0.00 mm
- net MRSTEP: track 37.7 -> 0.00 mm
- net N$14: track 29.6 -> 0.00 mm
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
Commit message: sds
Parts:
- removed SJ3, SJ6: (no value), jumper:SJ
- added JP1, JP2, JP3, JP4, JP5: 5PIN, jst_eph:B5B-PH-K-S
- moved C5 2.54 mm to (11.1, 10.5)
Connections:
- removed net LM0: MOTORL.2, U$1.40
- removed net LM1: MOTORL.3, U$1.39
- removed net MLEN: MOTORL.1, R17.1, U$1.38
- removed net MREN: MOTOTR.1, R16.1, U$1.37
- removed net N$38: U$1.9
- removed net N$42: U$1.8
- removed net N$43: U$1.10
- removed net N$52: MOTORL.4, SJ3.1
- removed net N$66: MOTOTR.4, SJ6.1
- removed net N$68: U$1.64
- removed net N$79: U$1.63
- removed net RM0: MOTOTR.2, U$1.45
- removed net RM1: MOTOTR.3, U$1.46
- new net I2C1_SCL: JP1.4, JP2.4, JP3.4, JP4.4, JP5.4, U$1.63
- new net I2C1_SDA: JP1.3, JP2.3, JP3.3, JP4.3, JP5.3, U$1.64
- new net M0: MOTORL.2, MOTOTR.2, U$1.46
- new net M1: MOTORL.3, MOTOTR.3, U$1.45
- new net M2: MOTORL.4, MOTOTR.4, U$1.40
- new net MEN: MOTORL.1, MOTOTR.1, R16.1, R17.1, U$1.39
- new net TOF1: JP1.5, U$1.7
- new net TOF2: JP2.5, U$1.8
- new net TOF3: JP3.5, U$1.9
- new net TOF4: JP4.5, U$1.10
- new net TOF5: JP5.5, U$1.11
- net +3V3: now also JP1.1, JP2.1, JP3.1, JP4.1, JP5.1
- net +5V: no longer SJ3.2, SJ6.2
- net GND: now also JP1.2, JP2.2, JP3.2, JP4.2, JP5.2
- net N$23: now also U$1.37; no longer U$1.11
- net N$37: now also U$1.38; no longer U$1.7

Commit message: sdsd
Parts:
- moved MOTORR1 13.4 mm to (48.6, 29.5), turned to 90 degrees
- moved MOTORL 12.7 mm to (14.3, 29.5)
- moved MOTORL1 12.7 mm to (27.0, 29.5)
- moved MOTOTR 12.1 mm to (35.9, 29.5), turned to 270 degrees
- moved MCONL 0.63 mm to (21.9, 13.0)
- moved MCONR 0.63 mm to (43.5, 13.0)

Commit message: v3-ready
Parts:
- X1: value 5566-2 -> (none); device con-molex:5566-2 -> con-molex-micro-fit-3_0:43045-0212
- moved C2 27.6 mm to (7.62, 11.1), turned to 0 degrees
- moved R16 24.3 mm to (32.7, 34.6)
- moved C5 23.5 mm to (34.6, 12.1)
- moved R17 13.0 mm to (11.1, 36.8)
- moved SV1 9.23 mm to (58.7, 37.8)
- moved MCONL 2.62 mm to (19.4, 13.7), turned to 270 degrees
- moved MCONR 2.62 mm to (41.0, 13.7), turned to 270 degrees
- moved X1 2.29 mm to (64.8, 45.7), turned to 270 degrees
- moved JP4 2.22 mm to (22.5, 45.7)
- moved JP5 1.91 mm to (36.2, 45.7)
- moved JP3 1.90 mm to (9.53, 45.7)
- moved JP1 1.80 mm to (6.35, 22.2)
- moved JP2 1.42 mm to (6.35, 35.6)
- moved C6 0.95 mm to (29.2, 12.1)
- moved MOTORL 0.64 mm to (14.3, 28.9)
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Connections:
- removed net N$61: U$1.50
- new net ENABLE: SV1.1
- net +12V: now also SV1.2, X1.P$2; no longer SV1.3, X1.2
- net +3V3: now also U$1.50
- net GND: now also X1.P$1; no longer X1.1
- net M0: now also U$1.41; no longer U$1.46
- net M1: now also U$1.44; no longer U$1.45
- net M2: now also U$1.43; no longer U$1.40
- net MEN: now also U$1.42; no longer U$1.39
- net MLDIR: now also U$1.39; no longer U$1.41
- net MLSTEP: now also U$1.40; no longer U$1.42
- net MRDIR: now also U$1.45; no longer U$1.44
- net MRSTEP: now also U$1.46; no longer U$1.43
- net N$1: now also MCONL.P$4; no longer MCONL.P$3
- net N$10: now also MCONL.P$2; no longer MCONL.P$1
- net N$11: now also MCONL.P$3; no longer MCONL.P$4
- net N$12: now also MCONR.P$1; no longer MCONR.P$2
- net N$13: now also MCONR.P$2, MOTORR1.5; no longer MCONR.P$3, MOTORR1.4
- net N$14: now also MOTORR1.4; no longer MOTORR1.3
- net N$15: now also MCONR.P$3, MOTORR1.3; no longer MCONR.P$1, MOTORR1.5
- net N$9: now also MCONL.P$1; no longer MCONL.P$2
Routing:
- net GND: track 79.5 -> 370.8 mm, vias 0 -> 2
- net +3V3: track 2.80 -> 163.9 mm, vias 0 -> 4
- net +5V: track 2.54 -> 154.3 mm, vias 0 -> 1
- net I2C1_SCL: track 0.00 -> 87.7 mm
- net +12V: track 0.00 -> 86.7 mm
- net I2C1_SDA: track 0.00 -> 83.7 mm
- net MLSTEP: track 0.00 -> 64.1 mm, vias 0 -> 1
- net MLDIR: track 0.00 -> 63.8 mm, vias 0 -> 1
- net MEN: track 0.00 -> 58.8 mm
- net M1: track 0.00 -> 55.8 mm
- net M2: track 0.00 -> 54.9 mm
- net M0: track 0.00 -> 50.6 mm
- net MRSTEP: track 0.00 -> 46.2 mm
- net CELL1: track 2.86 -> 48.5 mm, vias 0 -> 1
- net MRDIR: track 0.00 -> 45.5 mm
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Other:
- board text added: "BIONIK"

Commit message: ojojoj
Parts:
- removed C2: 33u, rcl:153CLV-0405
- removed X2: 04-JST-B4B-XH-A, bt_con-jst-xh:B4B-XH
- added JP6: 3PIN, jst_eph:B3B-PH-K-S
- R4, R5, R6, R7, R8, R9: device rcl:R0805 -> rcl:R0603
- X1: device con-molex-micro-fit-3_0:43045-0212 -> con-molex-micro-fit-3_0:43045-0412
- moved R5 9.71 mm to (69.5, 33.7), turned to 90 degrees
- moved R6 8.54 mm to (64.5, 33.7), turned to 90 degrees
- moved R7 7.63 mm to (64.5, 37.5), turned to 90 degrees
- moved R4 7.62 mm to (67.6, 33.7), turned to 90 degrees
- moved R8 7.44 mm to (69.5, 37.5), turned to 90 degrees
- moved R9 4.76 mm to (67.6, 37.5), turned to 90 degrees
- moved X1 3.24 mm to (65.4, 42.5), turned to 0 degrees
- moved SV1 3.14 mm to (56.5, 35.6), turned to 270 degrees
- moved U1 2.01 mm to (67.3, 20.3)
- moved JP1 0.63 mm to (6.35, 22.9)
Connections:
- removed net N$4: R7.2, X2.P$1
- removed net N$67: U$1.81
- removed net N$7: R8.2, X2.P$2
- removed net N$8: R9.2, X2.P$3
- new net 3V5: R9.2, X1.P$2
- new net 7V: R8.2, X1.P$3
- new net TEMPSENS: JP6.2, U$1.82
- net +12V: now also R7.2, X1.P$4; no longer X1.P$2
- net +5V: now also JP6.1; no longer C2.+
- net CELL1: now also U$1.81; no longer U$1.82
- net GND: now also JP6.3; no longer C2.-, X2.P$4
Routing:
- net GND: track 370.8 -> 274.0 mm, vias 2 -> 1
- net +3V3: track 163.9 -> 108.8 mm, vias 4 -> 2
- net CELL1: track 48.5 -> 0.00 mm, vias 1 -> 0
- net TEMPSENS: track 0.00 -> 46.0 mm, vias 0 -> 1
- net CELL2: track 35.2 -> 0.00 mm, vias 1 -> 0
- net CELL3: track 31.7 -> 0.00 mm, vias 1 -> 0
- net +12V: track 86.7 -> 56.1 mm
- net DWMRES: track 45.0 -> 26.6 mm, vias 2 -> 1
- net +5V: track 154.3 -> 141.9 mm
- net N$3: track 20.4 -> 8.46 mm
- net IRQ: track 29.6 -> 19.8 mm
- net N$2: track 17.0 -> 7.30 mm
- net CSN: track 26.7 -> 33.2 mm
- net N$8: track 5.18 -> 0.00 mm
- net N$7: track 4.92 -> 0.00 mm
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
Commit message: report
Parts:
- moved R6 6.68 mm to (71.1, 34.0)
- moved R7 6.68 mm to (71.1, 37.1)
- moved R9 3.82 mm to (63.8, 37.1)
- moved R4 3.82 mm to (63.8, 34.0)
- moved R8 1.62 mm to (67.9, 37.1)
- moved R5 1.62 mm to (67.9, 34.0)
Routing:
- net GND: track 274.0 -> 356.4 mm
- net CELL1: track 0.00 -> 42.5 mm, vias 0 -> 1
- net CELL3: track 0.00 -> 41.7 mm, vias 0 -> 1
- net CELL2: track 0.00 -> 40.3 mm, vias 0 -> 1
- net +3V3: track 108.8 -> 148.4 mm
- net +12V: track 56.1 -> 95.5 mm
- net DWMRES: track 26.6 -> 43.9 mm, vias 1 -> 2
- net N$3: track 8.46 -> 22.2 mm
- net N$2: track 7.30 -> 18.5 mm
- net 7V: track 0.00 -> 9.29 mm
- net IRQ: track 19.8 -> 28.3 mm
- net 3V5: track 0.00 -> 4.58 mm
- net +5V: track 141.9 -> 140.0 mm, vias 1 -> 0
- net MOSI: track 24.1 -> 25.7 mm
- net SCK: track 26.9 -> 28.2 mm
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Other:
- board text added: "iRYS 3"
- board text removed: "iRYS v2.2"

Commit message: gerbery
Parts:
- moved R17 2.22 mm to (11.1, 34.6)
Routing:
- net +5V: track 140.0 -> 137.8 mm
- net MEN: track 58.8 -> 60.0 mm
- net +12V: track 95.5 -> 94.4 mm
Changed lines of the file:
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@@
 <?xml version="1.0" encoding="utf-8"?>
 <!DOCTYPE eagle SYSTEM "eagle.dtd">
-<eagle version="8.1.1">
+<eagle version="7.7.0">
 <drawing>
 <settings>
@@
 </element>
 <element name="R16" library="rcl" package="R0805" value="10k" x="32.7025" y="34.6075" rot="R270"/>
-<element name="R17" library="rcl" package="R0805" value="10k" x="11.1125" y="36.83" rot="R270"/>
+<element name="R17" library="rcl" package="R0805" value="10k" x="11.1125" y="34.6075" rot="R270"/>
 <element name="JP1" library="jst_eph" package="B5B-PH-K-S" value="5PIN" x="6.35" y="22.86" rot="R90"/>
 <element name="JP2" library="jst_eph" package="B5B-PH-K-S" value="5PIN" x="6.35" y="35.56" rot="R90"/>
@@
 <contactref element="X1" pad="P$4"/>
 <wire x1="71.12" y1="37.9975" x2="71.12" y2="45.4025" width="0.3048" layer="1"/>
-<wire x1="71.12" y1="45.4025" x2="67.31" y2="49.2125" width="0.3048" layer="1"/>
-<wire x1="67.31" y1="49.2125" x2="66.3575" y2="49.2125" width="0.3048" layer="1"/>
-<wire x1="66.3575" y1="49.2125" x2="64.135" y2="46.99" width="0.3048" layer="1"/>
+<wire x1="71.12" y1="45.4025" x2="68.58" y2="47.9425" width="0.3048" layer="1"/>
+<wire x1="68.58" y1="47.9425" x2="65.0875" y2="47.9425" width="0.3048" layer="1"/>
+<wire x1="65.0875" y1="47.9425" x2="64.135" y2="46.99" width="0.3048" layer="1"/>
 <wire x1="64.135" y1="46.99" x2="64.135" y2="45.775" width="0.3048" layer="1"/>
 <wire x1="64.135" y1="45.775" x2="63.905" y2="45.545" width="0.3048" layer="1"/>
@@
 <wire x1="11.43" y1="6.35" x2="10.16" y2="5.08" width="0.6096" layer="16"/>
 <wire x1="35.8775" y1="25.0825" x2="35.8775" y2="27.6225" width="0.6096" layer="16"/>
-<wire x1="11.1125" y1="35.88" x2="11.1125" y2="30.7975" width="0.3048" layer="1"/>
 <wire x1="11.1125" y1="30.7975" x2="14.2875" y2="27.6225" width="0.3048" layer="1"/>
 <wire x1="32.7025" y1="33.6575" x2="32.7025" y2="30.7975" width="0.3048" layer="1"/>
@@
 <wire x1="57.785" y1="29.21" x2="56.515" y2="30.48" width="0.6096" layer="16"/>
 <wire x1="32.385" y1="10.16" x2="46.0375" y2="10.16" width="0.6096" layer="16"/>
+<wire x1="11.1125" y1="30.7975" x2="11.1125" y2="33.6575" width="0.3048" layer="1"/>
 </signal>
 <signal name="CSN">
@@
 <contactref element="MOTORL" pad="7"/>
 <contactref element="U$1" pad="40"/>
-<wire x1="53.34" y1="53.34" x2="53.34" y2="53.0225" width="0.3048" layer="16"/>
-<wire x1="53.34" y1="53.0225" x2="52.07" y2="51.7525" width="0.3048" layer="16"/>
-<wire x1="52.07" y1="51.7525" x2="52.07" y2="46.99" width="0.3048" layer="16"/>
+<wire x1="53.34" y1="53.34" x2="52.07" y2="52.07" width="0.3048" layer="16"/>
+<wire x1="52.07" y1="52.07" x2="52.07" y2="46.99" width="0.3048" layer="16"/>
 <wire x1="52.07" y1="46.99" x2="48.5775" y2="43.4975" width="0.3048" layer="16"/>
 <wire x1="48.5775" y1="43.4975" x2="44.7675" y2="43.4975" width="0.3048" layer="16"/>
@@
 <contactref element="U$1" pad="81"/>
 <wire x1="48.26" y1="2.54" x2="49.53" y2="3.81" width="0.3048" layer="16"/>
-<wire x1="54.630071875" y1="19.238065625" x2="57.973065625" y2="22.413065625" width="0.3048" layer="16"/>
-<wire x1="57.973065625" y1="22.413065625" x2="62.5475" y2="26.9875" width="0.3048" layer="16"/>
-<wire x1="49.53" y1="14.45549375" x2="54.630071875" y2="19.238065625" width="0.3048" layer="16"/>
-<wire x1="49.53" y1="3.81" x2="49.53" y2="14.45549375" width="0.3048" layer="16"/>
-<wire x1="62.5475" y1="26.9875" x2="62.5475" y2="35.56" width="0.3048" layer="16"/>
+<wire x1="49.53" y1="3.81" x2="49.53" y2="14.2875" width="0.3048" layer="16"/>
 <via x="62.5475" y="35.56" extent="1-16" drill="0.5"/>
+<wire x1="62.5475" y1="27.305" x2="62.5475" y2="35.56" width="0.3048" layer="16"/>
 <wire x1="62.5475" y1="35.56" x2="63.715" y2="35.56" width="0.3048" layer="1"/>
 <wire x1="63.8175" y1="36.2975" x2="63.715" y2="35.56" width="0.3048" layer="1"/>
 <wire x1="63.8175" y1="34.8225" x2="63.8175" y2="36.2975" width="0.3048" layer="1"/>
+<wire x1="49.53" y1="14.2875" x2="62.5475" y2="27.305" width="0.3048" layer="16"/>
 </signal>
 <signal name="CELL2">
@@
 <contactref element="R8" pad="1"/>
 <wire x1="50.8" y1="5.08" x2="50.8" y2="13.6525" width="0.3048" layer="16"/>
-<wire x1="50.8" y1="13.6525" x2="54.947571875" y2="17.800071875" width="0.3048" layer="16"/>
-<wire x1="54.947571875" y1="17.800071875" x2="59.075071875" y2="21.610071875" width="0.3048" layer="16"/>
-<wire x1="59.075071875" y1="21.610071875" x2="66.675" y2="28.8925" width="0.3048" layer="16"/>
-<wire x1="66.675" y1="28.8925" x2="66.675" y2="35.56" width="0.3048" layer="16"/>
 <via x="66.675" y="35.56" extent="1-16" drill="0.5"/>
+<wire x1="66.675" y1="29.5275" x2="66.675" y2="35.56" width="0.3048" layer="16"/>
 <wire x1="66.675" y1="35.56" x2="67.2075" y2="35.56" width="0.3048" layer="1"/>
 <wire x1="67.945" y1="36.2975" x2="67.2075" y2="35.56" width="0.3048" layer="1"/>
 <wire x1="67.945" y1="34.8225" x2="67.945" y2="36.2975" width="0.3048" layer="1"/>
+<wire x1="50.8" y1="13.6525" x2="66.675" y2="29.5275" width="0.3048" layer="16"/>
 </signal>
 <signal name="CELL3">
@@
 <wire x1="53.34" y1="5.3975" x2="52.07" y2="6.6675" width="0.3048" layer="16"/>
 <wire x1="52.07" y1="6.6675" x2="52.07" y2="13.0175" width="0.3048" layer="16"/>
-<wire x1="52.07" y1="13.0175" x2="55.245" y2="16.1925" width="0.3048" layer="16"/>
-<wire x1="55.245" y1="16.1925" x2="60.0075" y2="20.6375" width="0.3048" layer="16"/>
-<wire x1="60.0075" y1="20.6375" x2="69.5325" y2="30.1625" width="0.3048" layer="16"/>
-<wire x1="69.5325" y1="30.1625" x2="69.5325" y2="35.56" width="0.3048" layer="16"/>
 <via x="69.5325" y="35.56" extent="1-16" drill="0.5"/>
+<wire x1="69.5325" y1="30.48" x2="69.5325" y2="35.56" width="0.3048" layer="16"/>
 <wire x1="69.5325" y1="35.56" x2="70.3825" y2="35.56" width="0.3048" layer="1"/>
 <wire x1="71.12" y1="36.2975" x2="70.3825" y2="35.56" width="0.3048" layer="1"/>
 <wire x1="71.12" y1="34.8225" x2="71.12" y2="36.2975" width="0.3048" layer="1"/>
+<wire x1="52.07" y1="13.0175" x2="69.5325" y2="30.48" width="0.3048" layer="16"/>
 </signal>
 <signal name="N$17">
@@
 <wire x1="29.332575" y1="32.7025" x2="28.213175" y2="33.8219" width="0.3048" layer="16"/>
 <wire x1="25.761825" y1="33.8219" x2="24.642425" y2="32.7025" width="0.3048" layer="16"/>
-<wire x1="58.42" y1="53.34" x2="58.42" y2="52.705" width="0.3048" layer="16"/>
-<wire x1="58.42" y1="52.705" x2="57.15" y2="51.435" width="0.3048" layer="16"/>
-<wire x1="57.15" y1="51.435" x2="57.15" y2="48.26" width="0.3048" layer="16"/>
+<wire x1="58.42" y1="53.34" x2="57.15" y2="52.07" width="0.3048" layer="16"/>
+<wire x1="57.15" y1="52.07" x2="57.15" y2="48.26" width="0.3048" layer="16"/>
 <wire x1="57.15" y1="48.26" x2="49.8475" y2="40.9575" width="0.3048" layer="16"/>
 <wire x1="46.0375" y1="40.9575" x2="37.7825" y2="32.7025" width="0.3048" layer="16"/>
@@
 <wire x1="29.332575" y1="37.7825" x2="28.213175" y2="38.9019" width="0.3048" layer="16"/>
 <wire x1="25.761825" y1="38.9019" x2="24.642425" y2="37.7825" width="0.3048" layer="16"/>
-<wire x1="55.88" y1="53.34" x2="55.88" y2="52.705" width="0.3048" layer="16"/>
-<wire x1="55.88" y1="52.705" x2="54.61" y2="51.435" width="0.3048" layer="16"/>
-<wire x1="54.61" y1="51.435" x2="54.61" y2="47.625" width="0.3048" layer="16"/>
+<wire x1="55.88" y1="53.34" x2="54.61" y2="52.07" width="0.3048" layer="16"/>
+<wire x1="54.61" y1="52.07" x2="54.61" y2="47.625" width="0.3048" layer="16"/>
 <wire x1="54.61" y1="47.625" x2="49.2125" y2="42.2275" width="0.3048" layer="16"/>
 <wire x1="49.2125" y1="42.2275" x2="45.4025" y2="42.2275" width="0.3048" layer="16"/>
 <wire x1="45.4025" y1="42.2275" x2="40.9575" y2="37.7825" width="0.3048" layer="16"/>
 <wire x1="40.9575" y1="37.7825" x2="35.8775" y2="37.7825" width="0.3048" layer="16"/>
-<wire x1="11.1125" y1="37.78" x2="14.285" y2="37.78" width="0.3048" layer="1"/>
 <wire x1="14.285" y1="37.78" x2="14.2875" y2="37.7825" width="0.3048" layer="1"/>
-<wire x1="32.7025" y1="35.5575" x2="33.6525" y2="35.5575" width="0.3048" layer="1"/>
-<wire x1="33.6525" y1="35.5575" x2="35.8775" y2="37.7825" width="0.3048" layer="1"/>
+<wire x1="11.1125" y1="35.5575" x2="11.1125" y2="35.8775" width="0.3048" layer="1"/>
+<wire x1="11.1125" y1="35.8775" x2="13.0175" y2="37.7825" width="0.3048" layer="1"/>
+<wire x1="13.0175" y1="37.7825" x2="14.2875" y2="37.7825" width="0.3048" layer="1"/>
+<wire x1="32.7025" y1="35.5575" x2="32.7025" y2="35.56" width="0.3048" layer="1"/>
+<wire x1="32.7025" y1="35.56" x2="34.925" y2="37.7825" width="0.3048" layer="1"/>
+<wire x1="34.925" y1="37.7825" x2="35.8775" y2="37.7825" width="0.3048" layer="1"/>
 </signal>
 <signal name="N$23">
