File: board_v3.1/beagleboard.brd (EAGLE design)
At the start: 69.8 x 54.6 mm, 27 parts

Commit message: board3.1: updated resistors on voltage divider for power
Parts:
- R4, R5, R6: value 10k -> 4.7k
- R7: value 90k -> 45.3k
- R8: value 60k -> 27k
- R9: value 30k -> 10k
Changed lines of the file:
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@@
 <?xml version="1.0" encoding="utf-8"?>
 <!DOCTYPE eagle SYSTEM "eagle.dtd">
-<eagle version="8.2.2">
+<eagle version="8.4.0">
 <drawing>
 <settings>
 <setting alwaysvectorfont="no"/>
+<setting keepoldvectorfont="yes"/>
 <setting verticaltext="up"/>
 </settings>
@@
 <param name="dpMaxLengthDifference" value="10mm"/>
 <param name="dpGapFactor" value="2.5"/>
-<param name="checkGrid" value="0"/>
-<param name="checkAngle" value="0"/>
 <param name="checkFont" value="1"/>
 <param name="checkRestrict" value="1"/>
+<param name="checkStop" value="0"/>
 <param name="useDiameter" value="13"/>
 <param name="maxErrors" value="50"/>
@@
 <element name="MOTORL" library="pinhead" package="1X08" value="" x="14.2875" y="28.8925" rot="R270"/>
 <element name="BBGW_CONN" library="adafruit" package="BEAGLEBONE_SHIELD" value="BEAGLEBONE_OUTLINE" x="2.54" y="55.245" rot="R270"/>
-<element name="R4" library="rcl" package="R0603" value="10k" x="66.3575" y="33.9725" rot="R90"/>
-<element name="R5" library="rcl" package="R0603" value="10k" x="68.8975" y="33.9725" rot="R90"/>
-<element name="R6" library="rcl" package="R0603" value="10k" x="63.5" y="33.9725" rot="R90"/>
-<element name="R7" library="rcl" package="R0603" value="90k" x="63.5" y="37.1475" rot="R90"/>
-<element name="R8" library="rcl" package="R0603" value="60k" x="68.8975" y="37.1475" rot="R90"/>
-<element name="R9" library="rcl" package="R0603" value="30k" x="66.3575" y="37.1475" rot="R90"/>
+<element name="R4" library="rcl" package="R0603" value="4.7k" x="66.3575" y="33.9725" rot="R90"/>
+<element name="R5" library="rcl" package="R0603" value="4.7k" x="68.8975" y="33.9725" rot="R90"/>
+<element name="R6" library="rcl" package="R0603" value="4.7k" x="63.5" y="33.9725" rot="R90"/>
+<element name="R7" library="rcl" package="R0603" value="45.3k" x="63.5" y="37.1475" rot="R90"/>
+<element name="R8" library="rcl" package="R0603" value="27k" x="68.8975" y="37.1475" rot="R90"/>
+<element name="R9" library="rcl" package="R0603" value="10k" x="66.3575" y="37.1475" rot="R90"/>
 <element name="PWR_CONV" library="con-lstb" package="MA05-1" value="" x="57.785" y="35.2425" rot="R270">
 <attribute name="MF" value="" x="57.785" y="35.2425" size="1.778" layer="27" rot="R270" display="off"/>
@@
 <compatibility>
 <note version="8.2" severity="warning">
-Since Version 8.2, Eagle supports online libraries. The ids
+Since Version 8.2, EAGLE supports online libraries. The ids
 of those online libraries will not be understood (or retained)
 with this version.
