File: rysboard/rysboard.sch (KiCad schematic (older format))
At the start: 13 parts, among them J1 RPi4, J17 Conn_01x03, Q1 MBT3946DW1T1

Commit message: rysboard 4.2: * add converter output protection (shottky, D8) * fix converter resistor values (R13/R14) * add 5Vgood LED (D9) * add PWR_FLAGs for KiCAD's ERC * add NAND for motor driver's output flags * add pull-ups for motor driver's FLAG outputs
Connections:
- net ~MOTOR_BUSY renamed MOTOR_BUSY
- net ~MOTOR_FLAG renamed MOTOR_FLAG
Changed lines of the file:
@@
 Raspberry Pi 4 connector
-$Sheet
-S 8250 1500 975  600
-U 5EB7428E
-F0 "Motor Drivers" 50
-F1 "motor_drivers.sch" 50
-F2 "~STBY" I L 8250 1575 50
-F3 "~SPI_CS" I R 9225 1875 50
-F4 "SPI_CLK" I R 9225 1775 50
-F5 "SPI_MISO" O R 9225 1575 50
-F6 "SPI_MOSI" I R 9225 1675 50
-F7 "~FLAG_1" O L 8250 1675 50
-F8 "~BUSY_1" O L 8250 1775 50
-F9 "~FLAG_2" O L 8250 1875 50
-F10 "~BUSY_2" O L 8250 1975 50
-$EndSheet
 $Sheet
 S 8250 2350 975  375
@@
 	2275 3150 1700 3150
 Text Label 1700 2450 0    50   ~ 0
-~MOTOR_FLAG
+MOTOR_FLAG
 Text Label 1700 3150 0    50   ~ 0
 ~MOTOR_STBY
 Text Label 1700 3650 0    50   ~ 0
-~MOTOR_BUSY
+MOTOR_BUSY
 Wire Wire Line
 	3875 3750 4325 3750
 Wire Wire Line
-	8250 1675 7675 1675
-Text Label 7675 1675 0    50   ~ 0
-~MOTOR_FLAG
+	8250 1775 7675 1775
+Text Label 7675 1775 0    50   ~ 0
+MOTOR_FLAG
 Wire Wire Line
 	8250 1575 7675 1575
@@
 ~MOTOR_STBY
 Wire Wire Line
-	8250 1775 7675 1775
-Text Label 7675 1775 0    50   ~ 0
-~MOTOR_BUSY
+	8250 1675 7675 1675
+Text Label 7675 1675 0    50   ~ 0
+MOTOR_BUSY
 Wire Wire Line
 	9225 1575 9675 1575
@@
 Text Notes 8125 5325 0    100  ~ 0
 I2C pullups
-Wire Wire Line
-	8250 1875 7675 1875
-Text Label 7675 1875 0    50   ~ 0
-~MOTOR_FLAG
-Wire Wire Line
-	8250 1975 7675 1975
-Text Label 7675 1975 0    50   ~ 0
-~MOTOR_BUSY
 Text Label 1700 3450 0    50   ~ 0
 SPI_IRQEXT
@@
 $EndComp
 NoConn ~ 2275 2550
+$Sheet
+S 8250 1500 975  600
+U 5EB7428E
+F0 "Motor Drivers" 50
+F1 "motor_drivers.sch" 50
+F2 "~STBY" I L 8250 1575 50
+F3 "~SPI_CS" I R 9225 1875 50
+F4 "SPI_CLK" I R 9225 1775 50
+F5 "SPI_MISO" O R 9225 1575 50
+F6 "SPI_MOSI" I R 9225 1675 50
+F7 "BUSY" O L 8250 1675 50
+F8 "FLAG" O L 8250 1775 50
+$EndSheet
+$Comp
+L power:PWR_FLAG #FLG0103
+U 1 1 5EE863F0
+P 3875 1650
+F 0 "#FLG0103" H 3875 1725 50  0001 C CNN
+F 1 "PWR_FLAG" H 3875 1823 50  0000 C CNN
+F 2 "" H 3875 1650 50  0001 C CNN
+F 3 "~" H 3875 1650 50  0001 C CNN
+	1    3875 1650
+	1    0    0    -1
+$EndComp
+Wire Wire Line
+	3525 1650 3875 1650
+Connection ~ 3525 1650
 $EndSCHEMATC

Commit message: rysboard v4.2: * route the whole board (TODO: ground fills, track width checks) * fix half of ToF connectors missing ground connection * swap LEDs for easier routing
Connections:
- net LED1: now also R10.2; no longer R7.2
- net LED2: now also R7.2; no longer R10.2
Changed lines of the file:
@@
 Wire Wire Line
 	2025 7025 1700 7025
+Text Label 1700 7025 0    50   ~ 0
+LED1
 Text Label 1700 6700 0    50   ~ 0
-LED1
-Text Label 1700 7025 0    50   ~ 0
 LED2
 $Comp

Commit message: rysboard v4.2: * re-add mountting holes * fix some layout errors * add ground fills * ensure proper track width * add front-side filkscreen
Parts:
- added H1, H2, H3, H4: MountingHole_Pad, MountingHole:MountingHole_2.7mm_M2.5_Pad, symbol Mechanical:MountingHole_Pad
Connections:
- net GND: now also H1.1, H2.1, H3.1, H4.1
Other:
- note added: "Raspberry Pi 4\nmounting holes (GND)"
Changed lines of the file:
@@
 	3525 1650 3875 1650
 Connection ~ 3525 1650
+$Comp
+L Mechanical:MountingHole_Pad H1
+U 1 1 5F1ECD3F
+P 5450 1650
+F 0 "H1" V 5404 1800 50  0000 L CNN
+F 1 "MountingHole_Pad" V 5495 1800 50  0000 L CNN
+F 2 "MountingHole:MountingHole_2.7mm_M2.5_Pad" H 5450 1650 50  0001 C CNN
+F 3 "~" H 5450 1650 50  0001 C CNN
+	1    5450 1650
+	0    1    1    0
+$EndComp
+$Comp
+L Mechanical:MountingHole_Pad H2
+U 1 1 5F1EDBBD
+P 5450 1825
+F 0 "H2" V 5404 1975 50  0000 L CNN
+F 1 "MountingHole_Pad" V 5495 1975 50  0000 L CNN
+F 2 "MountingHole:MountingHole_2.7mm_M2.5_Pad" H 5450 1825 50  0001 C CNN
+F 3 "~" H 5450 1825 50  0001 C CNN
+	1    5450 1825
+	0    1    1    0
+$EndComp
+$Comp
+L Mechanical:MountingHole_Pad H3
+U 1 1 5F1F15EF
+P 5450 2000
+F 0 "H3" V 5404 2150 50  0000 L CNN
+F 1 "MountingHole_Pad" V 5495 2150 50  0000 L CNN
+F 2 "MountingHole:MountingHole_2.7mm_M2.5_Pad" H 5450 2000 50  0001 C CNN
+F 3 "~" H 5450 2000 50  0001 C CNN
+	1    5450 2000
+	0    1    1    0
+$EndComp
+$Comp
+L power:GND #PWR022
+U 1 1 5F1F8BA9
+P 5250 2175
+F 0 "#PWR022" H 5250 1925 50  0001 C CNN
+F 1 "GND" H 5255 2002 50  0000 C CNN
+F 2 "" H 5250 2175 50  0001 C CNN
+F 3 "" H 5250 2175 50  0001 C CNN
+	1    5250 2175
+	1    0    0    -1
+$EndComp
+$Comp
+L Mechanical:MountingHole_Pad H4
+U 1 1 5F22CDB3
+P 5450 2175
+F 0 "H4" V 5404 2325 50  0000 L CNN
+F 1 "MountingHole_Pad" V 5495 2325 50  0000 L CNN
+F 2 "MountingHole:MountingHole_2.7mm_M2.5_Pad" H 5450 2175 50  0001 C CNN
+F 3 "~" H 5450 2175 50  0001 C CNN
+	1    5450 2175
+	0    1    1    0
+$EndComp
+Wire Wire Line
+	5250 2175 5350 2175
+Wire Wire Line
+	5350 2175 5350 2000
+Connection ~ 5350 2175
+Wire Wire Line
+	5350 1825 5350 2000
+Connection ~ 5350 2000
+Wire Wire Line
+	5350 1650 5350 1825
+Connection ~ 5350 1825
+Text Notes 5025 1450 0    100  ~ 0
+Raspberry Pi 4\nmounting holes (GND)
 $EndSCHEMATC

Commit message: rysboard v4.2: status LED transistor swapped for BC847BS; PCB design fixes after review (!1)
Parts:
- Q1: value MBT3946DW1T1 -> BC847BS; symbol Transistor_BJT:MBT3946DW1T1 -> Transistor_BJT:BC847BS; URL (none) -> https://www.tme.eu/pl/details/bc847bs.115/tranzystory-npn-s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
Changed lines of the file:
@@
 LED2
 $Comp
-L Transistor_BJT:MBT3946DW1T1 Q1
+L Transistor_BJT:BC847BS Q1
 U 1 1 5EAE7377
 P 3400 7025
 F 0 "Q1" H 3590 7071 50  0000 L CNN
-F 1 "MBT3946DW1T1" H 3590 6980 50  0000 L CNN
+F 1 "BC847BS" H 3590 6980 50  0000 L CNN
 F 2 "Package_TO_SOT_SMD:SOT-363_SC-70-6" H 3600 7125 50  0001 C CNN
-F 3 "http://www.onsemi.com/pub_link/Collateral/MBT3946DW1T1-D.PDF" H 3400 7025 50  0001 C CNN
+F 3 "https://assets.nexperia.com/documents/data-sheet/BC847BS.pdf" H 3400 7025 50  0001 C CNN
+F 4 "https://www.tme.eu/pl/details/bc847bs.115/tranzystory-npn-smd/nexperia/" H 3400 7025 50  0001 C CNN "URL"
 	1    3400 7025
 	1    0    0    -1
 $EndComp
 $Comp
-L Transistor_BJT:MBT3946DW1T1 Q1
+L Transistor_BJT:BC847BS Q1
 U 2 1 5EAE858D
 P 2575 6700
 F 0 "Q1" H 2765 6746 50  0000 L CNN
-F 1 "MBT3946DW1T1" H 2765 6655 50  0000 L CNN
+F 1 "BC847BS" H 2765 6655 50  0000 L CNN
 F 2 "Package_TO_SOT_SMD:SOT-363_SC-70-6" H 2775 6800 50  0001 C CNN
-F 3 "http://www.onsemi.com/pub_link/Collateral/MBT3946DW1T1-D.PDF" H 2575 6700 50  0001 C CNN
+F 3 "https://assets.nexperia.com/documents/data-sheet/BC847BS.pdf" H 2575 6700 50  0001 C CNN
+F 4 "https://www.tme.eu/pl/details/bc847bs.115/tranzystory-npn-smd/nexperia/" H 2575 6700 50  0001 C CNN "URL"
 	2    2575 6700
 	1    0    0    -1

Commit message: rysboard: remove additional i2c pullups; increase high-voltage track clearance
Parts:
- removed R15, R16, R17, R18: 3K3, Resistor_SMD:R_0603_1608Metric, symbol Device:R
Other:
- note added: "I2C Note:\nRPi4 has internal pull-ups for I2C-1 bus\nand the ToF sensor boards used have a set of pull-ups\neach for their respective buses (I2C-3 and -5);\nTherefore no additional pullups are required"
- note removed: "I2C pullups"
Changed lines of the file:
@@
 I2C5_SCL
-Wire Wire Line
-	8225 5975 8225 6325
-Wire Wire Line
-	9050 5975 9050 6325
-Text Label 8225 6325 1    50   ~ 0
-I2C3_SDA
-Text Label 9050 6325 1    50   ~ 0
-I2C3_SCL
-Wire Wire Line
-	8500 5975 8500 6325
-Wire Wire Line
-	8775 5975 8775 6325
-Text Label 8775 6325 1    50   ~ 0
-I2C5_SDA
-Text Label 8500 6325 1    50   ~ 0
-I2C5_SCL
-$Comp
-L Device:R R15
-U 1 1 5EA6930C
-P 8225 5825
-F 0 "R15" H 8295 5871 50  0000 L CNN
-F 1 "3K3" H 8295 5780 50  0000 L CNN
-F 2 "Resistor_SMD:R_0603_1608Metric" V 8155 5825 50  0001 C CNN
-F 3 "~" H 8225 5825 50  0001 C CNN
-	1    8225 5825
-	1    0    0    -1
-$EndComp
-$Comp
-L Device:R R16
-U 1 1 5EA716CA
-P 8500 5825
-F 0 "R16" H 8570 5871 50  0000 L CNN
-F 1 "3K3" H 8570 5780 50  0000 L CNN
-F 2 "Resistor_SMD:R_0603_1608Metric" V 8430 5825 50  0001 C CNN
-F 3 "~" H 8500 5825 50  0001 C CNN
-	1    8500 5825
-	1    0    0    -1
-$EndComp
-$Comp
-L Device:R R17
-U 1 1 5EA764DB
-P 8775 5825
-F 0 "R17" H 8845 5871 50  0000 L CNN
-F 1 "3K3" H 8845 5780 50  0000 L CNN
-F 2 "Resistor_SMD:R_0603_1608Metric" V 8705 5825 50  0001 C CNN
-F 3 "~" H 8775 5825 50  0001 C CNN
-	1    8775 5825
-	1    0    0    -1
-$EndComp
-$Comp
-L Device:R R18
-U 1 1 5EA764E1
-P 9050 5825
-F 0 "R18" H 9120 5871 50  0000 L CNN
-F 1 "3K3" H 9120 5780 50  0000 L CNN
-F 2 "Resistor_SMD:R_0603_1608Metric" V 8980 5825 50  0001 C CNN
-F 3 "~" H 9050 5825 50  0001 C CNN
-	1    9050 5825
-	1    0    0    -1
-$EndComp
-Wire Wire Line
-	8225 5675 8500 5675
-Wire Wire Line
-	8500 5675 8650 5675
-Connection ~ 8500 5675
-Wire Wire Line
-	8775 5675 9050 5675
-Connection ~ 8775 5675
-Wire Wire Line
-	8650 5675 8650 5625
-Connection ~ 8650 5675
-Wire Wire Line
-	8650 5675 8775 5675
-$Comp
-L power:+3V3 #PWR0102
-U 1 1 5EA8A6C8
-P 8650 5625
-F 0 "#PWR0102" H 8650 5475 50  0001 C CNN
-F 1 "+3V3" H 8665 5798 50  0000 C CNN
-F 2 "" H 8650 5625 50  0001 C CNN
-F 3 "" H 8650 5625 50  0001 C CNN
-	1    8650 5625
-	1    0    0    -1
-$EndComp
 Wire Wire Line
 	2275 2950 1700 2950
@@
 Text Notes 5175 5675 0    100  ~ 0
 UART connector
-Text Notes 8125 5325 0    100  ~ 0
-I2C pullups
 Text Label 1700 3450 0    50   ~ 0
 SPI_IRQEXT
@@
 Text Notes 5025 1450 0    100  ~ 0
 Raspberry Pi 4\nmounting holes (GND)
+Text Notes 7950 5450 0    50   ~ 0
+I2C Note:\nRPi4 has internal pull-ups for I2C-1 bus\nand the ToF sensor boards used have a set of pull-ups\neach for their respective buses (I2C-3 and -5);\nTherefore no additional pullups are required
 $EndSCHEMATC

Commit message: rysboard: changed LED and sensors' VCC to 5V
Parts:
- D6: value LED_GREEN -> GREEN
- D7: value LED_RED -> RED
- R10, R7: value 4K7 -> 10k
- R11: value 43R -> 680R
- R12: value 82R -> 680R
Connections:
- net +3V3: no longer R11.2, R12.1
- net +5V: now also R11.2, R12.1
Changed lines of the file:
@@
-$EndComp
-$Comp
-L Transistor_BJT:BC847BS Q1
-U 2 1 5EAE858D
-P 2575 6700
-F 0 "Q1" H 2765 6746 50  0000 L CNN
-F 1 "BC847BS" H 2765 6655 50  0000 L CNN
-F 2 "Package_TO_SOT_SMD:SOT-363_SC-70-6" H 2775 6800 50  0001 C CNN
-F 3 "https://assets.nexperia.com/documents/data-sheet/BC847BS.pdf" H 2575 6700 50  0001 C CNN
-F 4 "https://www.tme.eu/pl/details/bc847bs.115/tranzystory-npn-smd/nexperia/" H 2575 6700 50  0001 C CNN "URL"
-	2    2575 6700
-	1    0    0    -1
 $EndComp
 $Comp
@@
 U 1 1 5EAEADD4
 P 3500 6625
-F 0 "D7" V 3600 6700 50  0000 C CNN
-F 1 "LED_RED" V 3600 6450 50  0000 C CNN
+F 0 "D7" V 3525 6525 50  0000 C CNN
+F 1 "RED" V 3450 6500 50  0000 C CNN
 F 2 "LED_SMD:LED_0805_2012Metric" H 3500 6625 50  0001 C CNN
 F 3 "~" H 3500 6625 50  0001 C CNN
@@
 U 1 1 5EAEBD9B
 P 2675 6300
-F 0 "D6" V 2775 6375 50  0000 C CNN
-F 1 "LED_GREEN" V 2775 6075 50  0000 C CNN
+F 0 "D6" V 2700 6200 50  0000 C CNN
+F 1 "GREEN" V 2625 6125 50  0000 C CNN
 F 2 "LED_SMD:LED_0805_2012Metric" H 2675 6300 50  0001 C CNN
 F 3 "~" H 2675 6300 50  0001 C CNN
@@
 P 3500 6275
 F 0 "R12" H 3570 6321 50  0000 L CNN
-F 1 "82R" H 3570 6230 50  0000 L CNN
+F 1 "680R" H 3570 6230 50  0000 L CNN
 F 2 "Resistor_SMD:R_0603_1608Metric" V 3430 6275 50  0001 C CNN
 F 3 "~" H 3500 6275 50  0001 C CNN
@@
 P 2675 5950
 F 0 "R11" H 2605 5904 50  0000 R CNN
-F 1 "43R" H 2605 5995 50  0000 R CNN
+F 1 "680R" H 2605 5995 50  0000 R CNN
 F 2 "Resistor_SMD:R_0603_1608Metric" V 2605 5950 50  0001 C CNN
 F 3 "~" H 2675 5950 50  0001 C CNN
@@
 $EndComp
 $Comp
-L power:+3V3 #PWR0104
-U 1 1 5EB07778
-P 3500 5750
-F 0 "#PWR0104" H 3500 5600 50  0001 C CNN
-F 1 "+3V3" H 3515 5923 50  0000 C CNN
-F 2 "" H 3500 5750 50  0001 C CNN
-F 3 "" H 3500 5750 50  0001 C CNN
-	1    3500 5750
-	1    0    0    -1
-$EndComp
-$Comp
 L Device:R R7
 U 1 1 5EB16B2C
 P 2175 6700
 F 0 "R7" V 1968 6700 50  0000 C CNN
-F 1 "4K7" V 2059 6700 50  0000 C CNN
+F 1 "10k" V 2059 6700 50  0000 C CNN
 F 2 "Resistor_SMD:R_0603_1608Metric" V 2105 6700 50  0001 C CNN
 F 3 "~" H 2175 6700 50  0001 C CNN
@@
 P 2175 7025
 F 0 "R10" V 1968 7025 50  0000 C CNN
-F 1 "4K7" V 2059 7025 50  0000 C CNN
+F 1 "10k" V 2059 7025 50  0000 C CNN
 F 2 "Resistor_SMD:R_0603_1608Metric" V 2105 7025 50  0001 C CNN
 F 3 "~" H 2175 7025 50  0001 C CNN
@@
 Text Notes 7950 5450 0    50   ~ 0
 I2C Note:\nRPi4 has internal pull-ups for I2C-1 bus\nand the ToF sensor boards used have a set of pull-ups\neach for their respective buses (I2C-3 and -5);\nTherefore no additional pullups are required
+$Comp
+L Transistor_BJT:BC847BS Q1
+U 2 1 5EAE858D
+P 2575 6700
+F 0 "Q1" H 2765 6746 50  0000 L CNN
+F 1 "BC847BS" H 2765 6655 50  0000 L CNN
+F 2 "Package_TO_SOT_SMD:SOT-363_SC-70-6" H 2775 6800 50  0001 C CNN
+F 3 "https://assets.nexperia.com/documents/data-sheet/BC847BS.pdf" H 2575 6700 50  0001 C CNN
+F 4 "https://www.tme.eu/pl/details/bc847bs.115/tranzystory-npn-smd/nexperia/" H 2575 6700 50  0001 C CNN "URL"
+	2    2575 6700
+	1    0    0    -1
+$EndComp
+$Comp
+L power:+5V #PWR031
+U 1 1 5ECBA57D
+P 3500 5750
+F 0 "#PWR031" H 3500 5600 50  0001 C CNN
+F 1 "+5V" H 3515 5923 50  0000 C CNN
+F 2 "" H 3500 5750 50  0001 C CNN
+F 3 "" H 3500 5750 50  0001 C CNN
+	1    3500 5750
+	1    0    0    -1
+$EndComp
 $EndSCHEMATC
