File: rysboard/Analog_Sensors.sch (KiCad schematic (older format))
At the start: 25 parts, among them J14 BAT2_TH, J21 BAT3_TH, J8 BAT1_TH, Q10 DMP2075UFDB

Commit message: more work done
Parts:
- removed R59, R61: 10KR, Resistor_SMD:R_0603_1608Metric, symbol Device:R
- removed TH3, TH4: Thermistor_PTC, Resistor_SMD:R_0805_2012Metric_Pad1.15x1.40mm_HandSolder, symbol Device:Thermistor_PTC
- added J? (x2): BAT2_TH, symbol Connector_Generic:Conn_01x02
- added R? (x2): 10KR, Resistor_SMD:R_0603_1608Metric, symbol Device:R
Connections:
- net 3_3V_REF: now also R?.1, R?.1
- net BOARD_T_2: now also J?.2 (Pin_2), R?.2
- net BOARD_T_3: now also J?.2 (Pin_2), R?.2
- net GND: now also J?.1 (Pin_1), J?.1 (Pin_1)
Other:
- moved on the sheet: Q10A, R55, R64, R66, TH2
Changed lines of the file:
@@
 Text HLabel 4100 1300 0    50   Input ~ 0
 BAT_T_3
-Text HLabel 2750 2350 0    50   Input ~ 0
+Text HLabel 2500 2525 0    50   Input ~ 0
 BOARD_T_1
-Text HLabel 3400 2350 0    50   Input ~ 0
+Text HLabel 4975 1300 0    50   Input ~ 0
 BOARD_T_2
-Text HLabel 4200 2350 0    50   Input ~ 0
-BOARD_T_3
 Text HLabel 1700 4550 0    50   Input ~ 0
 V_P_20
@@
 $EndComp
 Wire Wire Line
-	2600 2000 2750 2000
-Wire Wire Line
-	2750 2000 2750 2050
-Wire Wire Line
-	2750 2000 3400 2000
-Wire Wire Line
-	3400 2000 3400 2050
-Connection ~ 2750 2000
-Wire Wire Line
-	4200 2000 4200 2050
-Wire Wire Line
-	3400 2000 4200 2000
-Connection ~ 3400 2000
+	2350 2175 2500 2175
+Wire Wire Line
+	2500 2175 2500 2225
 $Comp
 L power:GND #PWR049
 U 1 1 603EF9F9
-P 2350 2750
-F 0 "#PWR049" H 2350 2500 50  0001 C CNN
-F 1 "GND" H 2355 2577 50  0000 C CNN
-F 2 "" H 2350 2750 50  0001 C CNN
-F 3 "" H 2350 2750 50  0001 C CNN
-	1    2350 2750
+P 2100 2925
+F 0 "#PWR049" H 2100 2675 50  0001 C CNN
+F 1 "GND" H 2105 2752 50  0000 C CNN
+F 2 "" H 2100 2925 50  0001 C CNN
+F 3 "" H 2100 2925 50  0001 C CNN
+	1    2100 2925
 	-1   0    0    -1
 $EndComp
@@
 L Device:Thermistor_PTC TH2
 U 1 1 603F0105
-P 2750 2500
-F 0 "TH2" H 2848 2546 50  0000 L CNN
-F 1 "Thermistor_PTC" H 2848 2455 50  0000 L CNN
-F 2 "Resistor_SMD:R_0805_2012Metric_Pad1.15x1.40mm_HandSolder" H 2800 2300 50  0001 L CNN
-F 3 "~" H 2750 2500 50  0001 C CNN
-	1    2750 2500
-	1    0    0    -1
-$EndComp
-$Comp
-L Device:Thermistor_PTC TH3
-U 1 1 603F0A30
-P 3400 2500
-F 0 "TH3" H 3498 2546 50  0000 L CNN
-F 1 "Thermistor_PTC" H 3498 2455 50  0000 L CNN
-F 2 "Resistor_SMD:R_0805_2012Metric_Pad1.15x1.40mm_HandSolder" H 3450 2300 50  0001 L CNN
-F 3 "~" H 3400 2500 50  0001 C CNN
-	1    3400 2500
-	1    0    0    -1
-$EndComp
-$Comp
-L Device:Thermistor_PTC TH4
-U 1 1 603F0E2B
-P 4200 2500
-F 0 "TH4" H 4298 2546 50  0000 L CNN
-F 1 "Thermistor_PTC" H 4298 2455 50  0000 L CNN
-F 2 "Resistor_SMD:R_0805_2012Metric_Pad1.15x1.40mm_HandSolder" H 4250 2300 50  0001 L CNN
-F 3 "~" H 4200 2500 50  0001 C CNN
-	1    4200 2500
-	1    0    0    -1
-$EndComp
-Wire Wire Line
-	4200 2650 3400 2650
-Wire Wire Line
-	2350 2650 2350 2750
-Connection ~ 2750 2650
-Wire Wire Line
-	2750 2650 2350 2650
-Connection ~ 3400 2650
-Wire Wire Line
-	3400 2650 2750 2650
+P 2500 2675
+F 0 "TH2" H 2598 2721 50  0000 L CNN
+F 1 "Thermistor_PTC" H 2598 2630 50  0000 L CNN
+F 2 "Resistor_SMD:R_0805_2012Metric_Pad1.15x1.40mm_HandSolder" H 2550 2475 50  0001 L CNN
+F 3 "~" H 2500 2675 50  0001 C CNN
+	1    2500 2675
+	1    0    0    -1
+$EndComp
+Wire Wire Line
+	2100 2825 2100 2925
+Wire Wire Line
+	2500 2825 2100 2825
 $Comp
 L power:+24V #PWR026
@@
 $EndComp
 Connection ~ 3150 4550
-Text GLabel 6150 1100 1    50   Output ~ 0
+Text GLabel 8625 1800 1    50   Output ~ 0
 MCU_3.3V
-Text Label 2600 2000 0    50   ~ 0
+Text Label 2350 2175 0    50   ~ 0
 MCU_Sensor_3.3V
 Text Label 1900 900  0    50   ~ 0
@@
 Wire Wire Line
 	4150 900  4150 950
-Text Label 7150 1600 0    50   ~ 0
+Text Label 9625 2300 0    50   ~ 0
 MCU_Sensor_3.3V
 $Comp
 L Device:R R55
 U 1 1 603BD637
-P 2750 2200
-F 0 "R55" H 2820 2246 50  0000 L CNN
-F 1 "10KR" H 2820 2155 50  0000 L CNN
-F 2 "Resistor_SMD:R_0603_1608Metric" V 2680 2200 50  0001 C CNN
-F 3 "~" H 2750 2200 50  0001 C CNN
-	1    2750 2200
-	1    0    0    -1
-$EndComp
-$Comp
-L Device:R R59
-U 1 1 603BDD9E
-P 3400 2200
-F 0 "R59" H 3470 2246 50  0000 L CNN
-F 1 "10KR" H 3470 2155 50  0000 L CNN
-F 2 "Resistor_SMD:R_0603_1608Metric" V 3330 2200 50  0001 C CNN
-F 3 "~" H 3400 2200 50  0001 C CNN
-	1    3400 2200
-	1    0    0    -1
-$EndComp
-$Comp
-L Device:R R61
-U 1 1 603BDFD4
-P 4200 2200
-F 0 "R61" H 4270 2246 50  0000 L CNN
-F 1 "10KR" H 4270 2155 50  0000 L CNN
-F 2 "Resistor_SMD:R_0603_1608Metric" V 4130 2200 50  0001 C CNN
-F 3 "~" H 4200 2200 50  0001 C CNN
-	1    4200 2200
-	1    0    0    -1
-$EndComp
-Wire Wire Line
-	7150 1600 6750 1600
-Wire Wire Line
-	6150 1100 6300 1100
-Wire Wire Line
-	6750 1100 6750 1200
+P 2500 2375
+F 0 "R55" H 2570 2421 50  0000 L CNN
+F 1 "10KR" H 2570 2330 50  0000 L CNN
+F 2 "Resistor_SMD:R_0603_1608Metric" V 2430 2375 50  0001 C CNN
+F 3 "~" H 2500 2375 50  0001 C CNN
+	1    2500 2375
+	1    0    0    -1
+$EndComp
+Wire Wire Line
+	9625 2300 9225 2300
+Wire Wire Line
+	8625 1800 8775 1800
+Wire Wire Line
+	9225 1800 9225 1900
 $Comp
 L Device:R R66
 U 1 1 603C19CD
-P 6300 1250
-F 0 "R66" H 6370 1296 50  0000 L CNN
-F 1 "100KR" H 6370 1205 50  0000 L CNN
-F 2 "Resistor_SMD:R_0603_1608Metric" V 6230 1250 50  0001 C CNN
-F 3 "~" H 6300 1250 50  0001 C CNN
-	1    6300 1250
-	1    0    0    -1
-$EndComp
-Connection ~ 6300 1100
-Wire Wire Line
-	6300 1100 6750 1100
+P 8775 1950
+F 0 "R66" H 8845 1996 50  0000 L CNN
+F 1 "100KR" H 8845 1905 50  0000 L CNN
+F 2 "Resistor_SMD:R_0603_1608Metric" V 8705 1950 50  0001 C CNN
+F 3 "~" H 8775 1950 50  0001 C CNN
+	1    8775 1950
+	1    0    0    -1
+$EndComp
+Connection ~ 8775 1800
+Wire Wire Line
+	8775 1800 9225 1800
 $Comp
 L Device:R R64
 U 1 1 603C1DE2
-P 6150 1400
-F 0 "R64" H 6220 1446 50  0000 L CNN
-F 1 "10KR" H 6220 1355 50  0000 L CNN
-F 2 "Resistor_SMD:R_0603_1608Metric" V 6080 1400 50  0001 C CNN
-F 3 "~" H 6150 1400 50  0001 C CNN
-	1    6150 1400
+P 8625 2100
+F 0 "R64" H 8695 2146 50  0000 L CNN
+F 1 "10KR" H 8695 2055 50  0000 L CNN
+F 2 "Resistor_SMD:R_0603_1608Metric" V 8555 2100 50  0001 C CNN
+F 3 "~" H 8625 2100 50  0001 C CNN
+	1    8625 2100
 	0    1    1    0
 $EndComp
 Wire Wire Line
-	6300 1400 6450 1400
-Connection ~ 6300 1400
-Text HLabel 5850 1400 0    50   Input ~ 0
+	8775 2100 8925 2100
+Connection ~ 8775 2100
+Text HLabel 8325 2100 0    50   Input ~ 0
 S_E
 Wire Wire Line
-	5850 1400 6000 1400
+	8325 2100 8475 2100
 Text Notes 8450 1000 0    50   ~ 0
 When not used, thermistors do not need to be powered on.
@@
 	1    0    0    -1
 $EndComp
-Text HLabel 6950 1600 3    50   Input ~ 0
+Text HLabel 9425 2300 3    50   Input ~ 0
 3_3V_REF
 $Comp
 L rysboard:DMP2075UFDB Q10
 U 1 1 605EDFDE
-P 6650 1400
-F 0 "Q10" H 6855 1354 50  0000 L CNN
-F 1 "DMP2075UFDB" H 6855 1445 50  0000 L CNN
-F 2 "SamacSys_Parts:DMP2075UFDB7" H 6850 1325 50  0001 L CIN
-F 3 "" H 6650 1400 50  0001 L CNN
-	1    6650 1400
+P 9125 2100
+F 0 "Q10" H 9330 2054 50  0000 L CNN
+F 1 "DMP2075UFDB" H 9330 2145 50  0000 L CNN
+F 2 "SamacSys_Parts:DMP2075UFDB7" H 9325 2025 50  0001 L CIN
+F 3 "" H 9125 2100 50  0001 L CNN
+	1    9125 2100
 	1    0    0    1
 $EndComp
+Text Label 4325 900  0    50   ~ 0
+MCU_Sensor_3.3V
+Text Label 5100 900  0    50   ~ 0
+MCU_Sensor_3.3V
+$Comp
+L Device:R R?
+U 1 1 604C3349
+P 4975 1050
+F 0 "R?" H 5045 1096 50  0000 L CNN
+F 1 "10KR" H 5045 1005 50  0000 L CNN
+F 2 "Resistor_SMD:R_0603_1608Metric" V 4905 1050 50  0001 C CNN
+F 3 "~" H 4975 1050 50  0001 C CNN
+	1    4975 1050
+	1    0    0    -1
+$EndComp
+$Comp
+L Connector_Generic:Conn_01x02 J?
+U 1 1 604C3809
+P 5075 1550
+F 0 "J?" V 4947 1630 50  0000 L CNN
+F 1 "BAT2_TH" V 5038 1630 50  0000 L CNN
+F 2 "" H 5075 1550 50  0001 C CNN
+F 3 "~" H 5075 1550 50  0001 C CNN
+	1    5075 1550
+	0    1    1    0
+$EndComp
+$Comp
+L Connector_Generic:Conn_01x02 J?
+U 1 1 604C3EA4
+P 5850 1550
+F 0 "J?" V 5722 1630 50  0000 L CNN
+F 1 "BAT2_TH" V 5813 1630 50  0000 L CNN
+F 2 "" H 5850 1550 50  0001 C CNN
+F 3 "~" H 5850 1550 50  0001 C CNN
+	1    5850 1550
+	0    1    1    0
+$EndComp
+$Comp
+L Device:R R?
+U 1 1 604C4170
+P 5750 1050
+F 0 "R?" H 5820 1096 50  0000 L CNN
+F 1 "10KR" H 5820 1005 50  0000 L CNN
+F 2 "Resistor_SMD:R_0603_1608Metric" V 5680 1050 50  0001 C CNN
+F 3 "~" H 5750 1050 50  0001 C CNN
+	1    5750 1050
+	1    0    0    -1
+$EndComp
+Wire Wire Line
+	5100 900  5750 900
+Wire Wire Line
+	4325 900  4975 900
+Wire Wire Line
+	4975 1200 4975 1350
+Text HLabel 5750 1275 0    50   Input ~ 0
+BOARD_T_3
+Wire Wire Line
+	5750 1200 5750 1350
+$Comp
+L power:GND #PWR?
+U 1 1 604C7572
+P 5075 1350
+F 0 "#PWR?" H 5075 1100 50  0001 C CNN
+F 1 "GND" H 5080 1177 50  0000 C CNN
+F 2 "" H 5075 1350 50  0001 C CNN
+F 3 "" H 5075 1350 50  0001 C CNN
+	1    5075 1350
+	0    -1   -1   0
+$EndComp
+$Comp
+L power:GND #PWR?
+U 1 1 604C77C4
+P 5850 1350
+F 0 "#PWR?" H 5850 1100 50  0001 C CNN
+F 1 "GND" H 5855 1177 50  0000 C CNN
+F 2 "" H 5850 1350 50  0001 C CNN
+F 3 "" H 5850 1350 50  0001 C CNN
+	1    5850 1350
+	0    -1   -1   0
+$EndComp
 $EndSCHEMATC
