File: rysboard/Analog_Sensors.sch (KiCad schematic (older format))
At the start: 21 parts, among them J22 CH1_T, J23 CH2_T, Q2 DMP2075UFDB

Commit message: mcu IO
Parts:
- gave numbers to parts that had none: 2
Connections:
- net labels added: +BATT, BOARD_T_2
- net labels removed: +24V
Changed lines of the file:
@@
 	3150 3175 2750 3175
-$Comp
-L power:+24V #PWR026
-U 1 1 603F23C7
-P 2775 4075
-F 0 "#PWR026" H 2775 3925 50  0001 C CNN
-F 1 "+24V" H 2790 4248 50  0000 C CNN
-F 2 "" H 2775 4075 50  0001 C CNN
-F 3 "" H 2775 4075 50  0001 C CNN
-	1    2775 4075
-	1    0    0    -1
-$EndComp
 $Comp
 L power:+5V #PWR051
@@
 $EndComp
 $Comp
-L Device:Thermistor_PTC TH?
+L Device:Thermistor_PTC TH1
 U 1 1 6063752B
 P 3975 3025
-F 0 "TH?" H 4073 3071 50  0000 L CNN
+F 0 "TH1" H 4073 3071 50  0000 L CNN
 F 1 "Thermistor_PTC" H 4073 2980 50  0000 L CNN
 F 2 "Resistor_SMD:R_0805_2012Metric_Pad1.15x1.40mm_HandSolder" H 4025 2825 50  0001 L CNN
@@
 Connection ~ 3150 3175
 $Comp
-L Device:R R?
+L Device:R R31
 U 1 1 6063841E
 P 3975 2700
-F 0 "R?" H 4045 2746 50  0000 L CNN
+F 0 "R31" H 4045 2746 50  0000 L CNN
 F 1 "10KR" H 4045 2655 50  0000 L CNN
 F 2 "Resistor_SMD:R_0603_1608Metric" V 3905 2700 50  0001 C CNN
@@
 Wire Wire Line
 	3975 2875 3975 2850
+$Comp
+L power:+BATT #PWR0115
+U 1 1 60625717
+P 2775 4075
+F 0 "#PWR0115" H 2775 3925 50  0001 C CNN
+F 1 "+BATT" H 2790 4248 50  0000 C CNN
+F 2 "" H 2775 4075 50  0001 C CNN
+F 3 "" H 2775 4075 50  0001 C CNN
+	1    2775 4075
+	1    0    0    -1
+$EndComp
+Text HLabel 3975 2875 0    50   Input ~ 0
+BOARD_T_2
 $EndSCHEMATC

Commit message: MCU Sensors Done
Parts:
- added C32: 0,1uF, Capacitor_SMD:C_0603_1608Metric, symbol Device:C
Connections:
- net GND: now also C32.2
- net MCU_ANALOG_SENSOR_V: now also C32.1
Changed lines of the file:
@@
 When not used, thermistors do not need to be powered on.
-$Comp
-L rysboard:DMP2075UFDB Q2
-U 1 1 605EDFDE
-P 9125 2100
-F 0 "Q2" H 9330 2054 50  0000 L CNN
-F 1 "DMP2075UFDB" H 9330 2145 50  0000 L CNN
-F 2 "SamacSys_Parts:DMP2075UFDB7" H 9325 2025 50  0001 L CIN
-F 3 "" H 9125 2100 50  0001 L CNN
-	1    9125 2100
-	1    0    0    1
-$EndComp
 $Comp
 L Device:R R61
@@
 MCU_ANALOG_SENSOR_V
 Wire Wire Line
-	9850 2300 9225 2300
+	9850 2300 9600 2300
 Text GLabel 6150 925  2    50   Input ~ 0
 MCU_ANALOG_SENSOR_V
@@
 Text HLabel 3975 2875 0    50   Input ~ 0
 BOARD_T_2
+$Comp
+L rysboard:DMP2075UFDB Q2
+U 1 1 605EDFDE
+P 9125 2100
+F 0 "Q2" H 9330 2054 50  0000 L CNN
+F 1 "DMP2075UFDB" H 9330 2145 50  0000 L CNN
+F 2 "SamacSys_Parts:DMP2075UFDB7" H 9325 2025 50  0001 L CIN
+F 3 "" H 9125 2100 50  0001 L CNN
+	1    9125 2100
+	1    0    0    1
+$EndComp
+$Comp
+L Device:C C32
+U 1 1 6069F647
+P 9600 2450
+F 0 "C32" H 9715 2496 50  0000 L CNN
+F 1 "0,1uF" H 9715 2405 50  0000 L CNN
+F 2 "Capacitor_SMD:C_0603_1608Metric" H 9638 2300 50  0001 C CNN
+F 3 "~" H 9600 2450 50  0001 C CNN
+	1    9600 2450
+	1    0    0    -1
+$EndComp
+Connection ~ 9600 2300
+Wire Wire Line
+	9600 2300 9225 2300
+$Comp
+L power:GND #PWR0116
+U 1 1 6069FD9A
+P 9600 2600
+F 0 "#PWR0116" H 9600 2350 50  0001 C CNN
+F 1 "GND" H 9605 2427 50  0000 C CNN
+F 2 "" H 9600 2600 50  0001 C CNN
+F 3 "" H 9600 2600 50  0001 C CNN
+	1    9600 2600
+	-1   0    0    -1
+$EndComp
 $EndSCHEMATC

Commit message: version pre changes due to scarsity of parts
Parts:
- added Q?: AO3401A, Package_TO_SOT_SMD:SOT-23, symbol Transistor_FET:AO3401A
Changed lines of the file:
@@
 	-1   0    0    -1
 $EndComp
+$Comp
+L Transistor_FET:AO3401A Q?
+U 1 1 608D8760
+P 8125 2825
+F 0 "Q?" H 8330 2871 50  0000 L CNN
+F 1 "AO3401A" H 8330 2780 50  0000 L CNN
+F 2 "Package_TO_SOT_SMD:SOT-23" H 8325 2750 50  0001 L CIN
+F 3 "http://www.aosmd.com/pdfs/datasheet/AO3401A.pdf" H 8125 2825 50  0001 L CNN
+	1    8125 2825
+	1    0    0    -1
+$EndComp
 $EndSCHEMATC

Commit message: Bom finished pcb cleanup started
Parts:
- removed Q2: DMP2075UFDB, SamacSys_Parts:DMP2075UFDB7, symbol rysboard:DMP2075UFDB
- J22, J23: footprint Connector_PinHeader_1.00mm:PinHeader_1x02_P1.00mm_Vertical -> Connector_PinHeader_1.27mm:PinHeader_1x02_P1.27mm_Vertical
- gave numbers to parts that had none: 1
Connections:
- net MCU_3.3V: now also Q10.2 (S)
- net MCU_ANALOG_SENSOR_V: now also Q10.3 (D)
- net at R64.1, R66.2: now also Q10.1 (G)
Other:
- moved on the sheet: Q10
Changed lines of the file:
@@
 F 0 "J23" V 6122 1655 50  0000 L CNN
 F 1 "CH2_T" V 6213 1655 50  0000 L CNN
-F 2 "Connector_PinHeader_1.00mm:PinHeader_1x02_P1.00mm_Vertical" H 6250 1575 50  0001 C CNN
+F 2 "Connector_PinHeader_1.27mm:PinHeader_1x02_P1.27mm_Vertical" H 6250 1575 50  0001 C CNN
 F 3 "~" H 6250 1575 50  0001 C CNN
 	1    6250 1575
@@
 F 0 "J22" V 5222 1630 50  0000 L CNN
 F 1 "CH1_T" V 5313 1630 50  0000 L CNN
-F 2 "Connector_PinHeader_1.00mm:PinHeader_1x02_P1.00mm_Vertical" H 5350 1550 50  0001 C CNN
+F 2 "Connector_PinHeader_1.27mm:PinHeader_1x02_P1.27mm_Vertical" H 5350 1550 50  0001 C CNN
 F 3 "~" H 5350 1550 50  0001 C CNN
 	1    5350 1550
@@
 BOARD_T_2
 $Comp
-L rysboard:DMP2075UFDB Q2
-U 1 1 605EDFDE
-P 9125 2100
-F 0 "Q2" H 9330 2054 50  0000 L CNN
-F 1 "DMP2075UFDB" H 9330 2145 50  0000 L CNN
-F 2 "SamacSys_Parts:DMP2075UFDB7" H 9325 2025 50  0001 L CIN
-F 3 "" H 9125 2100 50  0001 L CNN
-	1    9125 2100
-	1    0    0    1
-$EndComp
-$Comp
 L Device:C C32
 U 1 1 6069F647
@@
 $EndComp
 $Comp
-L Transistor_FET:AO3401A Q?
+L Transistor_FET:AO3401A Q10
 U 1 1 608D8760
-P 8125 2825
-F 0 "Q?" H 8330 2871 50  0000 L CNN
-F 1 "AO3401A" H 8330 2780 50  0000 L CNN
-F 2 "Package_TO_SOT_SMD:SOT-23" H 8325 2750 50  0001 L CIN
-F 3 "http://www.aosmd.com/pdfs/datasheet/AO3401A.pdf" H 8125 2825 50  0001 L CNN
-	1    8125 2825
-	1    0    0    -1
+P 9125 2100
+F 0 "Q10" H 9330 2054 50  0000 L CNN
+F 1 "AO3401A" H 9330 2145 50  0000 L CNN
+F 2 "Package_TO_SOT_SMD:SOT-23" H 9325 2025 50  0001 L CIN
+F 3 "http://www.aosmd.com/pdfs/datasheet/AO3401A.pdf" H 9125 2100 50  0001 L CNN
+	1    9125 2100
+	1    0    0    1
 $EndComp
 $EndSCHEMATC

Commit message: bom + excel ready
Parts:
- added D7: CD0603-Z3, Diode_SMD:D_0603_1608Metric, symbol Device:D_Zener
- added R34: 10k1%, Resistor_SMD:R_0603_1608Metric, symbol Device:R
- added R35: 2.8KR, Resistor_SMD:R_0603_1608Metric, symbol Device:R
- C32: value 0,1uF -> 100n
- Q10: value AO3401A -> PMV28XPEAR
- R31, R55, R56, R59, R61, R62, R64, R70: value 10KR -> 10k1%
Connections:
- net GND: now also D7.2 (A), R35.2
- new net DC_IN_Voltage: R34.1
- new net V_IN_DIV: D7.1 (K), R34.2, R35.1
Other:
- note added: "3.6V zener diode prot\n"
Changed lines of the file:
@@
 P 6250 4400
 F 0 "R62" H 6320 4446 50  0000 L CNN
-F 1 "10KR" H 6320 4355 50  0000 L CNN
+F 1 "10k1%" H 6320 4355 50  0000 L CNN
 F 2 "Resistor_SMD:R_0603_1608Metric" V 6180 4400 50  0001 C CNN
 F 3 "~" H 6250 4400 50  0001 C CNN
@@
 Text Notes 6950 3650 0    50   ~ 0
 0-9.9V\n
-Text Notes 7750 3650 0    50   ~ 0
+Text Notes 7700 3650 0    50   ~ 0
 0-15.086V\n
-$Comp
-L Device:R R71
-U 1 1 603B8D2E
-P 7850 4400
-F 0 "R71" H 7920 4446 50  0000 L CNN
-F 1 "10KR" H 7920 4355 50  0000 L CNN
-F 2 "Resistor_SMD:R_0603_1608Metric" V 7780 4400 50  0001 C CNN
-F 3 "~" H 7850 4400 50  0001 C CNN
-	1    7850 4400
-	1    0    0    -1
-$EndComp
 $Comp
 L Device:R R56
@@
 P 3875 4225
 F 0 "R56" H 3945 4271 50  0000 L CNN
-F 1 "10KR" H 3945 4180 50  0000 L CNN
+F 1 "10k1%" H 3945 4180 50  0000 L CNN
 F 2 "Resistor_SMD:R_0603_1608Metric" V 3805 4225 50  0001 C CNN
 F 3 "~" H 3875 4225 50  0001 C CNN
@@
 P 3150 2725
 F 0 "R55" H 3220 2771 50  0000 L CNN
-F 1 "10KR" H 3220 2680 50  0000 L CNN
+F 1 "10k1%" H 3220 2680 50  0000 L CNN
 F 2 "Resistor_SMD:R_0603_1608Metric" V 3080 2725 50  0001 C CNN
 F 3 "~" H 3150 2725 50  0001 C CNN
@@
 P 8625 2100
 F 0 "R64" H 8695 2146 50  0000 L CNN
-F 1 "10KR" H 8695 2055 50  0000 L CNN
+F 1 "10k1%" H 8695 2055 50  0000 L CNN
 F 2 "Resistor_SMD:R_0603_1608Metric" V 8555 2100 50  0001 C CNN
 F 3 "~" H 8625 2100 50  0001 C CNN
@@
 P 6150 1075
 F 0 "R61" H 6220 1121 50  0000 L CNN
-F 1 "10KR" H 6220 1030 50  0000 L CNN
+F 1 "10k1%" H 6220 1030 50  0000 L CNN
 F 2 "Resistor_SMD:R_0603_1608Metric" V 6080 1075 50  0001 C CNN
 F 3 "~" H 6150 1075 50  0001 C CNN
@@
 P 5250 1050
 F 0 "R59" H 5320 1096 50  0000 L CNN
-F 1 "10KR" H 5320 1005 50  0000 L CNN
+F 1 "10k1%" H 5320 1005 50  0000 L CNN
 F 2 "Resistor_SMD:R_0603_1608Metric" V 5180 1050 50  0001 C CNN
 F 3 "~" H 5250 1050 50  0001 C CNN
@@
 P 7050 4400
 F 0 "R70" H 7120 4446 50  0000 L CNN
-F 1 "10KR" H 7120 4355 50  0000 L CNN
+F 1 "10k1%" H 7120 4355 50  0000 L CNN
 F 2 "Resistor_SMD:R_0603_1608Metric" V 6980 4400 50  0001 C CNN
 F 3 "~" H 7050 4400 50  0001 C CNN
@@
 P 3975 2700
 F 0 "R31" H 4045 2746 50  0000 L CNN
-F 1 "10KR" H 4045 2655 50  0000 L CNN
+F 1 "10k1%" H 4045 2655 50  0000 L CNN
 F 2 "Resistor_SMD:R_0603_1608Metric" V 3905 2700 50  0001 C CNN
 F 3 "~" H 3975 2700 50  0001 C CNN
@@
 P 9600 2450
 F 0 "C32" H 9715 2496 50  0000 L CNN
-F 1 "0,1uF" H 9715 2405 50  0000 L CNN
+F 1 "100n" H 9715 2405 50  0000 L CNN
 F 2 "Capacitor_SMD:C_0603_1608Metric" H 9638 2300 50  0001 C CNN
 F 3 "~" H 9600 2450 50  0001 C CNN
@@
 P 9125 2100
 F 0 "Q10" H 9330 2054 50  0000 L CNN
-F 1 "AO3401A" H 9330 2145 50  0000 L CNN
+F 1 "PMV28XPEAR" H 9330 2145 50  0000 L CNN
 F 2 "Package_TO_SOT_SMD:SOT-23" H 9325 2025 50  0001 L CIN
 F 3 "http://www.aosmd.com/pdfs/datasheet/AO3401A.pdf" H 9125 2100 50  0001 L CNN
@@
 	1    0    0    1
 $EndComp
+$Comp
+L Device:R R34
+U 1 1 6090FB78
+P 9100 4425
+F 0 "R34" H 9170 4471 50  0000 L CNN
+F 1 "10k1%" H 9170 4380 50  0000 L CNN
+F 2 "Resistor_SMD:R_0603_1608Metric" V 9030 4425 50  0001 C CNN
+F 3 "~" H 9100 4425 50  0001 C CNN
+	1    9100 4425
+	1    0    0    -1
+$EndComp
+$Comp
+L Device:R R35
+U 1 1 6090FD40
+P 9100 4725
+F 0 "R35" H 9170 4771 50  0000 L CNN
+F 1 "2.8KR" H 9170 4680 50  0000 L CNN
+F 2 "Resistor_SMD:R_0603_1608Metric" V 9030 4725 50  0001 C CNN
+F 3 "~" H 9100 4725 50  0001 C CNN
+	1    9100 4725
+	1    0    0    -1
+$EndComp
+$Comp
+L power:GND #PWR0117
+U 1 1 609100DD
+P 9100 4875
+F 0 "#PWR0117" H 9100 4625 50  0001 C CNN
+F 1 "GND" H 9105 4702 50  0000 C CNN
+F 2 "" H 9100 4875 50  0001 C CNN
+F 3 "" H 9100 4875 50  0001 C CNN
+	1    9100 4875
+	-1   0    0    -1
+$EndComp
+Text GLabel 9100 4275 1    50   Input ~ 0
+DC_IN_Voltage
+Text HLabel 8750 4575 0    50   Input ~ 0
+V_IN_DIV
+Wire Wire Line
+	8750 4575 8875 4575
+Connection ~ 9100 4575
+Connection ~ 8875 4575
+Wire Wire Line
+	8875 4575 9100 4575
+Wire Wire Line
+	8875 4875 9100 4875
+Connection ~ 9100 4875
+Text Notes 8900 3625 0    50   ~ 0
+0-15.086V\n
+Text Notes 8350 5225 0    50   ~ 0
+3.6V zener diode prot\n
+$Comp
+L Device:D_Zener D7
+U 1 1 6092677E
+P 8875 4725
+F 0 "D7" V 8829 4805 50  0000 L CNN
+F 1 "CD0603-Z3" V 8975 4200 50  0000 L CNN
+F 2 "Diode_SMD:D_0603_1608Metric" H 8875 4725 50  0001 C CNN
+F 3 "~" H 8875 4725 50  0001 C CNN
+	1    8875 4725
+	0    1    1    0
+$EndComp
+$Comp
+L Device:R R71
+U 1 1 603B8D2E
+P 7850 4400
+F 0 "R71" H 7920 4446 50  0000 L CNN
+F 1 "10KR" H 7920 4355 50  0000 L CNN
+F 2 "Resistor_SMD:R_0603_1608Metric" V 7780 4400 50  0001 C CNN
+F 3 "~" H 7850 4400 50  0001 C CNN
+	1    7850 4400
+	1    0    0    -1
+$EndComp
 $EndSCHEMATC

Commit message: New Layout done TODo Error Check
Parts:
- removed D7: CD0603-Z3, Diode_SMD:D_0603_1608Metric, symbol Device:D_Zener
- removed R34: 10k1%, Resistor_SMD:R_0603_1608Metric, symbol Device:R
- removed R35: 2.8KR, Resistor_SMD:R_0603_1608Metric, symbol Device:R
Other:
- note removed: "3.6V zener diode prot\n"
Changed lines of the file:
@@
 Text HLabel 1600 5650 0    50   Input ~ 0
 BAT_CS
-Text HLabel 6250 4550 0    50   Input ~ 0
+Text HLabel 6025 4550 0    50   Input ~ 0
 V_BAT_C1
 Text HLabel 7050 4550 0    50   Input ~ 0
@@
 $EndComp
 $Comp
-L Device:R R34
-U 1 1 6090FB78
-P 9100 4425
-F 0 "R34" H 9170 4471 50  0000 L CNN
-F 1 "10k1%" H 9170 4380 50  0000 L CNN
-F 2 "Resistor_SMD:R_0603_1608Metric" V 9030 4425 50  0001 C CNN
-F 3 "~" H 9100 4425 50  0001 C CNN
-	1    9100 4425
-	1    0    0    -1
-$EndComp
-$Comp
-L Device:R R35
-U 1 1 6090FD40
-P 9100 4725
-F 0 "R35" H 9170 4771 50  0000 L CNN
-F 1 "2.8KR" H 9170 4680 50  0000 L CNN
-F 2 "Resistor_SMD:R_0603_1608Metric" V 9030 4725 50  0001 C CNN
-F 3 "~" H 9100 4725 50  0001 C CNN
-	1    9100 4725
-	1    0    0    -1
-$EndComp
-$Comp
-L power:GND #PWR0117
-U 1 1 609100DD
-P 9100 4875
-F 0 "#PWR0117" H 9100 4625 50  0001 C CNN
-F 1 "GND" H 9105 4702 50  0000 C CNN
-F 2 "" H 9100 4875 50  0001 C CNN
-F 3 "" H 9100 4875 50  0001 C CNN
-	1    9100 4875
-	-1   0    0    -1
-$EndComp
-Text GLabel 9100 4275 1    50   Input ~ 0
-DC_IN_Voltage
-Text HLabel 8750 4575 0    50   Input ~ 0
-V_IN_DIV
-Wire Wire Line
-	8750 4575 8875 4575
-Connection ~ 9100 4575
-Connection ~ 8875 4575
-Wire Wire Line
-	8875 4575 9100 4575
-Wire Wire Line
-	8875 4875 9100 4875
-Connection ~ 9100 4875
-Text Notes 8900 3625 0    50   ~ 0
-0-15.086V\n
-Text Notes 8350 5225 0    50   ~ 0
-3.6V zener diode prot\n
-$Comp
-L Device:D_Zener D7
-U 1 1 6092677E
-P 8875 4725
-F 0 "D7" V 8829 4805 50  0000 L CNN
-F 1 "CD0603-Z3" V 8975 4200 50  0000 L CNN
-F 2 "Diode_SMD:D_0603_1608Metric" H 8875 4725 50  0001 C CNN
-F 3 "~" H 8875 4725 50  0001 C CNN
-	1    8875 4725
-	0    1    1    0
-$EndComp
-$Comp
 L Device:R R71
 U 1 1 603B8D2E
@@
 	1    0    0    -1
 $EndComp
+Connection ~ 6250 4550
+Wire Wire Line
+	6025 4550 6250 4550
 $EndSCHEMATC
