File: rysboard/sensors.sch (KiCad schematic (older format))
At the start: 11 parts, among them J10 ToF1, J11 ToF2, J12 ToF3, J13 ToF4, J15 ToF5, J16 ToF6, J9 IMU, Q11 AO3401A, Q7 NST847BDP6T5G

Commit message: bom + excel ready
Parts:
- Q11: value AO3401A -> PMV28XPEAR
- R51: value 10KR -> 10k1%
Changed lines of the file:
@@
 P 4900 1400
 F 0 "R51" H 4970 1446 50  0000 L CNN
-F 1 "10KR" H 4970 1355 50  0000 L CNN
+F 1 "10k1%" H 4970 1355 50  0000 L CNN
 F 2 "Resistor_SMD:R_0603_1608Metric" V 4830 1400 50  0001 C CNN
 F 3 "~" H 4900 1400 50  0001 C CNN
@@
 P 5250 1350
 F 0 "Q11" V 5592 1350 50  0000 C CNN
-F 1 "AO3401A" V 5501 1350 50  0000 C CNN
+F 1 "PMV28XPEAR" V 5501 1350 50  0000 C CNN
 F 2 "Package_TO_SOT_SMD:SOT-23" H 5450 1275 50  0001 L CIN
 F 3 "http://www.aosmd.com/pdfs/datasheet/AO3401A.pdf" H 5250 1350 50  0001 L CNN
