File: rysboard/Battery_Balancing.sch (KiCad schematic (older format))
At the start: 45 parts, among them J4 Cell3, J5 Cell2, J6 Cell1, J7 Power_SW, Q12 Si7938DP-T1-GE3, Q13 SI7997DP-T1-GE3, Q14 DMP2075UFDB-7-alt, Q9 Si7938DP-T1-GE3, U11 bq77915, U9 INA181

Commit message: Even More footprints
Parts:
- added D15: KDZVTR2.0B, Diode_SMD:D_SOD-123F, symbol Device:D_Zener
- added R40: 10KR, Resistor_SMD:R_0603_1608Metric, symbol Device:R
- D16: value D_Zener -> TSZU52C10 RG; footprint (none) -> Diode_SMD:D_0603_1608Metric
- R35: footprint (none) -> Resistor_SMD:R_0603_1608Metric
Connections:
- net at U9.5 (REF): now also D15.1 (K), R40.2
- net MCU_3.3V renamed MCU_ANALOG_SENSOR_V
- net MCU_ANALOG_SENSOR_V: now also R40.1
- new net GND: D15.2 (A)
- no-connect marks 4 -> 3
Other:
- note added: "2V reference, for offset. \nUsed in ADC compensation,\n And measuring negative current"
- moved on the sheet: C33, U9
Changed lines of the file:
@@
 F 0 "R35" V 4893 5350 50  0000 C CNN
 F 1 "10KR" V 4984 5350 50  0000 C CNN
-F 2 "" V 5030 5350 50  0001 C CNN
+F 2 "Resistor_SMD:R_0603_1608Metric" V 5030 5350 50  0001 C CNN
 F 3 "~" H 5100 5350 50  0001 C CNN
 	1    5100 5350
@@
 P 4800 7600
 F 0 "D16" V 5200 7600 50  0000 C CNN
-F 1 "D_Zener" V 5100 7600 50  0000 C CNN
-F 2 "" H 4800 7600 50  0001 C CNN
+F 1 "TSZU52C10 RG" V 5100 7600 50  0000 C CNN
+F 2 "Diode_SMD:D_0603_1608Metric" H 4800 7600 50  0001 C CNN
 F 3 "~" H 4800 7600 50  0001 C CNN
 	1    4800 7600
@@
 Text Notes 900  9100 0    50   ~ 0
 Current Measurement Filters\n
-Text GLabel 3750 9550 2    50   Input ~ 0
+Text GLabel 3475 9275 2    50   Input ~ 0
 Bat_Current_Pos
 $Comp
@@
 L Amplifier_Current:INA181 U9
 U 1 1 60015B2B
-P 3050 9550
-F 0 "U9" H 3394 9596 50  0000 L CNN
-F 1 "INA181" H 3394 9505 50  0000 L CNN
-F 2 "Package_TO_SOT_SMD:SOT-23-6" H 3100 9600 50  0001 C CNN
-F 3 "http://www.ti.com/lit/ds/symlink/ina181.pdf" H 3200 9700 50  0001 C CNN
-	1    3050 9550
+P 3000 9275
+F 0 "U9" H 3300 9325 50  0000 L CNN
+F 1 "INA181" H 3200 9225 50  0000 L CNN
+F 2 "Package_TO_SOT_SMD:SOT-23-6" H 3050 9325 50  0001 C CNN
+F 3 "http://www.ti.com/lit/ds/symlink/ina181.pdf" H 3150 9425 50  0001 C CNN
+	1    3000 9275
 	1    0    0    -1
 $EndComp
-Wire Wire Line
-	3750 9550 3350 9550
-Text GLabel 3350 9250 2    50   Output ~ 0
-MCU_3.3V
-Text Label 2950 10000 3    50   ~ 0
+Text GLabel 3300 8975 2    50   Output ~ 0
+MCU_ANALOG_SENSOR_V
+Text Label 2900 9725 3    50   ~ 0
 V_BAT_AF_PROT-
 Wire Wire Line
-	2950 10000 2950 9850
+	2900 9725 2900 9575
 $Comp
 L Device:C C33
 U 1 1 600598E6
-P 3200 9100
-F 0 "C33" H 3085 9054 50  0000 R CNN
-F 1 "0.1uF10%" H 3085 9145 50  0000 R CNN
-F 2 "Capacitor_SMD:C_0603_1608Metric_Pad1.05x0.95mm_HandSolder" H 3238 8950 50  0001 C CNN
-F 3 "~" H 3200 9100 50  0001 C CNN
-	1    3200 9100
-	-1   0    0    1
-$EndComp
-Wire Wire Line
-	3350 9250 3200 9250
-Connection ~ 3200 9250
-Wire Wire Line
-	3200 9250 2950 9250
-Text Label 3200 8950 0    50   ~ 0
+P 3150 8825
+F 0 "C33" H 3035 8779 50  0000 R CNN
+F 1 "0.1uF10%" H 3035 8870 50  0000 R CNN
+F 2 "Capacitor_SMD:C_0603_1608Metric_Pad1.05x0.95mm_HandSolder" H 3188 8675 50  0001 C CNN
+F 3 "~" H 3150 8825 50  0001 C CNN
+	1    3150 8825
+	-1   0    0    1
+$EndComp
+Wire Wire Line
+	3300 8975 3150 8975
+Connection ~ 3150 8975
+Wire Wire Line
+	3150 8975 2900 8975
+Text Label 3150 8675 0    50   ~ 0
 V_BAT_AF_PROT-
-Text Label 2450 9650 0    50   ~ 0
+Text Label 2400 9375 0    50   ~ 0
 SRN_C
-Text Label 2450 9450 0    50   ~ 0
+Text Label 2400 9175 0    50   ~ 0
 SRP_C
 Wire Wire Line
-	2450 9450 2750 9450
-Wire Wire Line
-	2450 9650 2750 9650
-NoConn ~ 3150 9850
+	2400 9175 2700 9175
+Wire Wire Line
+	2400 9375 2700 9375
 Text HLabel 5600 7750 2    50   Output ~ 0
 PACK-
@@
 Wire Wire Line
 	3200 1200 3400 1200
+Wire Wire Line
+	3475 9275 3300 9275
+Text GLabel 3400 9575 2    50   Output ~ 0
+MCU_ANALOG_SENSOR_V
+$Comp
+L Device:R R40
+U 1 1 604D6224
+P 3250 9575
+F 0 "R40" V 3150 9575 50  0000 C CNN
+F 1 "10KR" V 3150 9750 50  0000 C CNN
+F 2 "Resistor_SMD:R_0603_1608Metric" V 3180 9575 50  0001 C CNN
+F 3 "~" H 3250 9575 50  0001 C CNN
+	1    3250 9575
+	0    1    1    0
+$EndComp
+$Comp
+L Device:D_Zener D15
+U 1 1 604D79E2
+P 3100 9725
+F 0 "D15" V 3054 9805 50  0000 L CNN
+F 1 "KDZVTR2.0B" V 3145 9805 50  0000 L CNN
+F 2 "Diode_SMD:D_SOD-123F" H 3100 9725 50  0001 C CNN
+F 3 "~" H 3100 9725 50  0001 C CNN
+	1    3100 9725
+	0    1    1    0
+$EndComp
+Connection ~ 3100 9575
+$Comp
+L power:GND #PWR017
+U 1 1 604D898C
+P 3100 9875
+F 0 "#PWR017" H 3100 9625 50  0001 C CNN
+F 1 "GND" H 3105 9702 50  0000 C CNN
+F 2 "" H 3100 9875 50  0001 C CNN
+F 3 "" H 3100 9875 50  0001 C CNN
+	1    3100 9875
+	1    0    0    -1
+$EndComp
+Text Notes 3700 9900 0    50   ~ 0
+2V reference, for offset. \nUsed in ADC compensation,\n And measuring negative current
 $EndSCHEMATC

Commit message: pre cleanup
Parts:
- R25: value 1mOhm1% -> 10mOhm1%
Changed lines of the file:
@@
 P 3050 7750
 F 0 "R25" V 2843 7750 50  0000 C CNN
-F 1 "1mOhm1%" V 2934 7750 50  0000 C CNN
+F 1 "10mOhm1%" V 2934 7750 50  0000 C CNN
 F 2 "Resistor_SMD:R_1206_3216Metric_Pad1.42x1.75mm_HandSolder" V 2980 7750 50  0001 C CNN
 F 3 "~" H 3050 7750 50  0001 C CNN
@@
 U 1 1 600100A1
 P 3150 5200
-F 0 "C32" V 3402 5200 50  0000 C CNN
-F 1 "1uF10%" V 3311 5200 50  0000 C CNN
+F 0 "C32" V 3075 5350 50  0000 C CNN
+F 1 "1uF10%" V 2975 5200 50  0000 C CNN
 F 2 "Capacitor_SMD:C_0603_1608Metric" H 3188 5050 50  0001 C CNN
 F 3 "~" H 3150 5200 50  0001 C CNN

Commit message: cleanup and energy managment scheeme started
Parts:
- removed C27, C28, C29, C30, C31, C32: 1uF10%, Capacitor_SMD:C_0603_1608Metric, symbol Device:C
- removed D16: TSZU52C10 RG, Diode_SMD:D_0603_1608Metric, symbol Device:D_Zener
- removed Q12: Si7938DP-T1-GE3, Package_SO:PowerPAK_SO-8_Dual, symbol rysboard:Si7938DP-T1-GE3
- removed R16: 1KR1%, Resistor_SMD:R_0603_1608Metric, symbol Device:R
- removed R17, R18, R19, R20: 33R5%, Resistor_SMD:R_0603_1608Metric, symbol Device:R
- removed R21, R30: 100R, Resistor_SMD:R_0603_1608Metric, symbol Device:R
- removed R25: 10mOhm1%, Resistor_SMD:R_1206_3216Metric_Pad1.42x1.75mm_HandSolder, symbol Device:R
- removed R31: 4.5KR, Resistor_SMD:R_0603_1608Metric_Pad1.05x0.95mm_HandSolder, symbol Device:R
- removed R32, R33: 1MR5%, symbol Device:R
- removed R34: 100KR, Resistor_SMD:R_0603_1608Metric_Pad1.05x0.95mm_HandSolder, symbol Device:R
- removed R35: 10KR, Resistor_SMD:R_0603_1608Metric, symbol Device:R
- removed R36: R, symbol Device:R
- removed R37: 470KR1%, Resistor_SMD:R_0603_1608Metric, symbol Device:R
- removed R38: 470KR5%, Resistor_SMD:R_0603_1608Metric, symbol Device:R
- removed TH1: Thermistor_NTC, symbol Device:Thermistor_NTC
- removed U11: bq77915, Package_SO:TSSOP-24_4.4x7.8mm_P0.65mm, symbol rysboard:bq77915
- added C?: 0.1uF, Capacitor_SMD:C_0603_1608Metric, symbol Device:C
- added D?: LED, LED_SMD:LED_0805_2012Metric, symbol Device:LED
- added F?: Fuse 3A, Fuse:Fuse_1206_3216Metric, symbol Device:Fuse
- added Q?: Si7938DP-T1-GE3, Package_SO:PowerPAK_SO-8_Dual, symbol rysboard:Si7938DP-T1-GE3
- added R?: 10mOhm1%, Resistor_SMD:R_1206_3216Metric_Pad1.42x1.75mm_HandSolder, symbol Device:R
- added R? (x5): 100R, Resistor_SMD:R_0603_1608Metric, symbol Device:R
- added R?: R, symbol Device:R
- added U?: LM74700, Package_TO_SOT_SMD:SOT-23-6, symbol Power_Management:LM74700
Connections:
- net PACK+: now also Q?.6 (D1), R?.1, U?.4 (CATHODE); no longer J7.2 (Pin_2)
- net PACK-: now also R?.1, R?.2
- net SRN_C: now also R?.1
- net SRP_C: now also R?.1
- net V_BAT_AF_PROT-: now also C?.1, D?.1 (K), R?.2, R?.2, U?.2 (GND)
- net V_CELL_3: now also R?.2; no longer J7.1 (Pin_1), Q13.6 (D1)
- net at D11.2 (A2), D12.1 (A1), Q14.6 (D1_1)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: now also R?.2; no longer J4.2 (Pin_2), J5.1 (Pin_1)
- net at D10.2 (A2), D11.1 (A1), Q14.3 (D2_1)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: now also R?.2; no longer J5.2 (Pin_2), J6.1 (Pin_1)
- net at D10.1 (A1), Q13.5 (D1): now also F?.1; no longer J6.2 (Pin_2)
- new net: J4.2 (Pin_2), J5.1 (Pin_1), R?.1
- new net: J5.2 (Pin_2), J6.1 (Pin_1), R?.1
- new net: F?.2, J6.2 (Pin_2)
- new net: J7.1 (Pin_1), Q13.6 (D1), R?.1
- new net: D?.2 (A), R?.2
- new net: C?.2, U?.1 (VCAP)
- new net: Q?.4 (G2), U?.5 (GATE)
- new net V_BAT_AF_PROT+: J7.2 (Pin_2), Q?.3 (S2), U?.3 (EN), U?.6 (ANODE)
- no-connect marks 3 -> 0
Other:
- note removed: "Balancing set at 50mA\n"
- note removed: "Battery Balancing\n"
- note removed: "Strona 29\n\n"
- note removed: "Table 9-3 \nPage 17"
- moved on the sheet: C24, C25, C26, C33, D10, D11, D12, D15, R40, U9

Commit message: started board project
Parts:
- added C27: 10uF, Capacitor_SMD:C_1206_3216Metric, symbol Device:C
- added C29: 47uF, Capacitor_Tantalum_SMD:CP_EIA-7343-31_Kemet-D, symbol Device:C
- R19: renamed from R?; value R -> 10K; footprint (none) -> Resistor_SMD:R_0603_1608Metric
- gave numbers to parts that had none: 11
- renumbered J7 to J20
Connections:
- net GND: now also C26.2
- net PACK+: now also C29.2
- net PACK-: now also C29.1
- net V_BAT_AF_PROT+: now also C27.2
- net V_BAT_AF_PROT-: now also C27.1; no longer C26.2
Other:
- note added: "Cap must be more than 0.07uF"
- note added: "ISO 7637-2 and ISO 16750-2 Compliant\n"
- note added: "Or More"
- moved on the sheet: C28, D7, Q9B, R19, R20, R21, R25, U7

Commit message: Bom finished pcb cleanup started
Parts:
- removed D10, D11, D12: TESDU5V0, Diode_SMD:D_0603_1608Metric_Pad1.05x0.95mm_HandSolder, symbol Device:D_TVS
- removed D7: LED, LED_SMD:LED_0805_2012Metric, symbol Device:LED
- removed Q13: SI7997DP-T1-GE3, Package_SO:PowerPAK_SO-8_Dual, symbol rysboard:SI7997DP-T1-GE3
- removed Q14: DMP2075UFDB-7-alt, SamacSys_Parts:DMP2075UFDB7, symbol SamacSys_Parts:DMP2075UFDB-7-alt
- removed U7: LM74700, Package_TO_SOT_SMD:SOT-23-6, symbol Power_Management:LM74700
- added IC1: LM74801QDRRRQ1, LM74801QDRRRQ1, symbol SamacSys_Parts:LM74801QDRRRQ1
- added Q2: FDG6304P, SOT65P210X110-6N, symbol SamacSys_Parts:FDG6304P
- added R10: 10KR, Resistor_SMD:R_0603_1608Metric, symbol Device:R
- added R8: 110KR, Resistor_SMD:R_0603_1608Metric, symbol Device:R
- R15: value 10KR -> 100R
- R16: value 100R -> 110KR
- R17: value 100R -> 10KR
- R19: value 10K -> 100R
- R22, R24: value 10KR -> 110KR
Connections:
- net PACK+: now also Q9.1 (S1), IC1.9 (OUT); no longer Q9.6 (D1), R19.1
- net V_BAT_AF_PROT+: now also J6.2 (Pin_2), IC1.2 (A), IC1.3 (VSNS); no longer J20.2 (Pin_2)
- net V_BAT_AF_PROT-: now also J20.1 (Pin_1), R17.2, IC1.7 (GND), R10.2; no longer C28.1, Q9.1 (S1)
- net V_CELL_1: now also R15.2; no longer R23.1
- net V_CELL_2: now also R19.2; no longer R22.1
- net at J4.1 (Pin_1): now also F1.2; no longer Q9.5 (D1)
- net at J4.2 (Pin_2), J5.1 (Pin_1): now also R16.2, Q2.3 (D2); no longer R17.1
- net at J5.2 (Pin_2), J6.1 (Pin_1): now also Q2.6 (D1), R8.2; no longer R16.1
- net at R18.1: now also IC1.4 (SW); no longer J20.1 (Pin_1)
- net at R15.1: now also Q2.4 (S2); no longer Q9.2 (G1)
- net at F1.1: now also J20.2 (Pin_2)
- net EN_12V: now reaches R24.2
- net EN_12V: now also IC1.6 (EN/UVLO)
- net at R23.2: now also R22.2, IC1.5 (OV)
- net +BATT: now reaches C28.2
- net +BATT: now also Q9.5 (D1), Q9.6 (D1), R22.1, IC1.10 (VS), IC1.12 (C)
- net at Q9.4 (G2): now also IC1.1 (DGATE)
- new net: C28.1, IC1.11 (CAP)
- new net: Q2.1 (S1), R19.1
- new net: IC1.8 (HGATE), Q9.2 (G1)
- new net: Q2.2 (G1), R10.1, R8.1
- new net: Q2.5 (G2), R16.1, R17.1
- no-connect marks 0 -> 1
Other:
- note added: "Overvoltage protection @ 15V"
- note removed: "ISO 7637-2 and ISO 16750-2 Compliant\n"
- moved on the sheet: C27, C28, C29, F1, J20, J4, J5, J6, R18, R20, R21, R25

Commit message: bom + excel ready
Parts:
- added R33: 10k1%, Resistor_SMD:R_0603_1608Metric, symbol Device:R
- C24, C25, C26, C28: value 0.1uF -> 100n
- C27: value 10uF -> 10u
- C33: value 0.1uF10% -> 100n
- IC1: footprint LM74801QDRRRQ1 -> SamacSys_Parts:LM74801QDRRRQ1
- Q2: footprint SOT65P210X110-6N -> SamacSys_Parts:SOT65P210X110-6N
- R10, R17, R23, R40: value 10KR -> 10k1%
Connections:
- net EN_12V: now also R33.2; no longer IC1.6 (EN/UVLO), R24.2
- net V_BAT_AF_PROT-: now also R23.1
- new net: IC1.6 (EN/UVLO), R24.2, R33.1
Other:
- moved on the sheet: R20, R21, R25
Changed lines of the file:
@@
 P 3125 8225
 F 0 "C25" V 3377 8225 50  0000 C CNN
-F 1 "0.1uF" V 3575 8225 50  0000 C CNN
+F 1 "100n" V 3575 8225 50  0000 C CNN
 F 2 "Capacitor_SMD:C_0603_1608Metric" H 3163 8075 50  0001 C CNN
 F 3 "~" H 3125 8225 50  0001 C CNN
@@
 P 2825 8375
 F 0 "C24" H 2675 8375 50  0000 C CNN
-F 1 "0.1uF" H 2675 8225 50  0000 C CNN
+F 1 "100n" H 2675 8225 50  0000 C CNN
 F 2 "Capacitor_SMD:C_0603_1608Metric" H 2863 8225 50  0001 C CNN
 F 3 "~" H 2825 8375 50  0001 C CNN
@@
 $EndComp
 Connection ~ 2825 8225
-$Comp
-L Device:C C26
-U 1 1 5FFFC289
-P 3425 8375
-F 0 "C26" H 3575 8375 50  0000 C CNN
-F 1 "0.1uF" H 3575 8225 50  0000 C CNN
-F 2 "Capacitor_SMD:C_0603_1608Metric" H 3463 8225 50  0001 C CNN
-F 3 "~" H 3425 8375 50  0001 C CNN
-	1    3425 8375
-	1    0    0    -1
-$EndComp
-Connection ~ 3425 8225
 Text Label 2875 8525 0    20   ~ 0
 V_BAT_AF_PROT-
@@
 P 4925 8150
 F 0 "R40" V 4825 8150 50  0000 C CNN
-F 1 "10KR" V 4825 8325 50  0000 C CNN
+F 1 "10k1%" V 4825 8325 50  0000 C CNN
 F 2 "Resistor_SMD:R_0603_1608Metric" V 4855 8150 50  0001 C CNN
 F 3 "~" H 4925 8150 50  0001 C CNN
@@
 P 4325 5125
 F 0 "C28" H 4500 5125 50  0000 C CNN
-F 1 "0.1uF" H 4500 5050 50  0000 C CNN
+F 1 "100n" H 4500 5050 50  0000 C CNN
 F 2 "Capacitor_SMD:C_0603_1608Metric" H 4363 4975 50  0001 C CNN
 F 3 "~" H 4325 5125 50  0001 C CNN
@@
 	0    -1   -1   0
 $EndComp
-Text Label 725  6575 0    50   ~ 0
+Text Label 725  6600 0    50   ~ 0
 V_BAT_AF_PROT-
 Connection ~ 4825 7550
@@
 Text Label 6575 7075 2    50   ~ 0
 SRP_C
-Text HLabel 7350 6575 2    50   Output ~ 0
+Text HLabel 7350 6600 2    50   Output ~ 0
 PACK-
 $Comp
 L Device:R R25
 U 1 1 6056575C
-P 7050 6800
-F 0 "R25" H 7200 6800 50  0000 R CNN
-F 1 "100R" H 7000 6800 50  0000 R CNN
-F 2 "Resistor_SMD:R_0603_1608Metric" V 6980 6800 50  0001 C CNN
-F 3 "~" H 7050 6800 50  0001 C CNN
-	1    7050 6800
+P 7050 6825
+F 0 "R25" H 7200 6825 50  0000 R CNN
+F 1 "100R" H 7000 6825 50  0000 R CNN
+F 2 "Resistor_SMD:R_0603_1608Metric" V 6980 6825 50  0001 C CNN
+F 3 "~" H 7050 6825 50  0001 C CNN
+	1    7050 6825
 	-1   0    0    1
 $EndComp
@@
 L Device:R R20
 U 1 1 6056538A
-P 6325 6800
-F 0 "R20" H 6275 6800 50  0000 R CNN
-F 1 "100R" H 6600 6800 50  0000 R CNN
-F 2 "Resistor_SMD:R_0603_1608Metric" V 6255 6800 50  0001 C CNN
-F 3 "~" H 6325 6800 50  0001 C CNN
-	1    6325 6800
+P 6325 6825
+F 0 "R20" H 6275 6825 50  0000 R CNN
+F 1 "100R" H 6600 6825 50  0000 R CNN
+F 2 "Resistor_SMD:R_0603_1608Metric" V 6255 6825 50  0001 C CNN
+F 3 "~" H 6325 6825 50  0001 C CNN
+	1    6325 6825
 	-1   0    0    1
 $EndComp
@@
 L Device:R R21
 U 1 1 60564FC5
-P 6675 6575
-F 0 "R21" V 6468 6575 50  0000 C CNN
-F 1 "10mOhm1%" V 6559 6575 50  0000 C CNN
-F 2 "Resistor_SMD:R_1206_3216Metric_Pad1.42x1.75mm_HandSolder" V 6605 6575 50  0001 C CNN
-F 3 "~" H 6675 6575 50  0001 C CNN
-	1    6675 6575
+P 6675 6600
+F 0 "R21" V 6468 6600 50  0000 C CNN
+F 1 "10mOhm1%" V 6559 6600 50  0000 C CNN
+F 2 "Resistor_SMD:R_1206_3216Metric_Pad1.42x1.75mm_HandSolder" V 6605 6600 50  0001 C CNN
+F 3 "~" H 6675 6600 50  0001 C CNN
+	1    6675 6600
 	0    1    1    0
 $EndComp
@@
 P 4825 7400
 F 0 "C33" H 4710 7354 50  0000 R CNN
-F 1 "0.1uF10%" H 4710 7445 50  0000 R CNN
+F 1 "100n" H 4710 7445 50  0000 R CNN
 F 2 "Capacitor_SMD:C_0603_1608Metric_Pad1.05x0.95mm_HandSolder" H 4863 7250 50  0001 C CNN
 F 3 "~" H 4825 7400 50  0001 C CNN
@@
 $EndComp
 Wire Wire Line
-	6325 6650 6325 6575
-Wire Wire Line
-	6325 6575 6525 6575
-Wire Wire Line
-	7050 6575 6825 6575
-Wire Wire Line
-	6325 7075 6325 6950
+	6325 6675 6325 6600
+Wire Wire Line
+	6325 6600 6525 6600
+Wire Wire Line
+	7050 6600 6825 6600
 Wire Wire Line
 	6800 7075 7050 7075
@@
 	6325 7075 6575 7075
 Wire Wire Line
-	7050 6650 7050 6575
-Wire Wire Line
-	7050 6950 7050 7075
-Connection ~ 7050 6575
+	7050 6675 7050 6600
+Wire Wire Line
+	7050 6975 7050 7075
+Connection ~ 7050 6600
 Text Label 600  4750 0    50   ~ 0
 V_BAT_AF_PROT+
@@
 P 2475 5950
 F 0 "C27" H 2650 5950 50  0000 C CNN
-F 1 "10uF" H 2650 5875 50  0000 C CNN
+F 1 "10u" H 2650 5875 50  0000 C CNN
 F 2 "Capacitor_SMD:C_1206_3216Metric" H 2513 5800 50  0001 C CNN
 F 3 "~" H 2475 5950 50  0001 C CNN
@@
 $EndComp
 Wire Wire Line
-	725  6575 2475 6575
-Wire Wire Line
-	2475 6100 2475 6575
-Connection ~ 2475 6575
+	725  6600 2475 6600
 $Comp
 L Device:C C29
@@
 Or More
 Wire Wire Line
-	7050 6575 7250 6575
-Connection ~ 7250 6575
-Wire Wire Line
-	7250 6575 7350 6575
+	7050 6600 7250 6600
+Connection ~ 7250 6600
+Wire Wire Line
+	7250 6600 7350 6600
 Wire Wire Line
 	7250 4725 7250 5125
@@
 	0    1    1    0
 $EndComp
-Text Label 4875 1150 2    50   ~ 0
+Text Label 4400 1150 2    50   ~ 0
 V_BAT_AF_PROT+
 Text Notes 4425 950  0    50   ~ 0
@@
 U 1 1 5FE3248E
 P 1750 3650
-F 0 "J20" H 1668 3325 50  0000 C CNN
-F 1 "Power_SW" H 1668 3416 50  0000 C CNN
+F 0 "J20" V 1950 3650 50  0000 C CNN
+F 1 "Power_SW" V 1850 3650 50  0000 C CNN
 F 2 "Connector_Molex:Molex_Micro-Fit_3.0_43045-0212_2x01_P3.00mm_Vertical" H 1750 3650 50  0001 C CNN
 F 3 "~" H 1750 3650 50  0001 C CNN
@@
 Wire Wire Line
 	1075 2950 1075 3250
-Wire Wire Line
-	1075 1150 4875 1150
 $Comp
 L SamacSys_Parts:FDG6304P Q2
@@
 F 0 "Q2" H 2550 2615 50  0000 C CNN
 F 1 "FDG6304P" H 2550 2524 50  0000 C CNN
-F 2 "SOT65P210X110-6N" H 2900 2450 50  0001 L CNN
+F 2 "SamacSys_Parts:SOT65P210X110-6N" H 2900 2450 50  0001 L CNN
 F 3 "https://componentsearchengine.com/Datasheets/1/FDG6304P.pdf" H 2900 2350 50  0001 L CNN
 F 4 "Mosfet Array 2 P-Channel (Dual) 25V 410mA 300mW Surface Mount SC-70-6" H 2900 2250 50  0001 L CNN "Description"
@@
 P 3100 3300
 F 0 "R17" V 2893 3300 50  0000 C CNN
-F 1 "10KR" V 2984 3300 50  0000 C CNN
+F 1 "10k1%" V 2984 3300 50  0000 C CNN
 F 2 "Resistor_SMD:R_0603_1608Metric" V 3030 3300 50  0001 C CNN
 F 3 "~" H 3100 3300 50  0001 C CNN
@@
 P 1925 3300
 F 0 "R10" V 1718 3300 50  0000 C CNN
-F 1 "10KR" V 1809 3300 50  0000 C CNN
+F 1 "10k1%" V 1809 3300 50  0000 C CNN
 F 2 "Resistor_SMD:R_0603_1608Metric" V 1855 3300 50  0001 C CNN
 F 3 "~" H 1925 3300 50  0001 C CNN
@@
 Wire Wire Line
 	6225 4750 6225 4725
-Wire Wire Line
-	2475 5800 2475 4750
-Connection ~ 2475 4750
-Wire Wire Line
-	2475 4750 3600 4750
-Wire Wire Line
-	600  4750 2475 4750
 Connection ~ 3600 5600
 Wire Wire Line
@@
 F 0 "IC1" H 4400 5800 50  0000 C CNN
 F 1 "LM74801QDRRRQ1" H 4400 5625 50  0000 C CNN
-F 2 "LM74801QDRRRQ1" H 5625 5850 50  0001 L CNN
+F 2 "SamacSys_Parts:LM74801QDRRRQ1" H 5625 5850 50  0001 L CNN
 F 3 "https://www.ti.com/lit/gpn/LM7480-Q1" H 5625 5750 50  0001 L CNN
 F 4 "3-V TO 65-V, AUTOMOTIVE IDEAL DI" H 5625 5650 50  0001 L CNN "Description"
@@
 Wire Wire Line
 	5600 4750 6225 4750
-Connection ~ 4375 6575
-Connection ~ 6325 6575
+Connection ~ 6325 6600
 $Comp
 L power:+BATT #PWR024
@@
 Wire Wire Line
 	4450 4750 4625 4750
-Wire Wire Line
-	7250 5425 7250 6575
-Wire Wire Line
-	4375 6575 5250 6575
 $Comp
 L Device:R R24
 U 1 1 60A297BF
 P 5250 6425
-F 0 "R24" V 5043 6425 50  0000 C CNN
-F 1 "110KR" V 5134 6425 50  0000 C CNN
+F 0 "R24" H 5425 6500 50  0000 C CNN
+F 1 "110KR" H 5425 6425 50  0000 C CNN
 F 2 "Resistor_SMD:R_0603_1608Metric" V 5180 6425 50  0001 C CNN
 F 3 "~" H 5250 6425 50  0001 C CNN
@@
 	-1   0    0    1
 $EndComp
-Connection ~ 5250 6575
 Wire Wire Line
 	5250 6275 5250 6125
@@
 	5250 6125 5150 6125
 Wire Wire Line
-	5250 6575 6325 6575
-Text HLabel 5250 6125 2    50   Input ~ 0
+	5250 6600 6325 6600
+Text HLabel 5550 6125 2    50   Input ~ 0
 EN_12V
 $Comp
@@
 P 3600 6450
 F 0 "R23" V 3393 6450 50  0000 C CNN
-F 1 "10KR" V 3484 6450 50  0000 C CNN
+F 1 "10k1%" V 3484 6450 50  0000 C CNN
 F 2 "Resistor_SMD:R_0603_1608Metric" V 3530 6450 50  0001 C CNN
 F 3 "~" H 3600 6450 50  0001 C CNN
@@
 Wire Wire Line
 	4525 5125 4625 5125
-Wire Wire Line
-	2475 6575 4375 6575
+$Comp
+L Device:R R33
+U 1 1 60917467
+P 5400 6125
+F 0 "R33" V 5193 6125 50  0000 C CNN
+F 1 "10k1%" V 5284 6125 50  0000 C CNN
+F 2 "Resistor_SMD:R_0603_1608Metric" V 5330 6125 50  0001 C CNN
+F 3 "~" H 5400 6125 50  0001 C CNN
+	1    5400 6125
+	0    -1   -1   0
+$EndComp
+Connection ~ 5250 6125
+Wire Wire Line
+	2475 6600 3600 6600
+Wire Wire Line
+	4375 6600 4375 6575
+Connection ~ 3600 6600
+Wire Wire Line
+	3600 6600 4375 6600
+Wire Wire Line
+	5250 6575 5250 6600
+Wire Wire Line
+	5250 6600 4375 6600
+Connection ~ 4375 6600
+Connection ~ 5250 6600
+Wire Wire Line
+	6325 7075 6325 6975
+Wire Wire Line
+	7250 5425 7250 6600
+Connection ~ 2475 6600
+Wire Wire Line
+	2475 6100 2475 6600
+Wire Wire Line
+	4400 1150 1075 1150
+Wire Wire Line
+	600  4750 2475 4750
+Wire Wire Line
+	2475 5800 2475 4750
+Connection ~ 2475 4750
+Wire Wire Line
+	2475 4750 3600 4750
+Connection ~ 3425 8225
+$Comp
+L Device:C C26
+U 1 1 5FFFC289
+P 3425 8375
+F 0 "C26" H 3575 8375 50  0000 C CNN
+F 1 "100n" H 3575 8225 50  0000 C CNN
+F 2 "Capacitor_SMD:C_0603_1608Metric" H 3463 8225 50  0001 C CNN
+F 3 "~" H 3425 8375 50  0001 C CNN
+	1    3425 8375
+	1    0    0    -1
+$EndComp
 $EndSCHEMATC

Commit message: New Layout done TODo Error Check
Parts:
- removed C29: 47uF, Capacitor_Tantalum_SMD:CP_EIA-7343-31_Kemet-D, symbol Device:C
Other:
- note removed: "Or More"
Changed lines of the file:
@@
 Wire Wire Line
 	725  6600 2475 6600
-$Comp
-L Device:C C29
-U 1 1 6059B38B
-P 7250 5275
-F 0 "C29" H 7425 5275 50  0000 C CNN
-F 1 "47uF" H 7425 5200 50  0000 C CNN
-F 2 "Capacitor_Tantalum_SMD:CP_EIA-7343-31_Kemet-D" H 7288 5125 50  0001 C CNN
-F 3 "~" H 7250 5275 50  0001 C CNN
-	1    7250 5275
-	-1   0    0    1
-$EndComp
-Connection ~ 7250 4725
-Wire Wire Line
-	7250 4725 7325 4725
-Text Notes 7450 5250 0    50   ~ 0
-Or More
-Wire Wire Line
-	7050 6600 7250 6600
-Connection ~ 7250 6600
-Wire Wire Line
-	7250 6600 7350 6600
-Wire Wire Line
-	7250 4725 7250 5125
 Wire Wire Line
 	2825 8525 2875 8525
@@
 	3600 4750 3775 4750
 Wire Wire Line
-	6225 4725 7250 4725
-Wire Wire Line
 	5025 4750 5600 4750
 Wire Wire Line
@@
 Wire Wire Line
 	6325 7075 6325 6975
-Wire Wire Line
-	7250 5425 7250 6600
 Connection ~ 2475 6600
 Wire Wire Line
@@
 	1    0    0    -1
 $EndComp
+Wire Wire Line
+	7050 6600 7350 6600
+Wire Wire Line
+	6225 4725 7325 4725
 $EndSCHEMATC
