File: s24v_capacitor_banks.kicad_sch (KiCad schematic)
At the start: 18 parts

Commit message: Finished motor drivers schematic
Still need to connect all the connectors and sort out old unused connections
Parts:
- removed C15, C16, C17, C18, C19, C20, C21, C22, C23, C24, C25, C26, C27, C28, C29, C30, C31, C32: 22uF, Capacitor_SMD:C_0805_2012Metric, symbol Device:C
Other:
- note removed: "Input Rail Capacitor Bank (110uF)"
- note removed: "Output Rail Capacitor Bank (286uF)"
